File: site/public/schematics/5f6a.kicad_sch (KiCad schematic)
At the start: 59 parts, among them T3 2R sec

Commit message: BOMs for 5E3/5F6-A, cross-artifact CI gates, visitor-voice notes, REVIEW.md
- bom.yaml for both new amps (60+ designators), refs matching their
  schematics exactly; 5F6-A PI tubes renamed V3A/V3B for consistent
  bottle numbering
- validate.py: verified amps now require the full artifact set
  (netlist, voltages, notes, schematic, BOM) and every BOM designator
  must reconcile with the schematic in both directions
- All three circuit stories rewritten in visitor voice (internal
  working-notes language removed — e.g. the 5E3 "secondary sources
  garble" heading)
- docs/REVIEW.md: the two-layer QA contract (deterministic CI gates +
  post-deploy editorial/accuracy judge pass on rendered pages)

Co-Authored-By: Claude Opus 4.8 (1M context) <noreply@anthropic.com>
Parts:
- removed PIA, PIB: 12AX7, symbol cx:TRIODE
- added V3A, V3B: 12AX7, symbol cx:TRIODE
Connections:
- net at C8.1, RLA.2: now also V3A.1 (P)
- net at C7.2, RGB.2: now also V3B.2 (G)
- net at C9.1, RLB.2: now also V3B.1 (P)
- net at RTAIL.1: now also V3A.3 (K), V3B.3 (K)
- net at C6.2, RGA.1: now also V3A.2 (G)
Other:
- note added: "47 pF balance cap V3A grid-plate omitted (AC only) · NFB 27k + presence 5k join the tail foot at ~0 V DC"
- note removed: "47 pF balance cap PIA grid-plate omitted (AC only) · NFB 27k + presence 5k join the tail foot at ~0 V DC"
Changed lines of the file:
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@@
   (symbol (lib_id "cx:TRIODE") (at 176.53 92 0) (unit 1)
     (in_bom yes) (on_board yes)
-    (property "Reference" "PIA" (at 182.53 85.6 0) (effects (font (size 1.27 1.27)) (justify left)))
+    (property "Reference" "V3A" (at 182.53 85.6 0) (effects (font (size 1.27 1.27)) (justify left)))
     (property "Value" "12AX7" (at 182.53 88 0) (effects (font (size 1.27 1.27)) (justify left))))
   (wire (pts (xy 168.91 92) (xy 168.91 92))
@@
   (symbol (lib_id "cx:TRIODE") (at 176.53 126 0) (unit 1)
     (in_bom yes) (on_board yes)
-    (property "Reference" "PIB" (at 182.53 119.6 0) (effects (font (size 1.27 1.27)) (justify left)))
+    (property "Reference" "V3B" (at 182.53 119.6 0) (effects (font (size 1.27 1.27)) (justify left)))
     (property "Value" "12AX7" (at 182.53 122 0) (effects (font (size 1.27 1.27)) (justify left))))
   (wire (pts (xy 176.53 84.38) (xy 176.53 80.9))
@@
   (wire (pts (xy 158.75 116.62) (xy 168.91 116.62))
     (stroke (width 0) (type default)))
-  (text "47 pF balance cap PIA grid-plate omitted (AC only) · NFB 27k + presence 5k join the tail foot at ~0 V DC" (at 150 145 0)
+  (text "47 pF balance cap V3A grid-plate omitted (AC only) · NFB 27k + presence 5k join the tail foot at ~0 V DC" (at 150 145 0)
     (effects (font (size 1.1 1.1)) (justify left)))
   (wire (pts (xy 176.53 80.9) (xy 194.31 80.9))
@@
   (global_label "GND" (shape input) (at 142.24 185.42 270)
     (effects (font (size 1.27 1.27)) (justify left)))
-  (global_label "HT_B" (shape input) (at 165.1 172.72 180)
-    (effects (font (size 1.27 1.27)) (justify left)))
-  (wire (pts (xy 165.1 172.72) (xy 168.91 172.72))
-    (stroke (width 0) (type default)))
-  (symbol (lib_id "cx:DIODE_SS") (at 173.99 172.72 0) (unit 1)
-    (in_bom yes) (on_board yes)
-    (property "Reference" "D1" (at 171.99 167.32 0) (effects (font (size 1.27 1.27)) (justify left)))
-    (property "Value" "SEL" (at 171.99 169.72 0) (effects (font (size 1.27 1.27)) (justify left))))
-  (wire (pts (xy 179.07 172.72) (xy 182.88 172.72))
-    (stroke (width 0) (type default)))
-  (symbol (lib_id "cx:R") (at 186.69 172.72 90) (unit 1)
-    (in_bom yes) (on_board yes)
-    (property "Reference" "RB1" (at 183.49 166.72 270) (effects (font (size 1.27 1.27)) (justify left)))
-    (property "Value" "15k" (at 183.49 169.12 270) (effects (font (size 1.27 1.27)) (justify left))))
-  (wire (pts (xy 182.88 172.72) (xy 182.88 172.72))
-    (stroke (width 0) (type default)))
-  (wire (pts (xy 190.5 172.72) (xy 198.12 172.72))
-    (stroke (width 0) (type default)))
-  (junction (at 193.04 172.72) (diameter 0) (color 0 0 0 0))
-  (symbol (lib_id "cx:R") (at 193.04 176.53 0) (unit 1)
-    (in_bom yes) (on_board yes)
-    (property "Reference" "RB2" (at 195.24 173.33 0) (effects (font (size 1.27 1.27)) (justify left)))
-    (property "Value" "56k" (at 195.24 175.73 0) (effects (font (size 1.27 1.27)) (justify left))))
-  (global_label "GND" (shape input) (at 193.04 180.34 270)
-    (effects (font (size 1.27 1.27)) (justify left)))
-  (junction (at 195.58 172.72) (diameter 0) (color 0 0 0 0))
-  (symbol (lib_id "cx:C") (at 195.58 176.53 0) (unit 1)
-    (in_bom yes) (on_board yes)
-    (property "Reference" "C15" (at 197.78 173.33 0) (effects (font (size 1.27 1.27)) (justify left)))
-    (property "Value" "8u" (at 197.78 175.73 0) (effects (font (size 1.27 1.27)) (justify left))))
-  (global_label "GND" (shape input) (at 195.58 180.34 270)
-    (effects (font (size 1.27 1.27)) (justify left)))
-  (global_label "-48V" (shape input) (at 198.12 172.72 0)
-    (effects (font (size 1.27 1.27)) (justify left)))
-  (text "bias caps 8u/150V x2 (one shown)" (at 168 186 0)
+  (global_label "HT_B" (shape input) (at 138.1 172.72 180)
+    (effects (font (size 1.27 1.27)) (justify left)))
+  (wire (pts (xy 138.1 172.72) (xy 141.91 172.72))
+    (stroke (width 0) (type default)))
+  (symbol (lib_id "cx:DIODE_SS") (at 146.99 172.72 0) (unit 1)
+    (in_bom yes) (on_board yes)
+    (property "Reference" "D1" (at 144.99 167.32 0) (effects (font (size 1.27 1.27)) (justify left)))
+    (property "Value" "SEL" (at 144.99 169.72 0) (effects (font (size 1.27 1.27)) (justify left))))
+  (wire (pts (xy 152.07 172.72) (xy 155.88 172.72))
+    (stroke (width 0) (type default)))
+  (symbol (lib_id "cx:R") (at 159.69 172.72 90) (unit 1)
+    (in_bom yes) (on_board yes)
+    (property "Reference" "RB1" (at 156.49 166.72 270) (effects (font (size 1.27 1.27)) (justify left)))
+    (property "Value" "15k" (at 156.49 169.12 270) (effects (font (size 1.27 1.27)) (justify left))))
+  (wire (pts (xy 155.88 172.72) (xy 155.88 172.72))
+    (stroke (width 0) (type default)))
+  (wire (pts (xy 163.5 172.72) (xy 171.12 172.72))
+    (stroke (width 0) (type default)))
+  (junction (at 166.04 172.72) (diameter 0) (color 0 0 0 0))
+  (symbol (lib_id "cx:R") (at 166.04 176.53 0) (unit 1)
+    (in_bom yes) (on_board yes)
+    (property "Reference" "RB2" (at 168.24 173.33 0) (effects (font (size 1.27 1.27)) (justify left)))
+    (property "Value" "56k" (at 168.24 175.73 0) (effects (font (size 1.27 1.27)) (justify left))))
+  (global_label "GND" (shape input) (at 166.04 180.34 270)
+    (effects (font (size 1.27 1.27)) (justify left)))
+  (junction (at 168.58 172.72) (diameter 0) (color 0 0 0 0))
+  (symbol (lib_id "cx:C") (at 168.58 176.53 0) (unit 1)
+    (in_bom yes) (on_board yes)
+    (property "Reference" "C15" (at 170.78 173.33 0) (effects (font (size 1.27 1.27)) (justify left)))
+    (property "Value" "8u" (at 170.78 175.73 0) (effects (font (size 1.27 1.27)) (justify left))))
+  (global_label "GND" (shape input) (at 168.58 180.34 270)
+    (effects (font (size 1.27 1.27)) (justify left)))
+  (global_label "-48V" (shape input) (at 171.12 172.72 0)
+    (effects (font (size 1.27 1.27)) (justify left)))
+  (text "bias caps 8u/150V x2 (one shown)" (at 145 186.5 0)
     (effects (font (size 1.1 1.1)) (justify left)))
   (sheet_instances (path "/" (page "1")))
