File: site/public/schematics/5f4.kicad_sch (KiCad schematic)
At the start: 66 parts, among them T3 45216

Commit message: Fix: site copies of 29 sheets re-synced; regenerate step syncs before the drift check
- the drawing scripts write amps/; site/public/schematics is refreshed by
  site/scripts/sync-assets.mjs, which CI only ran inside the site build, so
  the fixer commits carried stale copies and the new drift gate caught them
- CI now syncs immediately after regenerating and diffs both trees; the
  AGENTS.md regenerate command does the same

Co-Authored-By: Claude Fable 5.1 <noreply@anthropic.com>
Claude-Session: https://claude.ai/code/session_01KBMfdh37HmCL2iWcBiL5J1
Parts:
- removed RB1: 6.8k, symbol cx:R
- removed RD1, RD2: 10k, symbol cx:R
- added C12, C13: 16u, symbol cx:C
- added D1: SEL, symbol cx:DIODE_SS
- RB1: renamed from D1; value SEL -> 6.8k; symbol cx:DIODE_SS -> cx:R
- RD1: renamed from C12; value 16u -> 10k; symbol cx:C -> cx:R
- RD2: renamed from C13; value 16u -> 10k; symbol cx:C -> cx:R
Connections:
- net -40V: now also RB1.2
- net B+2: now also C12.1
- net B+3: now also RD1.2, C13.1
- net B+4: now also RD2.2
- net GND: now also VR1.3, VR2.3, C12.2, C13.2; no longer RD1.2, RD2.2
- net HT_B: now also D1.1 (A); no longer RB1.1 (A)
- net at C9.2, R5s.1: no longer RGL1.1
- net at R6s.2, V5.2 (G1): now also RGL2.1
- net at R5s.2, V4.2 (G1): now also RGL1.1
- net at C10.2, R6s.1: no longer RGL2.1
- new net: D1.2 (K), RB1.1
Other:
- moved on the sheet: R5s
Changed lines of the file:
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@@
   (symbol (lib_id "cx:POT") (at 64.678 30.988 0) (unit 1)
     (in_bom yes) (on_board yes)
-    (property "Reference" "VR1" (at 63.662 35.328 0) (effects (font (size 1.27 1.27)) (justify left)))
-    (property "Value" "1M vol" (at 63.662 37.728 0) (effects (font (size 1.27 1.27)) (justify left))))
-  (global_label "GND" (shape input) (at 64.678 38.608 270)
+    (property "Reference" "VR1" (at 49.9568 29.348 0) (effects (font (size 1.27 1.27)) (justify left)))
+    (property "Value" "1M vol" (at 49.9568 31.748 0) (effects (font (size 1.27 1.27)) (justify left))))
+  (global_label "GND" (shape input) (at 64.678 34.798 270)
     (effects (font (size 1.27 1.27)) (justify right)))
   (wire (pts (xy 69.758 30.988) (xy 72.298 30.988))
@@
     (property "Reference" "VR2" (at 56.5568 63.348 0) (effects (font (size 1.27 1.27)) (justify left)))
     (property "Value" "1M vol" (at 56.5568 65.748 0) (effects (font (size 1.27 1.27)) (justify left))))
-  (global_label "GND" (shape input) (at 64.678 72.608 270)
+  (global_label "GND" (shape input) (at 64.678 68.798 270)
     (effects (font (size 1.27 1.27)) (justify right)))
   (wire (pts (xy 69.758 64.988) (xy 72.298 64.988))
@@
   (wire (pts (xy 196.758 27.178) (xy 196.758 30.278))
     (stroke (width 0) (type default)))
-  (wire (pts (xy 196.758 30.278) (xy 199.298 30.278))
-    (stroke (width 0) (type default)))
-  (symbol (lib_id "cx:R") (at 203.108 30.278 90) (unit 1)
-    (in_bom yes) (on_board yes)
-    (property "Reference" "R5s" (at 199.908 24.278 270) (effects (font (size 1.27 1.27)) (justify left)))
-    (property "Value" "1.5k" (at 199.908 26.678 270) (effects (font (size 1.27 1.27)) (justify left))))
   (symbol (lib_id "cx:PENTODE") (at 212.618 29.643 0) (unit 1)
     (in_bom yes) (on_board yes)
     (property "Reference" "V4" (at 218.818 22.043 0) (effects (font (size 1.27 1.27)) (justify left)))
     (property "Value" "6L6G" (at 218.818 24.443 0) (effects (font (size 1.27 1.27)) (justify left))))
-  (wire (pts (xy 206.918 30.278) (xy 204.998 30.278))
-    (stroke (width 0) (type default)))
-  (junction (at 199.298 30.278) (diameter 0) (color 0 0 0 0))
-  (symbol (lib_id "cx:R") (at 199.298 34.088 0) (unit 1)
-    (in_bom yes) (on_board yes)
-    (property "Reference" "RGL1" (at 201.214 32.448 0) (effects (font (size 1.27 1.27)) (justify left)))
-    (property "Value" "220k" (at 201.214 34.848 0) (effects (font (size 1.27 1.27)) (justify left))))
-  (wire (pts (xy 199.298 37.898) (xy 199.298 40.438))
-    (stroke (width 0) (type default)))
-  (global_label "-40V" (shape input) (at 199.298 40.438 270)
+  (symbol (lib_id "cx:R") (at 201.188 30.278 90) (unit 1)
+    (in_bom yes) (on_board yes)
+    (property "Reference" "R5s" (at 197.988 24.278 270) (effects (font (size 1.27 1.27)) (justify left)))
+    (property "Value" "1.5k" (at 197.988 26.678 270) (effects (font (size 1.27 1.27)) (justify left))))
+  (wire (pts (xy 196.758 30.278) (xy 197.378 30.278))
+    (stroke (width 0) (type default)))
+  (junction (at 204.998 30.278) (diameter 0) (color 0 0 0 0))
+  (symbol (lib_id "cx:R") (at 204.998 34.088 0) (unit 1)
+    (in_bom yes) (on_board yes)
+    (property "Reference" "RGL1" (at 195.598 35.088 0) (effects (font (size 1.27 1.27)) (justify left)))
+    (property "Value" "220k" (at 195.598 37.488 0) (effects (font (size 1.27 1.27)) (justify left))))
+  (wire (pts (xy 204.998 37.898) (xy 204.998 40.438))
+    (stroke (width 0) (type default)))
+  (global_label "-40V" (shape input) (at 204.998 40.438 270)
     (effects (font (size 1.27 1.27)) (justify right)))
   (wire (pts (xy 220.238 29.008) (xy 222.778 29.008))
@@
   (wire (pts (xy 187.018 82.278) (xy 196.758 82.278))
     (stroke (width 0) (type default)))
-  (wire (pts (xy 196.758 82.278) (xy 199.298 82.278))
-    (stroke (width 0) (type default)))
-  (symbol (lib_id "cx:R") (at 203.108 82.278 90) (unit 1)
-    (in_bom yes) (on_board yes)
-    (property "Reference" "R6s" (at 199.908 76.278 270) (effects (font (size 1.27 1.27)) (justify left)))
-    (property "Value" "1.5k" (at 199.908 78.678 270) (effects (font (size 1.27 1.27)) (justify left))))
   (symbol (lib_id "cx:PENTODE") (at 212.618 81.643 0) (unit 1)
     (in_bom yes) (on_board yes)
     (property "Reference" "V5" (at 218.818 74.043 0) (effects (font (size 1.27 1.27)) (justify left)))
     (property "Value" "6L6G" (at 218.818 76.443 0) (effects (font (size 1.27 1.27)) (justify left))))
-  (wire (pts (xy 206.918 82.278) (xy 204.998 82.278))
-    (stroke (width 0) (type default)))
-  (junction (at 199.298 82.278) (diameter 0) (color 0 0 0 0))
-  (symbol (lib_id "cx:R") (at 199.298 86.088 0) (unit 1)
-    (in_bom yes) (on_board yes)
-    (property "Reference" "RGL2" (at 201.214 84.448 0) (effects (font (size 1.27 1.27)) (justify left)))
-    (property "Value" "220k" (at 201.214 86.848 0) (effects (font (size 1.27 1.27)) (justify left))))
-  (wire (pts (xy 199.298 89.898) (xy 199.298 92.438))
-    (stroke (width 0) (type default)))
-  (global_label "-40V" (shape input) (at 199.298 92.438 270)
+  (symbol (lib_id "cx:R") (at 201.188 82.278 90) (unit 1)
+    (in_bom yes) (on_board yes)
+    (property "Reference" "R6s" (at 197.988 76.278 270) (effects (font (size 1.27 1.27)) (justify left)))
+    (property "Value" "1.5k" (at 197.988 78.678 270) (effects (font (size 1.27 1.27)) (justify left))))
+  (wire (pts (xy 196.758 82.278) (xy 197.378 82.278))
+    (stroke (width 0) (type default)))
+  (junction (at 204.998 82.278) (diameter 0) (color 0 0 0 0))
+  (symbol (lib_id "cx:R") (at 204.998 86.088 0) (unit 1)
+    (in_bom yes) (on_board yes)
+    (property "Reference" "RGL2" (at 195.598 87.088 0) (effects (font (size 1.27 1.27)) (justify left)))
+    (property "Value" "220k" (at 195.598 89.488 0) (effects (font (size 1.27 1.27)) (justify left))))
+  (wire (pts (xy 204.998 89.898) (xy 204.998 92.438))
+    (stroke (width 0) (type default)))
+  (global_label "-40V" (shape input) (at 204.998 92.438 270)
     (effects (font (size 1.27 1.27)) (justify right)))
   (wire (pts (xy 220.238 81.008) (xy 222.778 81.008))
