File: site/public/schematics/jtm45.kicad_sch (KiCad schematic)
At the start: 63 parts, among them T3 OT

Commit message: Re-export the worklists, site copies and card for the JTM45 corrections
op-points, loadlines, sheet-board, electrolytics (JTM45 7/7 cans right)
and verification-freshness regenerated by their own exporters; the site's
schematic and layout copies re-synced and the JTM45 link card re-rendered.
JTM45 stays "never stamped" in the freshness list with a new fingerprint.

Co-Authored-By: Claude Opus 5.5 <noreply@anthropic.com>
Claude-Session: https://claude.ai/code/session_01KBMfdh37HmCL2iWcBiL5J1
Signed-off-by: AnalogMaker <theanalogmaker@gmail.com>
Parts:
- removed C13: 16u, symbol cx:C
- removed C17: .1u, symbol cx:C
- removed C5: .02u, symbol cx:C
- removed L1: 20H, symbol cx:CHOKE
- removed RD1: 8.2k, symbol cx:R
- removed RK1: 820, symbol cx:R
- removed RL3: 100k, symbol cx:R
- removed RSL: 56k, symbol cx:R
- removed RT2: 10k, symbol cx:R
- removed V6: KT66, symbol cx:PENTODE
- removed VR6: 5k pres, symbol cx:POT
- added C15: .05u, symbol cx:C
- added C18: 8u, symbol cx:C
- added C19: 56p, symbol cx:C
- added C20: C, symbol cx:C
- added C4: 270p, symbol cx:C
- added C6: .02u, symbol cx:C
- added D1: diode, symbol cx:DIODE_SS
- added RB2: R, symbol cx:R
- added RB3: 16k, symbol cx:R
- added RD2: 10k, symbol cx:R
- added RGA: 1M, symbol cx:R
- added RGL1: 220k, symbol cx:R
- added RS3: 1k 2W, symbol cx:R
- added T3: OT, symbol cx:OT_PP
- added V3A: ECC83, symbol cx:TRIODE
- added V3B: ECC83 CF, symbol cx:TRIODE
- added V5: KT66, symbol cx:PENTODE
- C12: value 16u -> 32u
- C13: renamed from C15; value .05u -> 16u
- C16: value 25u -> elec
- C17: renamed from RGL1; value 220k -> .1u; symbol cx:R -> cx:C
- C5: renamed from VR4; value 1M bass -> .02u; symbol cx:POT -> cx:C
- L1: renamed from RD2; value 10k -> 20H; symbol cx:R -> cx:CHOKE
- RB1: value 150k -> R
- RD1: renamed from D1; value 1N4007 -> 8.2k; symbol cx:DIODE_SS -> cx:R
- RK1: renamed from V3A; value ECC83 -> 820; symbol cx:TRIODE -> cx:R
- RL3: renamed from V3B; value ECC83 CF -> 100k; symbol cx:TRIODE -> cx:R
- RS1, RS2: value 1k 2W -> 470 1W
- RSL: renamed from C4; value 270p -> 56k; symbol cx:C -> cx:R
- RT2: renamed from RGA; value 1M -> 10k
- V6: renamed from T3; value OT -> KT66; symbol cx:OT_PP -> cx:PENTODE
- VR4: renamed from C6; value .02u -> 1M bass; symbol cx:C -> cx:POT
- VR6: renamed from V5; value KT66 -> 5k pres; symbol cx:PENTODE -> cx:POT
Connections:
- net B+1: now also L1.1, C15.1; no longer V6.2 (CT)
- net B+2: now also L1.2, RD1.1, RS3.1, T3.2 (CT); no longer RS1.2, RS2.2
- net B+3: now also C13.1, RD1.2, RD2.1; no longer L1.1
- net B+4: now also RD2.2, V3B.1 (P); no longer L1.2
- net BRIGHT: now also R2s.1; no longer R1s.1
- net GND: now also C17.2, RK1.2, V6.4 (K), VR6.3, C15.2, C18.2, RB2.2, T3.5 (SEC_C), V5.4 (K); no longer V6.5 (SEC_C), VR6.4 (K)
- net HT_B: now also RB1.1; no longer RD1.2 (K)
- net NORMAL: now also R1s.1; no longer R2s.1
- net PRES: now also RT2.2, VR6.1
- net SPKR: now also T3.4 (SEC_H); no longer V6.4 (SEC_H)
- net at C10.1, RLB.2, V4B.1 (P): now also C20.2
- net at C10.2, RGL2.1: now also V6.2 (G1)
- net at RKCF.1, RSL.1: now also C4.1, V3B.3 (K); no longer RL3.3 (K)
- net at RSL.2: now also C5.1, C6.1; no longer VR3.1
- net at V6.1 (P): now also T3.3 (PRI_B); no longer VR6.1 (P)
- net at C17.1, VR6.2 (W): no longer C9.2
- net at RS1.1: now also V5.3 (G2); no longer VR6.3 (G2)
- net at V6.3 (G2): now also RS2.1
- net at VR3.3: now also C5.2, VR4.1; no longer C5.1
- net at RL3.2: now also V3A.1 (P), V3B.2 (G); no longer RK1.1 (P)
- net at RM1.2, RM2.2: now also C19.2, V3A.2 (G); no longer RK1.2 (G)
- net at RK2.1: now also V3A.3 (K); no longer RK1.3 (K)
- net at C3.1, V1A.3 (K), V1B.3 (K): now also RK1.1
- net at C7.2, V4A.2 (G): now also RGA.1; no longer RT2.1
- net at VR5.2 (W): now also C6.2; no longer VR4.2
- net at C9.1, RLA.2, V4A.1 (P): now also C20.1
- net at RGB.1, RTAIL.2: now also RT2.1, RGA.2; no longer RT2.2
- net at RM2.1, VR2.2 (W): now also C19.1
- removed net -50V: C13.1, C16.1, C17.2, RB1.2, RGL2.2
- new net: C18.1, D1.1 (A), RB3.1
- new net: T3.1 (PRI_A), V5.1 (P)
- new net: C9.2, RGL1.1, V5.2 (G1)
- new net: VR4.2 (W), VR4.3, VR5.1
- new net: D1.2 (K), RB1.2
- new net: C4.2, VR3.1
- new net -BIAS: C16.1, RB2.1, RB3.2, RGL1.2, RGL2.2
- new net SCR: RS1.2, RS2.2, RS3.2
Other:
- note added: "100 pF bright cap across VR2 omitted (AC only)"
- note added: "Power — 360-0-360 HT, GZ34, 20H choke (OT centre tap after it)"
- note added: "standby switch between the GZ34 cathode (C15 side) and the +450 V reservoir B+1 (omitted)"
- note removed: "100 pF bright cap across VR1 omitted (AC only)"
- note removed: "Power — 360-0-360 HT, GZ34, 20H choke · bias: HT-tap diode, 150k, .05u + 25u -> -50V"
- note removed: "standby switch between reservoir and B+1 (omitted)"
- moved on the sheet: C13, RT2, V6
