File: amps/ac15/schematic.kicad_sch (KiCad schematic)
At the start: 78 parts, among them SW1 DPST, SW2 5-pos, SW7 standby, T1 Haddon OF 031, T2 8/15 ohm

Commit message: Fix: schematic sheets — real title block, fitted paper, no lettering through circuitry
Every sheet in the corpus shipped with an EMPTY title block ("Title:" and
"Date:" blank, default "Sheet /" furniture) laid onto a fixed A4/A3 page
regardless of the drawing's size, with prose annotations placed by hand
wherever a coordinate looked free when the amp was first drawn. The result
read as an unfinished alpha under a `verified` badge: KiCanvas's default view
is `zoom_to_page()`, so a 150 x 110 mm circuit on an A3 sheet opened as a
postage stamp, and later edits had pushed live circuitry under the prose.

schematic_lib.py — the builder now records each element as a (kind, points,
extra) tuple instead of a finished string, so `write()` can measure and move
what it emits:

- emits a real `(title_block …)` read from the amp's own meta.yaml — Title =
  designation + style, Date = the verification (or added) date, Rev = the
  verification status, Company = Circuit Codex, plus the licence and source
  URL as comments. Fixes all 34 sheets from one place;
- emits `(paper "User" w h)` cut to the drawing, translated to a fixed margin,
  with the bottom 34 mm strip reserved for the worksheet's title block. Sheet
  utilisation of the drawable area went from as low as ~20% to 92-98%;
- `note()` queues prose into a wrapped band under the circuit, and `caption()`
  places a section heading over the block it names, nudging it clear if it
  would print through anything;
- per-symbol default label offsets (the old single default printed every pot's
  value through its own wiper arrow and every transformer's designator through
  its body), plus `place_labels()`, which moves any designator/value block that
  would print over ink;
- transformers and chokes are drawn, not boxed: iron core between two windings,
  centre taps where the part has them, and an optional `spec` lettering slot for
  a ratio or impedance;
- `gnd()` takes a direction, because a flag defaulting to "down" at the HEAD of
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
Connections:
- net GND: no longer T1.4 (HT_CT)
- net HT_A: no longer T1.3 (HT_A)
- net HT_B: no longer T1.5 (HT_B)
Other:
- note added: "The two-position TONE network, the five-section phase-shift ladder, the ECC82 modulator network and the ECC83 oscillator network (with Depth, Speed, the fast/slow switch and the footswitch jack) are listed part by part in bom.yaml. The published drawing resolves their VALUES but not their interconnection, so this sheet names the interfaces and asserts nothing further. The phase-shift vibrato bend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"
- note removed: "AC15 — Vox AC15-style, JMI circuit No. 3 (OA/031, 29-4-60) · Circuit Codex · CC-BY-SA 4.0 · redrawn from circuit facts"
- note removed: "The published drawing resolves their VALUES but not their interconnection, so"
- note removed: "The two-position TONE network, the five-section phase-shift ladder, the ECC82"
- note removed: "fast/slow switch and the footswitch jack) are listed part by part in bom.yaml."
- note removed: "modulator network and the ECC83 oscillator network (with Depth, Speed, the"
- note removed: "this sheet names the interfaces and asserts nothing further. The phase-shift"
- note removed: "vibrato bends pitch rather than gating level — see notes.md."
- company: (none) -> Circuit Codex
- title: (none) -> AC15 — Vox AC15-style
