File: amps/ac15/schematic.kicad_sch (KiCad schematic)
At the start: 78 parts, among them SW1 DPST, SW2 5-pos, SW7 standby, T1 Haddon OF 031, T2 8/15 ohm

Commit message: Fix: AC15 schematic never rendered — raw quotes broke KiCanvas's tokenizer
The annotation (text "… "Vibravox"") round-trips through kiutils, so the
CI gate passed while the live viewer threw at index 32980 and drew a
blank panel. Three layers: schematic_lib.text() now escapes quotes and
backslashes so no draw script can ship the fault; the AC15 annotation
uses typographic quotes; check_schematics gains a KiCanvas-strict
tokenization pass proven to catch the original fault.

Co-Authored-By: Claude Fable 5 <noreply@anthropic.com>
Other:
- note added: "Vibrato/Tremolo channel — ‘Vibravox’"
- note removed: "Vibrato/Tremolo channel —"
Changed lines of the file:
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@@
   (global_label "NORM VOL" (shape input) (at 156 42.075 0)
     (effects (font (size 1.27 1.27)) (justify left)))
-  (text "Vibrato/Tremolo channel — "Vibravox"" (at 16 89.5 0)
+  (text "Vibrato/Tremolo channel — ‘Vibravox’" (at 16 89.5 0)
     (effects (font (size 1.6 1.6)) (justify left)))
   (symbol (lib_id "cx:JACK") (at 20 100.54 0) (mirror y) (unit 1)

Commit message: Fix: one lettering convention per surface, engine-enforced; legend inside the viewBox
WS3 — layout pipeline + cross-surface value-consistency engine.

## One convention per surface (docs/lettering-conventions.md, new)

The same part stated its value in several notations at once. 5E3 C6 and 5D3 C6
rendered "5n" on the schematic, "0.005 µF · 600 V" in the parts list and
"0.005 µF" on the board. 5F6-A RD1 printed "4,700 Ω" beside neighbours printing
"15 kΩ". check_value_consistency proves the surfaces name the same QUANTITY; it
cannot see that they name it three ways. So each surface now has exactly one
convention and every one of them is gated:

* house units in bom.yaml/prose — engineering prefix with the mantissa 1…999,
  pF below 1000 pF and µF at and above it, no comma-grouped thousands. 19 values
  normalised (5E6-A, 5F6-A, 5F10, 6161, 6G2, 6G5, 6G6-B).
* schematic drafting shorthand — the unit letter is the SI prefix of the house
  unit, in the amp's declared idiom (meta.yaml conventions.notation: us|uk).
  British RKM/nanofarad practice on the Hiwatt and the 2204 is DECLARED, not
  normalised away; it is what those source drawings letter. Secondary ratings
  are space-separated fields with their own unit ("20u 600V"), never the era's
  dashed shorthand and never the house middot. 30 symbol values corrected across
  ten draw scripts.
* era sheet lettering — generated only, by era_pair(); documented cases and a
  corpus round-trip sweep in test_era_values.py, now 57 cases.

## Era-lettering fall-throughs closed

A value era_pair() refuses came back as the house string, and a house string can
be a whole sentence. Fixed at the source rather than per case:

* body_value() — a parenthetical GLOSS is never lettered on a component body.
  "selenium (silicon diode in modern builds)" was lettered in full on the 5E4-A
  and ran off the left edge of the page.
* twin cans letter as the era sheets did: 25 µF + 25 µF -> "25/25MFD".
* a repeat count is not a rating: "(×2)" com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
Parts:
- removed SW-BRIL: SPST, symbol cx:SWITCH
- added SWBRIL: SPST, symbol cx:SWITCH
Connections:
- net at CBR.1, CO1.2: now also SWBRIL.1
- net at CBR.2, VR1.1: now also SWBRIL.2
Changed lines of the file:
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@@
   (symbol (lib_id "cx:SWITCH") (at 131 38.265 0) (unit 1)
     (in_bom yes) (on_board yes)
-    (property "Reference" "SW-BRIL" (at 127.6 43.865 0) (effects (font (size 1.27 1.27)) (justify left)))
+    (property "Reference" "SWBRIL" (at 127.6 43.865 0) (effects (font (size 1.27 1.27)) (justify left)))
     (property "Value" "SPST" (at 127.6 46.265 0) (effects (font (size 1.27 1.27)) (justify left))))
   (wire (pts (xy 120 38.265) (xy 125.92 38.265))

Commit message: Update: regenerate every drawing the four merged units changed
The four parallel units all rewrote generators, so their committed artifacts
were each generated against only their own third of the merged pipeline. Every
schematic, both layout styles, the social cards and the manifest are rebuilt
here from the merged sources, so what ships is what the merged generators draw.

One integration fault the rebuild exposed, invisible to any single unit:

- 5E5-A: the note explaining that the Presence wiper and the 100k feedback
  resistor land on V3A's GRID (not its cathode, as on the 5F4) was added as a
  hand-placed `s.text()` at a coordinate chosen before the sheet gained a
  reserved notes band. Merged, it printed through the -32V bias label. Moved to
  `note()`, which wraps prose into that band — the exact failure mode the band
  was built to end.

Three conflicts resolved against docs/lettering-conventions.md rather than by
picking a side, since two units had corrected the same lines for different
reasons:

- 5E5-A tone/feedback caps take the corrected designators (C7, C8, C9, RNF —
  `C_tr1`/`C_NFB` were generator identifiers that had leaked onto a published
  board) with the house-derived lettering (`.01u 400V`, `500p`, `.1u 200V`).
  Dropping the working voltage or writing `.0005u` would have lost a rating the
  source prints and re-broken the pF/µF decade rule.
- 5D3 C6 and 6G6-B's three cathode resistors take the SI-prefix form the
  convention binds (`.005u`, `2.7k`, `1.5k`), keeping the ground-flag direction
  fix and the removal of the second `gnd()` that shorted each cathode it biased.
- 5F6-A's bias supply keeps both 8 µF cans drawn — the second was previously a
  parenthetical claiming one of two was shown — at the coordinates that clear
  the title-block strip.

All gates green, including check_value_consistency at zero disagreements.

🤖 Generated with [Claude Code](https://claude.com/claude-code)

Co-Authored-By: Claude Fable 5 <noreply@anthropic.com>
Connections:
- net GND: no longer T1.4 (HT_CT)
- net HT_A: no longer T1.3 (HT_A)
- net HT_B: no longer T1.5 (HT_B)
Other:
- note added: "The two-position TONE network, the five-section phase-shift ladder, the ECC82 modulator network and the ECC83 oscillator network (with Depth, Speed, the fast/slow switch and the footswitch jack) are listed part by part in bom.yaml. The published drawing resolves their VALUES but not their interconnection, so this sheet names the interfaces and asserts nothing further. The phase-shift vibrato bend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"
- note removed: "AC15 — Vox AC15-style, JMI circuit No. 3 (OA/031, 29-4-60) · Circuit Codex · CC-BY-SA 4.0 · redrawn from circuit facts"
- note removed: "The published drawing resolves their VALUES but not their interconnection, so"
- note removed: "The two-position TONE network, the five-section phase-shift ladder, the ECC82"
- note removed: "fast/slow switch and the footswitch jack) are listed part by part in bom.yaml."
- note removed: "modulator network and the ECC83 oscillator network (with Depth, Speed, the"
- note removed: "this sheet names the interfaces and asserts nothing further. The phase-shift"
- note removed: "vibrato bends pitch rather than gating level — see notes.md."
- company: (none) -> Circuit Codex
- title: (none) -> AC15 — Vox AC15-style

Commit message: Fix: rotated global labels lettered their net names outside the flag
Every global label this pipeline emitted carried (justify left) regardless of
rotation. KiCanvas — like KiCad — draws label text horizontally at 0/180 and
vertically at 90/270 and reads WHICH SIDE of the anchor it letters on from the
justification, so at 180 and 270 the name printed outside an empty flag
outline, struck through by the very wire it names: 219 labels at 180 deg
(including the input-jack flags at top-left of nearly every sheet, the first
glyphs a visitor reads) and 792 GND/rail flags at 270 whose names squeezed at
the flag mouth instead of lettering down the body. The library already
compensated rotation for property text (`pa`); this mirrors that logic for
global labels: justify right at 180/270, left at 0/90.

check_schematics gains the geometry clause whose absence let all 1011
instances through a "no lettering through circuitry" pass: it modelled the
flag box but never the label TEXT, so a name rendered on the wrong side was
invisible to it. The gate now proves justification compensates rotation on
every global label.

Two more things this exposed, fixed in the same engine pass:

- Placement now measures with the renderer's own Newstroke advance table
  (extracted from the vendored kicanvas.js) instead of a flat 0.68-em prose
  average that under-read part lettering by a quarter — the mechanism behind
  every "metered clean, printed through its neighbour" incident. The GATE
  deliberately keeps the coarse ruler: re-ruling it with renderer truth was
  tried and red-flagged 28 of 34 sheets over abutments three visual passes
  had already judged sub-visual (the two-rulers note in schematic_lib.py).
- place_captions' escape ladder runs further, because a banner caption
  measured truly is half again wider than the old estimate believed.

All 34 schematics regenerated; full gate suite green.

🤖 Generated with [Claude Code](https://claude.com/claude-code)

Co-Authored-By: Claude Fable 5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
Other:
- note added: "gating level — see notes.md."

Commit message: Fix: deterministic schematic ids and wires split at every join
- _u() is uuid5 over (amp id, emission order), so a regeneration of an
  unchanged script is byte-identical and a drift gate becomes possible
- write() splits wire segments at symbol pins, wire ends and junction dots,
  so the file connects exactly what the drawing shows under KiCad's
  endpoint-only semantics (270 pins were on a wire's interior; net
  partitions unchanged on all 38 sheets)
- all sheets regenerated; aa864-bassman title block was stale (draft) and
  now matches meta.yaml (verified)

Co-Authored-By: Claude Fable 5.1 <noreply@anthropic.com>
Claude-Session: https://claude.ai/code/session_01KBMfdh37HmCL2iWcBiL5J1
Changed lines of the file:
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@@
   (global_label "GND" (shape input) (at 34.4724 61.9 270)
     (effects (font (size 1.27 1.27)) (justify right)))
-  (wire (pts (xy 64.4724 25.82) (xy 64.4724 53.82))
+  (wire (pts (xy 64.4724 25.82) (xy 64.4724 39.82))
+    (stroke (width 0) (type default)))
+  (wire (pts (xy 64.4724 39.82) (xy 64.4724 53.82))
     (stroke (width 0) (type default)))
   (junction (at 64.4724 39.82) (diameter 0) (color 0 0 0 0))
@@
   (global_label "GND" (shape input) (at 34.4724 123.9 270)
     (effects (font (size 1.27 1.27)) (justify right)))
-  (wire (pts (xy 64.4724 87.82) (xy 64.4724 115.82))
+  (wire (pts (xy 64.4724 87.82) (xy 64.4724 101.82))
+    (stroke (width 0) (type default)))
+  (wire (pts (xy 64.4724 101.82) (xy 64.4724 115.82))
     (stroke (width 0) (type default)))
   (junction (at 64.4724 101.82) (diameter 0) (color 0 0 0 0))
@@
     (property "Reference" "V5B" (at 150.472 95.42 0) (effects (font (size 1.27 1.27)) (justify left)))
     (property "Value" "ECC83" (at 150.472 97.82 0) (effects (font (size 1.27 1.27)) (justify left))))
-  (wire (pts (xy 124.282 101.82) (xy 136.852 101.82))
+  (wire (pts (xy 124.282 101.82) (xy 130.472 101.82))
+    (stroke (width 0) (type default)))
+  (wire (pts (xy 130.472 101.82) (xy 136.852 101.82))
     (stroke (width 0) (type default)))
   (junction (at 130.472 101.82) (diameter 0) (color 0 0 0 0))
@@
     (property "Reference" "RGA" (at 198.072 55.43 0) (effects (font (size 1.27 1.27)) (justify left)))
     (property "Value" "1M" (at 198.072 57.83 0) (effects (font (size 1.27 1.27)) (justify left))))
-  (wire (pts (xy 207.472 62.44) (xy 207.472 76.44))
+  (wire (pts (xy 207.472 62.44) (xy 207.472 65.82))
+    (stroke (width 0) (type default)))
+  (wire (pts (xy 207.472 65.82) (xy 207.472 76.44))
     (stroke (width 0) (type default)))
   (symbol (lib_id "cx:R") (at 207.472 80.25 0) (unit 1)
@@
   (wire (pts (xy 219.472 55.44) (xy 219.472 58.2))
     (stroke (width 0) (type default)))
-  (wire (pts (xy 219.472 58.2) (xy 232.472 58.2))
+  (wire (pts (xy 219.472 58.2) (xy 226.472 58.2))
+    (stroke (width 0) (type default)))
+  (wire (pts (xy 226.472 58.2) (xy 232.472 58.2))
     (stroke (width 0) (type default)))
   (wire (pts (xy 219.472 101.44) (xy 219.472 103.82))
@@
     (property "Reference" "VR3" (at 254.674 59.99 0) (effects (font (size 1.27 1.27)) (justify left)))
     (property "Value" "250k top cut" (at 254.674 62.39 0) (effects (font (size 1.27 1.27)) (justify left))))
-  (wire (pts (xy 250.472 65.44) (xy 250.472 82.72))
+  (wire (pts (xy 250.472 65.44) (xy 250.472 68.82))
+    (stroke (width 0) (type default)))
+  (wire (pts (xy 250.472 68.82) (xy 250.472 82.72))
     (stroke (width 0) (type default)))
   (junction (at 250.472 82.72) (diameter 0) (color 0 0 0 0))
@@
   (wire (pts (xy 304.472 109.82) (xy 316.472 109.82))
     (stroke (width 0) (type default)))
-  (wire (pts (xy 316.472 49.82) (xy 316.472 115.82))
+  (wire (pts (xy 316.472 49.82) (xy 316.472 109.82))
+    (stroke (width 0) (type default)))
+  (wire (pts (xy 316.472 109.82) (xy 316.472 115.82))
     (stroke (width 0) (type default)))
   (junction (at 316.472 109.82) (diameter 0) (color 0 0 0 0))
@@
   (wire (pts (xy 365.362 53.28) (xy 404.472 53.28))
     (stroke (width 0) (type default)))
-  (wire (pts (xy 404.472 53.28) (xy 404.472 91.82))
+  (wire (pts (xy 404.472 53.28) (xy 404.472 75.82))
+    (stroke (width 0) (type default)))
+  (wire (pts (xy 404.472 75.82) (xy 404.472 91.82))
     (stroke (width 0) (type default)))
   (symbol (lib_id "cx:JACK") (at 390.472 78.36 0) (mirror y) (unit 1)
@@
   (wire (pts (xy 150.472 202.44) (xy 150.472 207.82))
     (stroke (width 0) (type default)))
-  (wire (pts (xy 132.472 207.82) (xy 176.852 207.82))
+  (wire (pts (xy 132.472 207.82) (xy 150.472 207.82))
+    (stroke (width 0) (type default)))
+  (wire (pts (xy 150.472 207.82) (xy 164.472 207.82))
+    (stroke (width 0) (type default)))
+  (wire (pts (xy 164.472 207.82) (xy 176.852 207.82))
     (stroke (width 0) (type default)))
   (junction (at 150.472 207.82) (diameter 0) (color 0 0 0 0))
@@
   (wire (pts (xy 192.092 207.82) (xy 203.392 207.82))
     (stroke (width 0) (type default)))
-  (wire (pts (xy 213.552 207.82) (xy 244.472 207.82))
+  (wire (pts (xy 213.552 207.82) (xy 226.472 207.82))
+    (stroke (width 0) (type default)))
+  (wire (pts (xy 226.472 207.82) (xy 244.472 207.82))
     (stroke (width 0) (type default)))
   (junction (at 226.472 207.82) (diameter 0) (color 0 0 0 0))
@@
   (wire (pts (xy 244.472 207.82) (xy 250.472 207.82))
     (stroke (width 0) (type default)))
-  (wire (pts (xy 250.472 207.82) (xy 250.472 239.82))
+  (wire (pts (xy 250.472 207.82) (xy 250.472 223.82))
+    (stroke (width 0) (type default)))
+  (wire (pts (xy 250.472 223.82) (xy 250.472 239.82))
     (stroke (width 0) (type default)))
   (junction (at 250.472 207.82) (diameter 0) (color 0 0 0 0))
@@
   (wire (pts (xy 254.472 207.82) (xy 256.662 207.82))
     (stroke (width 0) (type default)))
-  (wire (pts (xy 264.282 207.82) (xy 280.472 207.82))
+  (wire (pts (xy 264.282 207.82) (xy 272.472 207.82))
+    (stroke (width 0) (type default)))
+  (wire (pts (xy 272.472 207.82) (xy 280.472 207.82))
     (stroke (width 0) (type default)))
   (junction (at 272.472 207.82) (diameter 0) (color 0 0 0 0))
@@
   (wire (pts (xy 254.472 223.82) (xy 256.662 223.82))
     (stroke (width 0) (type default)))
-  (wire (pts (xy 264.282 223.82) (xy 280.472 223.82))
+  (wire (pts (xy 264.282 223.82) (xy 272.472 223.82))
+    (stroke (width 0) (type default)))
+  (wire (pts (xy 272.472 223.82) (xy 280.472 223.82))
     (stroke (width 0) (type default)))
   (junction (at 272.472 223.82) (diameter 0) (color 0 0 0 0))
@@
   (wire (pts (xy 254.472 239.82) (xy 256.662 239.82))
     (stroke (width 0) (type default)))
-  (wire (pts (xy 264.282 239.82) (xy 280.472 239.82))
+  (wire (pts (xy 264.282 239.82) (xy 272.472 239.82))
+    (stroke (width 0) (type default)))
+  (wire (pts (xy 272.472 239.82) (xy 280.472 239.82))
     (stroke (width 0) (type default)))
   (junction (at 272.472 239.82) (diameter 0) (color 0 0 0 0))

Commit message: Fix: schematic wiring on ac15 and b15n
- ac15: the B+1 label named only the EL84 plates/screens and the OT centre
  tap; the standby switch, reservoir and dropper column were a separate
  net the drawing never joined (orphaned rail label)
- b15n: the R38 branch dropped through C16A's grounded pin, shorting the
  screen rail BP2 to chassis (six dependent findings); the paraphase
  divider halves R28/R29 were drawn against each other's anodes and are
  swapped to match netlist and parts list
- both sheets pass connectivity and verify_schematic_nets

Co-Authored-By: Claude Fable 5.1 <noreply@anthropic.com>
Claude-Session: https://claude.ai/code/session_01KBMfdh37HmCL2iWcBiL5J1
Connections:
- net B+1: now also CR2.1, RD1.1, RD2.1, RD3.1, SW7.2
Changed lines of the file:
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@@
   (text "+315 V" (at 232.472 201.82 0)
     (effects (font (size 1.15 1.15)) (justify left)))
+  (wire (pts (xy 244.472 207.82) (xy 244.472 199.82))
+    (stroke (width 0) (type default)))
+  (global_label "B+1" (shape input) (at 244.472 199.82 90)
+    (effects (font (size 1.27 1.27)) (justify left)))
   (junction (at 244.472 207.82) (diameter 0) (color 0 0 0 0))
   (wire (pts (xy 244.472 207.82) (xy 250.472 207.82))

Commit message: Add: real tube pin numbers and readable valve glyphs on every schematic
Phase B of the drawing program. A factory service sheet numbers every tube
pin, because the number is what a technician puts a probe on. This corpus
printed none, and the numbers hidden in its symbols were positional
placeholders (P=1, G=2, K=3) that would have published a 6V6GT's plate as
pin 1 when it is pin 3.

1055 electrodes now carry the real number, 1027 lettered (27 are shared
filaments deduped, 1 dropped for want of clear space on the 6G2). Resolved per
instance from reference/tubes/<slug>.yaml through the same alias resolution the
layout renderer uses, so a 12AX7 section and a 6SL7 section each get their own
basing. A valve whose basing the corpus does not carry prints nothing rather
than a wrong number.

Section letters and basing units are now separate things, which cost a detour
worth recording. The RCA 12AX7-A sheet reads "Pin 1 - Plate of Unit No.2 ...
Pin 6 - Plate of Unit No.1", so unit numbering is not pin order; the 5Y3 and
GZ34 number their units in opposite pin order, so nothing positional can
express it. But the section LETTER is a designator, not a basing fact: this
corpus, like every technician, calls the first stage in signal order V1A, and
five amps' prose already did. On four amps the factory sheets put that first
stage on the other half -- the AA764's own schematic prints +200 V on pin 1 --
so those drawings now state their unit explicitly, each citing its source, and
no letter, netlist, parts list or layout comment changed. 183 layout comments
agree with the printed numbers, 0 disagree. A guard fires if two halves of one
bottle resolve to the same unit, which is exactly how this was found.

Glyphs: the cathode gains a bracket and filament hairpin so it can no longer be
confused with the plate bar, the pentode's screen sits on its own row, and a
rectifier draws as one envelope over its sections instead of two apparent
bottles. Line weights are scaled per sheet to a co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
Other:
- note added: "1"
- note added: "2"
- note added: "3"
- note added: "6"
- note added: "7"
- note added: "8"
- note added: "9"
