File: amps/ac15/schematic.kicad_sch (KiCad schematic)
At the start: 78 parts, among them SW1 DPST, SW2 5-pos, SW7 standby, T1 Haddon OF 031, T2 8/15 ohm

Commit message: Fix: schematic sheet notes no longer name repository files
Thirty-seven committed sheets rendered footnotes and section notes such as
"Heaters and PT primary omitted — see netlist.cir and meta.yaml" or
"excluded from netlist.cir (notes.md)" to visitors through KiCanvas. The
prose sweeps never counted sheets. Rewritten in the site's own words — the
netlist, the sources list, the circuit story, the parts list, the board
drawing — in 59 strings across 33 draw scripts, keeping every technical
claim as it was; the three tone sheets (6G4, 6G5, 6G6-B) are under repair
elsewhere and keep theirs for now. The sweep touched only strings passed to
the sheet's note, text, caption and footnote calls, never a path or a value.

Gates: check_schematics 40/0, connectivity 0 isolated pins;
verify_schematic_nets 40 clean; only the regenerated sheets and their served
copies changed.

Co-Authored-By: Claude Fable 5.1 <noreply@anthropic.com>
Claude-Session: https://claude.ai/code/session_01KBMfdh37HmCL2iWcBiL5J1
Other:
- note added: "Heaters, the 6.3 V winding and the pilot-lamp wiring are an annotation layer — see the netlist, the parts list and the board drawing."
- note added: "The two-position TONE network, the five-section phase-shift ladder, the ECC82 modulator network and the ECC83 oscillator network (with Depth, Speed, the fast/slow switch and the footswitch jack) are listed part by part in the parts list. The published drawing resolves their VALUES but not their interconnection, so this sheet names the interfaces and asserts nothing further. The phase-shift vibrat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"
- note added: "gating level — see the circuit story."
- note removed: "Heaters, the 6.3 V winding and the pilot-lamp wiring are an annotation layer — see netlist.cir, bom.yaml and layout.yaml."
- note removed: "The two-position TONE network, the five-section phase-shift ladder, the ECC82 modulator network and the ECC83 oscillator network (with Depth, Speed, the fast/slow switch and the footswitch jack) are listed part by part in bom.yaml. The published drawing resolves their VALUES but not their interconnection, so this sheet names the interfaces and asserts nothing further. The phase-shift vibrato bend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"
- note removed: "gating level — see notes.md."
Changed lines of the file:
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@@
   (text "No tone stack · no bias supply · no negative feedback. Both channels mix INSIDE the phase inverter, at opposite grids. Rails: B+1 +315 V · B+N Normal · B+P inverter · B+V vibrato" (at 12.7 258.598 0)
     (effects (font (size 1.2 1.2)) (justify left)))
-  (text "Heaters, the 6.3 V winding and the pilot-lamp wiring are an annotation layer — see netlist.cir, bom.yaml and layout.yaml." (at 12.7 262.998 0)
+  (text "Heaters, the 6.3 V winding and the pilot-lamp wiring are an annotation layer — see the netlist, the parts list and the board drawing." (at 12.7 262.998 0)
     (effects (font (size 1.2 1.2)) (justify left)))
-  (text "The two-position TONE network, the five-section phase-shift ladder, the ECC82 modulator network and the ECC83 oscillator network (with Depth, Speed, the fast/slow switch and the footswitch jack) are listed part by part in bom.yaml. The published drawing resolves their VALUES but not their interconnection, so this sheet names the interfaces and asserts nothing further. The phase-shift vibrato bends pitch rather than" (at 12.7 267.398 0)
+  (text "The two-position TONE network, the five-section phase-shift ladder, the ECC82 modulator network and the ECC83 oscillator network (with Depth, Speed, the fast/slow switch and the footswitch jack) are listed part by part in the parts list. The published drawing resolves their VALUES but not their interconnection, so this sheet names the interfaces and asserts nothing further. The phase-shift vibrato bends pitch rather than" (at 12.7 267.398 0)
     (effects (font (size 1.2 1.2)) (justify left)))
-  (text "gating level — see notes.md." (at 12.7 271.798 0)
+  (text "gating level — see the circuit story." (at 12.7 271.798 0)
     (effects (font (size 1.2 1.2)) (justify left)))
   (sheet_instances (path "/" (page "1")))
