File: amps/5f6a/schematic.kicad_sch (KiCad schematic)
At the start: 59 parts, among them T3 2R sec

Commit message: BOMs for 5E3/5F6-A, cross-artifact CI gates, visitor-voice notes, REVIEW.md
- bom.yaml for both new amps (60+ designators), refs matching their
  schematics exactly; 5F6-A PI tubes renamed V3A/V3B for consistent
  bottle numbering
- validate.py: verified amps now require the full artifact set
  (netlist, voltages, notes, schematic, BOM) and every BOM designator
  must reconcile with the schematic in both directions
- All three circuit stories rewritten in visitor voice (internal
  working-notes language removed — e.g. the 5E3 "secondary sources
  garble" heading)
- docs/REVIEW.md: the two-layer QA contract (deterministic CI gates +
  post-deploy editorial/accuracy judge pass on rendered pages)

Co-Authored-By: Claude Opus 4.8 (1M context) <noreply@anthropic.com>
Parts:
- removed PIA, PIB: 12AX7, symbol cx:TRIODE
- added V3A, V3B: 12AX7, symbol cx:TRIODE
Connections:
- net at C9.1, RLB.2: now also V3B.1 (P)
- net at C7.2, RGB.2: now also V3B.2 (G)
- net at RTAIL.1: now also V3A.3 (K), V3B.3 (K)
- net at C8.1, RLA.2: now also V3A.1 (P)
- net at C6.2, RGA.1: now also V3A.2 (G)
Other:
- note added: "47 pF balance cap V3A grid-plate omitted (AC only) · NFB 27k + presence 5k join the tail foot at ~0 V DC"
- note removed: "47 pF balance cap PIA grid-plate omitted (AC only) · NFB 27k + presence 5k join the tail foot at ~0 V DC"
Changed lines of the file:
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@@
   (symbol (lib_id "cx:TRIODE") (at 176.53 92 0) (unit 1)
     (in_bom yes) (on_board yes)
-    (property "Reference" "PIA" (at 182.53 85.6 0) (effects (font (size 1.27 1.27)) (justify left)))
+    (property "Reference" "V3A" (at 182.53 85.6 0) (effects (font (size 1.27 1.27)) (justify left)))
     (property "Value" "12AX7" (at 182.53 88 0) (effects (font (size 1.27 1.27)) (justify left))))
   (wire (pts (xy 168.91 92) (xy 168.91 92))
@@
   (symbol (lib_id "cx:TRIODE") (at 176.53 126 0) (unit 1)
     (in_bom yes) (on_board yes)
-    (property "Reference" "PIB" (at 182.53 119.6 0) (effects (font (size 1.27 1.27)) (justify left)))
+    (property "Reference" "V3B" (at 182.53 119.6 0) (effects (font (size 1.27 1.27)) (justify left)))
     (property "Value" "12AX7" (at 182.53 122 0) (effects (font (size 1.27 1.27)) (justify left))))
   (wire (pts (xy 176.53 84.38) (xy 176.53 80.9))
@@
   (wire (pts (xy 158.75 116.62) (xy 168.91 116.62))
     (stroke (width 0) (type default)))
-  (text "47 pF balance cap PIA grid-plate omitted (AC only) · NFB 27k + presence 5k join the tail foot at ~0 V DC" (at 150 145 0)
+  (text "47 pF balance cap V3A grid-plate omitted (AC only) · NFB 27k + presence 5k join the tail foot at ~0 V DC" (at 150 145 0)
     (effects (font (size 1.1 1.1)) (justify left)))
   (wire (pts (xy 176.53 80.9) (xy 194.31 80.9))

Commit message: Fix: the drawn tone stacks now are the tone stack the lab plots, and a gate says so
The tone-stack lab solves one network — the FMV stack documented in
site/src/lib/tonestack.js — and fills its values from each amp's BOM by
reference designator. Nothing checked that the schematic drew those
designators into that network, and nine of the nine drawings did not.

What the drawings said, rebuilt from the committed .kicad_sch files rather
than from the generators:

- 5F6-A, JTM45, 1987, 1959 and 5F4 ran the treble capacitor off the slope
  resistor's FOOT instead of the stack input, and landed the treble pot's
  lower lug on the bass-capacitor node instead of the slope foot.
- Every three-knob drawing left the bass pot's wiper unwired, so the plotted
  output (treble wiper AND bass wiper) existed on no drawing.
- JTM45, 1987 and 1959 put the mid capacitor in series with the mid pot down
  to ground rather than from the slope foot to the mid leg's top.
- 5F6 tied its bass pot as a rheostat and fed the mid capacitor to the middle
  pot's wiper.
- The blackface circuits left the treble pot's lower lug on the bass-cap node
  and tied the bass wiper to its own lug; AB763 drew its 0.047 µF inline on
  top of the bass pot's lug.

The 5F6-A's own layout.yaml — redrawn from the published Fender 5F6-A layout
sheet — already wires the canonical network (treble low to the slope node,
both wipers to the phase-inverter coupler), and 5F4's does too, so the
drawings were corrected to that rather than the lab to the drawings.

Consequences beyond the wires:

- 5F6-A's parts list prints one 0.02 µF line covering the bass and middle
  positions; the drawing showed one capacitor where the circuit has two.
  Added C5b with the same value and the same printed line cited. The plotted
  curve does not move — both positions already used that value.
- The blackface stacks keep the capacitor that feeds the mid leg. With the
  lug corrected, CBN/CB1 (0.1 µF) feeds the bass pot and CBN2/CB2 (0.047 µ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
Parts:
- added C5b: .02u, symbol cx:C
Connections:
- net at C5.1, RSL.2: now also VR3.3, C5b.1; no longer C4.1
- net at C6.1, VR3.2 (W): now also VR4.2 (W)
- net at C5.2, VR4.1: no longer VR3.3
- net at VR4.3, VR5.1, VR5.2 (W): now also C5b.2
- net at RKCF.1, RSL.1, V2B.3 (K): now also C4.1
Changed lines of the file:
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@@
   (wire (pts (xy 116.84 119.5) (xy 124.46 119.5))
+    (stroke (width 0) (type default)))
+  (junction (at 124.46 119.5) (diameter 0) (color 0 0 0 0))
+  (wire (pts (xy 124.46 119.5) (xy 124.46 96))
+    (stroke (width 0) (type default)))
+  (wire (pts (xy 124.46 96) (xy 135.89 96))
     (stroke (width 0) (type default)))
   (symbol (lib_id "cx:R") (at 128.27 119.5 90) (unit 1)
@@
   (wire (pts (xy 132.08 119.5) (xy 135.89 119.5))
     (stroke (width 0) (type default)))
-  (wire (pts (xy 135.89 119.5) (xy 135.89 96))
+  (wire (pts (xy 135.89 119.5) (xy 135.89 103.62))
+    (stroke (width 0) (type default)))
+  (wire (pts (xy 135.89 103.62) (xy 147.32 103.62))
     (stroke (width 0) (type default)))
   (junction (at 135.89 108) (diameter 0) (color 0 0 0 0))
+  (junction (at 135.89 118) (diameter 0) (color 0 0 0 0))
   (symbol (lib_id "cx:C") (at 139.7 96 90) (unit 1)
     (in_bom yes) (on_board yes)
@@
   (wire (pts (xy 143.51 108) (xy 147.32 108))
     (stroke (width 0) (type default)))
-  (wire (pts (xy 147.32 103.62) (xy 147.32 108))
-    (stroke (width 0) (type default)))
   (symbol (lib_id "cx:POT") (at 147.32 111.81 0) (unit 1)
     (in_bom yes) (on_board yes)
     (property "Reference" "VR4" (at 149.52 108.61 0) (effects (font (size 1.27 1.27)) (justify left)))
     (property "Value" "1M bass" (at 149.52 111.01 0) (effects (font (size 1.27 1.27)) (justify left))))
+  (symbol (lib_id "cx:C") (at 139.7 118 90) (unit 1)
+    (in_bom yes) (on_board yes)
+    (property "Reference" "C5b" (at 136.5 111.8 270) (effects (font (size 1.27 1.27)) (justify left)))
+    (property "Value" ".02u" (at 136.5 114.2 270) (effects (font (size 1.27 1.27)) (justify left))))
+  (wire (pts (xy 143.51 118) (xy 147.32 118))
+    (stroke (width 0) (type default)))
   (wire (pts (xy 147.32 115.62) (xy 147.32 118))
     (stroke (width 0) (type default)))
@@
   (wire (pts (xy 152.4 99.81) (xy 156.21 99.81))
     (stroke (width 0) (type default)))
+  (wire (pts (xy 152.4 111.81) (xy 156.21 111.81))
+    (stroke (width 0) (type default)))
+  (wire (pts (xy 156.21 111.81) (xy 156.21 99.81))
+    (stroke (width 0) (type default)))
+  (junction (at 156.21 99.81) (diameter 0) (color 0 0 0 0))
   (wire (pts (xy 156.21 99.81) (xy 156.21 92))
     (stroke (width 0) (type default)))
