File: amps/6g5/schematic.kicad_sch (KiCad schematic)
At the start: 98 parts, among them SW1 AC

Commit message: Add: real tube pin numbers and readable valve glyphs on every schematic
Phase B of the drawing program. A factory service sheet numbers every tube
pin, because the number is what a technician puts a probe on. This corpus
printed none, and the numbers hidden in its symbols were positional
placeholders (P=1, G=2, K=3) that would have published a 6V6GT's plate as
pin 1 when it is pin 3.

1055 electrodes now carry the real number, 1027 lettered (27 are shared
filaments deduped, 1 dropped for want of clear space on the 6G2). Resolved per
instance from reference/tubes/<slug>.yaml through the same alias resolution the
layout renderer uses, so a 12AX7 section and a 6SL7 section each get their own
basing. A valve whose basing the corpus does not carry prints nothing rather
than a wrong number.

Section letters and basing units are now separate things, which cost a detour
worth recording. The RCA 12AX7-A sheet reads "Pin 1 - Plate of Unit No.2 ...
Pin 6 - Plate of Unit No.1", so unit numbering is not pin order; the 5Y3 and
GZ34 number their units in opposite pin order, so nothing positional can
express it. But the section LETTER is a designator, not a basing fact: this
corpus, like every technician, calls the first stage in signal order V1A, and
five amps' prose already did. On four amps the factory sheets put that first
stage on the other half -- the AA764's own schematic prints +200 V on pin 1 --
so those drawings now state their unit explicitly, each citing its source, and
no letter, netlist, parts list or layout comment changed. 183 layout comments
agree with the printed numbers, 0 disagree. A guard fires if two halves of one
bottle resolve to the same unit, which is exactly how this was found.

Glyphs: the cathode gains a bracket and filament hairpin so it can no longer be
confused with the plate bar, the pentode's screen sits on its own row, and a
rectifier draws as one envelope over its sections instead of two apparent
bottles. Line weights are scaled per sheet to a co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
Changed lines of the file:
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@@
   (global_label "-55V" (shape input) (at 240.745 199.82 0)
     (effects (font (size 1.27 1.27)) (justify left)))
-  (text "1" (at 63.5952 35.47 0)
+  (text "6" (at 63.5952 35.47 0)
     (effects (font (size 1.1 1.1)) (justify left)))
-  (text "2" (at 55.798 40.42 0)
+  (text "7" (at 55.798 40.42 0)
     (effects (font (size 1.1 1.1)) (justify left)))
-  (text "3" (at 63.5952 48.17 0)
+  (text "8" (at 63.5952 48.17 0)
     (effects (font (size 1.1 1.1)) (justify left)))
-  (text "6" (at 149.595 35.47 0)
+  (text "1" (at 149.595 35.47 0)
     (effects (font (size 1.1 1.1)) (justify left)))
-  (text "7" (at 141.798 40.42 0)
+  (text "2" (at 141.798 40.42 0)
     (effects (font (size 1.1 1.1)) (justify left)))
-  (text "8" (at 149.595 48.17 0)
+  (text "3" (at 149.595 48.17 0)
     (effects (font (size 1.1 1.1)) (justify left)))
-  (text "1" (at 63.5952 133.47 0)
+  (text "6" (at 63.5952 133.47 0)
     (effects (font (size 1.1 1.1)) (justify left)))
-  (text "2" (at 55.798 138.42 0)
+  (text "7" (at 55.798 138.42 0)
     (effects (font (size 1.1 1.1)) (justify left)))
-  (text "3" (at 63.5952 146.17 0)
+  (text "8" (at 63.5952 146.17 0)
     (effects (font (size 1.1 1.1)) (justify left)))
-  (text "6" (at 149.595 133.47 0)
+  (text "1" (at 149.595 133.47 0)
     (effects (font (size 1.1 1.1)) (justify left)))
-  (text "7" (at 141.798 138.42 0)
+  (text "2" (at 141.798 138.42 0)
     (effects (font (size 1.1 1.1)) (justify left)))
-  (text "8" (at 149.595 146.17 0)
+  (text "3" (at 149.595 146.17 0)
     (effects (font (size 1.1 1.1)) (justify left)))
-  (text "1" (at 269.595 73.47 0)
+  (text "6" (at 269.595 73.47 0)
     (effects (font (size 1.1 1.1)) (justify left)))
-  (text "2" (at 261.798 78.42 0)
+  (text "7" (at 261.798 78.42 0)
     (effects (font (size 1.1 1.1)) (justify left)))
-  (text "3" (at 269.595 86.17 0)
+  (text "8" (at 269.595 86.17 0)
     (effects (font (size 1.1 1.1)) (justify left)))
-  (text "6" (at 269.595 133.47 0)
+  (text "1" (at 269.595 133.47 0)
     (effects (font (size 1.1 1.1)) (justify left)))
-  (text "7" (at 261.798 138.42 0)
+  (text "2" (at 261.798 138.42 0)
     (effects (font (size 1.1 1.1)) (justify left)))
-  (text "8" (at 269.595 146.17 0)
+  (text "3" (at 269.595 146.17 0)
     (effects (font (size 1.1 1.1)) (justify left)))
   (text "3" (at 331.595 52.835 0)
