File: amps/6g5/schematic.kicad_sch (KiCad schematic)
At the start: 109 parts, among them SW1 AC

Commit message: Fix: the 6G5 is a harmonic vibrato on ten 7025 sections, not a photocell tremolo; channels paired by stage
The A-FJ drawing, read at its full 2153x1437 / 2224x1331 px, has no lamp or
photocell. Its five 7025s are shared by STAGE: V1 both first stages (cathodes
joined, one 820/25), V2 both second stages (one 820/25), V3 the vibrato
oscillator (pins 1-3) and its phase splitter (6-8), V4 the vibrato pair, V5
the inverter. The corpus had one bottle per channel, an invented optocoupler,
and one section of the vibrato pair modelled as a "driver".

- netlist: vibrato pair V4 and the band-splitting filters modelled; splitter
  V3B modelled (static stage); oscillator V3A excluded (no static point).
  Channel 1's second stage is 100k + 6.8k decoupler with the output at their
  junction; channel 2's is 220k — the +160/+120 V asymmetry. Every rail now
  derived through droppers the drawing letters (4.7k to +430, 56k to +260,
  56k to +350, 56k to +275; the layout page prints each); BP3/BDRV/BD driven
  anchors gone. Screens hang at the +458 V post-choke node: the old
  "4700 screen dropper" is the PI dropper. PI foot modelled (1500 + 22k NFB).
- voltages: 23 nodes compared, 1 null (JPI, printed nowhere); was 6 of 16.
- sheet: redrawn whole; unit= on every dual-triode section from the layout
  page's socket prints; vibrato block off the mains corner; JVIB wired (its
  open-pin waiver retired). Channel 2 has no bright cap on either page (CBR2
  deleted); the PI's .001 is its input coupler, 47MM sits across the plates,
  and a .1-200 grounds the cold grid to the tail foot.
- meta: sections block (V3A excluded); sources and verification prose.

The board still draws the old topology; it follows in the next commit.

Co-Authored-By: Claude Opus 5 (1M context) <noreply@anthropic.com>
Parts:
- removed CBR2: 47p, symbol cx:C
- removed CC1T, CMIX1, CMIX2: .05u, symbol cx:C
- removed CK1A, CK2A: 25u+25u, symbol cx:C
- removed CK1B, CK2B: 25u (info.), symbol cx:C
- removed CK5: 25u, symbol cx:C
- removed CT2: 250p, symbol cx:C
- removed CTO3: .02u, symbol cx:C
- removed D3, D5: 1N4007, symbol cx:DIODE_SS
- removed JVIB: vibrato pedal, symbol cx:JACK
- removed OPTO: optocoupler, symbol cx:OPTO
- removed RDSCR: 4.7k 1W, symbol cx:R
- removed RF1, RF2: 10k, symbol cx:R
- removed RFB1: 470k, symbol cx:R
- removed RFB2, RFB3: 220k, symbol cx:R
- removed RK1B, RK2B: 1.5k (info.), symbol cx:R
- removed RK2A, RK5: 820, symbol cx:R
- removed RL1A, RL2A, RL5: 100k, symbol cx:R
- removed RTOK: 1.5k, symbol cx:R
- removed V3, V6B: 7025, symbol cx:TRIODE
- added CC1D, CC2D, CSV: .05u, symbol cx:C
- added CF4, CF8: 20u 600V, symbol cx:C
- added CFS, CPIN: .001u, symbol cx:C
- added CGB, CTX: .1u 200V, symbol cx:C
- added CGS, CTW: .05u 200V, symbol cx:C
- added CK1, CK2, CKS, CTOK: 25u 25V, symbol cx:C
- added CPS: .25u, symbol cx:C
- added CTO1, CV1: .01u, symbol cx:C
- added CTOF: .005u, symbol cx:C
- added CTOP: .03u, symbol cx:C
- added CV2: 250p, symbol cx:C
- added DBIAS: Si, symbol cx:DIODE_SS
- added R2H: 68k, symbol cx:R
- added RBIAS2: 10k, symbol cx:R
- added RD3, RD4: 56k 1W, symbol cx:R
- added RG1A, RGS, RGV2, RM2, RTOG1, RWV: 1M, symbol cx:R
- added RHP1, RHP2: 220k, symbol cx:R
- added RK1, RK2: 820, symbol cx:R
- added RKS: 1.5k, symbol cx:R
- added RKV: 4.7k, symbol cx:R
- added RLB: 100k 5%, symbol cx:R
- added RLD1: 6.8k, symbol cx:R
- added RLP, RMV2: 470k, symbol cx:R
- added RLS, RLV1, RLV2, RS1T, RS2T, RSPD: 100k, symbol cx:R
- added RTOF: 4.7M, symbol cx:R
- added V1B, V2B, V3A, V3B, V4B, V5A, V5B: 7025, symbol cx:TRIODE
- added VRB2: 250k-A, symbol cx:POT
- CBR1: renamed from V1B; value 7025 -> 47p; symbol cx:TRIODE -> cx:C
- CC1T: renamed from RS1T; value 100k -> .05u; symbol cx:R -> cx:C
- CKV: renamed from RTOG1; value 1M -> 2u 25V; symbol cx:R -> cx:C
- CLP: renamed from RG5; value 1M -> .005u; symbol cx:R -> cx:C
- CPP: renamed from CF4; value 20u 600V -> 47p
- CT2: renamed from VRB2; value 250k-A -> 250p; symbol cx:POT -> cx:C
- CTO3: renamed from CTOK; value 25u+25u -> .02u
- D3: renamed from DBIAS; value Si -> 1N4007
- D5: renamed from RBIAS2; value 10k -> 1N4007; symbol cx:R -> cx:DIODE_SS
- JVIB: renamed from V6A; value 7025 -> vibrato pedal; symbol cx:TRIODE -> cx:JACK
- R1H: renamed from RG1A; value 1M -> 68k
- RD1: value 56k 1W -> 4.7k 1W
- RD2: value 10k -> 56k 1W
- RF1: renamed from CBR1; value 47p -> 10k; symbol cx:C -> cx:R
- RF2: renamed from V2B; value 7025 -> 10k; symbol cx:TRIODE -> cx:R
- RGV1: renamed from CFB1; value .0025u -> 1M; symbol cx:C -> cx:R
- RL1A: renamed from RK1A; value 820 -> 100k
- RL2B: value 100k -> 220k
- RMV1: renamed from CTO1; value .01u -> 470k; symbol cx:C -> cx:R
- RSV: renamed from CPID; value .001u -> 1M; symbol cx:C -> cx:R
- RTOK: renamed from RLB; value 100k 5% -> 4.7k
- RTOP: value 100k -> 470k
- V1A: Basing_unit (none) -> 1
- V2A: Basing_unit (none) -> 2
- V4A: renamed from V5; Basing_unit (none) -> 2
- VRINT: value 250k-L intens. -> 10M-L
- VRPRES: value 5k-L pres. -> 5k-L
- VRSPD: value 4M-RA speed -> 4M-RA
- renumbered RS2T to RL2A
Connections:
- net -55V: now also RBIAS2.2; no longer D5.2
- net BP1: now also RD1.1, RSC1.2, RSC2.2, CF4.1, RD3.1; no longer CPP.1, RTOP.1
- net B_RES: now also D3.2 (K)
- net GND: now also CKV.2, JSPK.2 (S), JVIB.2 (S), RF1.2, RF2.2, RG2A.1, RTOG2.2, RTOK.2, TR2.5 (SEC_C), CF4.2, CF8.2, CGS.2, CK1.2, CK2.2, CKS.2, CPS.2, CTOK.2, CTOP.2, CTW.2, CTX.2, RG1A.1, RGS.2, RHP2.2, RK1.2, RK2.2, RKS.2, RKV.2, RSPD.1, VRB2.3; no longer CPP.2, CT2.3, CTO3.2, R1H.2, RG2A.2, RGV1.1, RL1A.2, RTOG2.1, VRSPD.1, VRSPD.2 (W)
- net HT_TAP: now also DBIAS.2 (K); no longer D3.2 (K)
- net at VRT1.2 (W), VRV1.1: now also CBR1.1; no longer RF1.1
- net at CBR1.2, VRV1.2 (W): now also V2A.2 (G); no longer RF1.2
- net at CF1.2: now also RF1.1, VRB1.2 (W)
- net at C1.1, RLA.2: now also CPP.1, V5A.1 (P); no longer JVIB.1 (P), RSV.1
- net at CTO3.1: now also VRSPD.3, CTO1.2; no longer CKV.1
- net at RNFB.2, RPRES.1, RT2.1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: now also CGB.1
- net at V1A.1 (P): now also CC1T.1, RL1A.2
- net BA: now reaches RL1A.1
- net BA: now also CF6.1, RD2.2, RL2A.1, RL2B.1, RLD1.1; no longer V1A.3 (K)
- net at CF1.1, VRB1.1, VRT1.3: now also RS1T.2; no longer CC1T.2
- net at D6.1 (A): now also D5.2 (K)
- net at CTO2.1: now also RTOG2.1, V3A.2 (G); no longer RTOG2.2
- net at RTOP.2: now also CTO3.2, CTOP.1, RTOF.1, V3A.1 (P); no longer VRINT.1
- net at RL1B.2: now also V2A.1 (P); no longer CBR1.1 (P)
- net at RL2B.2: now also CC2D.1, V2B.1 (P); no longer RF2.1 (P)
- net at D4.2 (K): now also D5.1 (A)
- net VMIX: now reaches RMV1.2
- net VMIX: now also CPIN.1, RM2.2, RMV2.1; no longer VRSPD.3
- net at D2.2 (K): now also D3.1 (A)
- net at RGB.2: now also CGB.2, V5B.2 (G)
- net at RTAIL.2: now also V5A.3 (K), V5B.3 (K); no longer JVIB.3 (K)
- net at CF2.2: now also RF2.1, VRB2.2 (W)
- net at CT1.1: now also CC1T.2, RS1T.1; no longer CC1T.1
- net at VRT2.1: now also CT2.2
- net at CF2.1, VRT2.3: now also RS2T.2, VRB2.1; no longer CT2.1, RL2A.2
- net at VRINT.2 (W): now also CTW.1, RWV.1
- net at CC2T.1: now also RL2A.2, V1B.1 (P); no longer V2A.1 (P)
- net at CC2T.2: now also CT2.1, RS2T.1; no longer RL2A.1
- net at RGA.1: now also CPIN.2, V5A.2 (G); no longer JVIB.2 (G)
- net at VRV2.2 (W): now also V2B.2 (G); no longer RF2.2 (G)
- net at V4A.1 (P): now also RMV1.1, RLV1.2; no longer RGV1.2
- net K2: now reaches V2A.3 (K)
- net K2: now also CK2.1, RK2.1, V2B.3 (K)
- net KV: now reaches V4A.3 (K)
- net KV: now also CKV.1, RKV.1, V4B.3 (K)
- removed net BD: CF7.1, RD2.2, RL1B.1, RL2B.1
- removed net BP2: CF5.1, RD1.1, RSC1.2, RSC2.2
- net BP3 renamed BC
- net BC: now also CF5.1, RLB.1; no longer CF6.1, RTOK.1
- removed net BRT 1: R2N.2, RG2A.1, V2A.2 (G)
- net BRT 2 renamed CH2 IN 2
- net MIXG2: no longer names the net of CLP.1
- net MIXG2: now also CV1.1, RLP.2; no longer V4A.2 (G)
- net NORM 1: no longer names the net of R1N.2, V1A.2 (G)
- net NORM 1: now also R1H.2; no longer R1H.1
- net NORM 2 renamed CH1 IN 2
- new net: R2H.2, R2N.2, V1B.2 (G)
- new net: CC1D.2, RHP1.1, RLP.1
- new net: CC1D.1, RL1B.1, RLD1.2
- new net: RSPD.2, VRSPD.1, VRSPD.2 (W)
- new net: CV2.1, RHP1.2, RHP2.1
- new net: CFS.1, CPS.1, CSV.1, RLS.2, V3B.1 (P)
- new net: CKS.1, RKS.1, V3B.3 (K)
- new net: CBIAS.1, DBIAS.1 (A), RBIAS2.1
- new net: RLV2.2, RMV2.2, V4B.1 (P)
- new net: CC2D.2, RM2.1
- new net: CTOF.2, CTX.1, VRINT.1
- new net: C2.1, CPP.2, RLB.2, V5B.1 (P)
- new net: CSV.2, RSV.1
- new net: CTOF.1, RTOF.2
- new net: CTOK.1, RTOG1.2, RTOK.1, V3A.3 (K)
- new net: CTO1.1, CTO2.2, JVIB.1 (T), RTOG1.1
- new net BL: CF8.1, RD4.2, RLS.1, RTOP.1
- new net BV: CF7.1, RD3.2, RD4.1, RLV1.1, RLV2.1
- new net CH1 IN 1: R1H.1, RG1A.2
- new net CH2 IN 1: R2H.1, RG2A.2
- new net GS: CFS.2, CGS.1, RGS.1, RGV1.2, RGV2.1, V3B.2 (G)
- new net GV1: CV1.2, RGV1.1, RWV.2, V4A.2 (G)
- new net GV2: CV2.2, RGV2.2, RSV.2, V4B.2 (G)
- new net K1: CK1.1, RK1.1, V1A.3 (K), V1B.3 (K)
Other:
- note added: "+458 V"
- note added: "+460 V"
- note added: "Bias supply — TR1's bias tap, a rectifier, 8 µF, 10k, then 8 µF with a 56k bleeder: -55 V"
- note added: "Channel 1 — V1A, tone network and Volume, V2A (into the vibrato)"
- note added: "Channel 2 — V1B, tone network and Volume, V2B (to the mixing node)"
- note added: "Harmonic vibrato — the band-splitting filters and the vibrato pair V4"
- note added: "Heaters, the standby switch and the second of the two 20 µF reservoir cans are omitted here — see the sources list and the board drawing."
- note added: "Intensity"
- note added: "K1 and K2 are the two shared cathode pairs the factory sheet letters C and D: both first stages (V1) sit on one 820 Ω / 25 µF, both second stages (V2) on another."
- note added: "Long-tailed-pair phase inverter (V5)"
- note added: "Output pair — 6L6GC, grounded cathodes, fixed bias"
- note added: "Pilot lamp — across the 6.3 V heater supply"
- note added: "Power supply — silicon full-wave (two legs of three diodes), choke, and the dropper chain to every rail"
- note added: "Presence"
- note added: "Rails: BP1 +456 (6L6GC plates; the screens and every dropper hang at the drawing's +458 V post-choke node, choke and transformer resistance omitted) · BC +430 (phase inverter) · BA +260 (both channels) · BV +350 (vibrato pair) · BL +275 (oscillator and splitter) · bias -55 V"
- note added: "The vibrato oscillator V3A is drawn in full and excluded from the DC model — a running phase-shift oscillator has no static operating point. The splitter V3B and the vibrato pair V4 are modelled."
- note added: "Vibrato oscillator V3A (excluded from the DC model) and its phase splitter V3B"
- note removed: "+430 V"
- note removed: "+456 V"
- note removed: "+460 V reservoir"
- note removed: "56k/10k dropper — illustrative; BP3/BDRV/BD are driven anchors (see header). The driver rail sits above the reservoir this chain hangs from, so no tap off it is drawn."
- note removed: "Bias supply — TR1's bias tap, a rectifier, 8 uF, 10k, then 8 uF with a 56k bleeder, to -55 V (the netlist drives the -55 V line as an ideal source)"
- note removed: "Bright channel — V2 (both stages share one 7025)"
- note removed: "Channel-mixing node — both channels sum here; the tremolo photocell (below) also shunts it"
- note removed: "Driver — local feedback network read from the drawing but not confidently resolved (schematic-only; see the circuit story and the parts list)"
- note removed: "HT"
- note removed: "Heaters, PT primary/mains, pilot lamp and chassis switches are omitted here — see the netlist, the sources list and the board drawing. BP3/BDRV/BD are DRIVEN anchors, not derived through the dropper chain shown (see the circuit story)."
- note removed: "Long-tailed-pair phase inverter"
- note removed: "Mains cord not drawn — annotation layer (see the board drawing)"
- note removed: "Normal channel — V1 (both stages share one 7025)"
- note removed: "Output pair — grounded cathodes, fixed bias"
- note removed: "Phase-shift ladder values (RTOG1/RTOG2/CTO1-3) are a schematic-only reading, typical of this circuit family — not confidently resolved from the scan (see the parts list)."
- note removed: "Pilot lamp — fed from the 6.3 V heater chain (the board drawing's twisted pair)"
- note removed: "Power supply — silicon full-wave: two legs of three diodes off the centre-tapped HT winding (no tube rectifier); TR1 power, TR2 output (drawing's own designators)"
- note removed: "Rails: BP1 +456 (post-choke) · BP2 +430 screens · BP3 +410 (PI, driven anchor) · BDRV +480 (driver, driven anchor) · BD +300 (preamp, driven anchor) · bias -55 V"
- note removed: "The tremolo oscillator drives a lamp/photoresistor pair (OPTO) whose photocell shunts the channel-mixing node (see the circuit story)."
- note removed: "Tremolo — V3 phase-shift oscillator (DC point excluded from the netlist)"
- note removed: "Vibrato pedal"
- moved on the sheet: CPP, CTO3, D3, R1H, RL1A, RL2A, RTOK, V4A

Commit message: Fix: the 6G5's rectifier and bias sub-board drawn beside TR1; the OT centre tap on +460 V ahead of the choke
The A-FJ layout page boxes a sub-board beside the power transformer: each
RED HT lead through a leg of three silicon diodes, every one lettered
"- |> +" with the + toward the join, and the RED-BLUE tap through the bias
rectifier (+ toward the tap), 8-150 and 10K, then 8-150 and a 56K bleeder on
-55 V. The board declared all eleven parts not_on_board. They are now drawn
at the power end in the 6G6-B idiom: the diodes along row 1 banded at their
cathodes, both cans standing with the lead the page letters + on top and on
ground, row 0 left open for the labels. net_map.leads maps the sheet's TR1
pins 3, 5 and 6 to the two red leads and the red-blue tap, which resolves the
six diodes on the sheet-to-board gate (UNRESOLVED 6 -> 0). D3, D6 and DBIAS
read confirmed on both surfaces; D1, D2, D4, D5 sit inside their stacks, on
no modelled node, and are walked as part of them.

Both pages land the output transformer's red centre-tap lead on the +460 V
node ahead of the choke: the layout page's "RED +460V" eyelet, and on the
schematic page the centre-tap line runs to +460 while the screens' line runs
to +458 at B. The board had the lead on the screen node after the choke; with
the choke drawn, that is a different net, and the net gate says so
("netlist node BP1 is realised as 2 separate board nets"). The model now
drives BR at the printed +460 V (the centre tap, and the plates, OT winding
resistance omitted) and BP1 at the printed +458 V (screens and droppers). The
choke's resistance is not printed, so the 2 V between them cannot be derived;
both stay anchors. Derived rails move with BP1: BC 428.4 -> 430.3 (printed
430), BA 251.3 -> 252.5 (260), BV 357.4 -> 359.0 (350), BL 299.6 -> 300.9
(275), screens 455.9 -> 457.9 (458), PI plates 310.4/301.0 -> 311.8/302.3
(315/310), KPI 24.5 -> 24.6 (23).

Sheet: the OT centre tap on B_RES; sch_map TR2.1-3 -> BR. BOM: DBIAS loses
"(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
Connections:
- net BP1: no longer TR2.2 (CT)
- net B_RES: now also TR2.2 (CT)
Changed lines of the file:
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@@
   (wire (pts (xy 406.446 91.82) (xy 398.336 91.82))
     (stroke (width 0) (type default)))
-  (global_label "BP1" (shape input) (at 398.336 91.82 180)
+  (global_label "B_RES" (shape input) (at 398.336 91.82 180)
     (effects (font (size 1.27 1.27)) (justify right)))
   (wire (pts (xy 424.226 89.28) (xy 428.336 89.28))
