File: amps/6161/schematic.kicad_sch (KiCad schematic)
At the start: 80 parts, among them SW1 SPST, T1 E-3693A, T2 340-6

Commit message: Fix: schematic sheets — real title block, fitted paper, no lettering through circuitry
Every sheet in the corpus shipped with an EMPTY title block ("Title:" and
"Date:" blank, default "Sheet /" furniture) laid onto a fixed A4/A3 page
regardless of the drawing's size, with prose annotations placed by hand
wherever a coordinate looked free when the amp was first drawn. The result
read as an unfinished alpha under a `verified` badge: KiCanvas's default view
is `zoom_to_page()`, so a 150 x 110 mm circuit on an A3 sheet opened as a
postage stamp, and later edits had pushed live circuitry under the prose.

schematic_lib.py — the builder now records each element as a (kind, points,
extra) tuple instead of a finished string, so `write()` can measure and move
what it emits:

- emits a real `(title_block …)` read from the amp's own meta.yaml — Title =
  designation + style, Date = the verification (or added) date, Rev = the
  verification status, Company = Circuit Codex, plus the licence and source
  URL as comments. Fixes all 34 sheets from one place;
- emits `(paper "User" w h)` cut to the drawing, translated to a fixed margin,
  with the bottom 34 mm strip reserved for the worksheet's title block. Sheet
  utilisation of the drawable area went from as low as ~20% to 92-98%;
- `note()` queues prose into a wrapped band under the circuit, and `caption()`
  places a section heading over the block it names, nudging it clear if it
  would print through anything;
- per-symbol default label offsets (the old single default printed every pot's
  value through its own wiper arrow and every transformer's designator through
  its body), plus `place_labels()`, which moves any designator/value block that
  would print over ink;
- transformers and chokes are drawn, not boxed: iron core between two windings,
  centre taps where the part has them, and an optional `spec` lettering slot for
  a ratio or impedance;
- `gnd()` takes a direction, because a flag defaulting to "down" at the HEAD of
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
Connections:
- net GND: no longer RI1.2, VR2.3
- net at CI1.1, CP2.2, RL2.2: no longer V1B.1 (P)
- net at CC1.2, V5.2 (G1): no longer RPA.1
Other:
- note added: "Channel 2 also carries a 500 pF cut on its plate, and its cathode is node C — shared with the tremolo follower."
- note added: "Channel 2 — 2.2 kΩ grid stopper, 1.5 kΩ cathode bypassed by 35 µF"
- note removed: "6161 — Valco 6161-style · Circuit Codex · CC-BY-SA 4.0 · redrawn from circuit facts"
- note removed: "Channel 2 — 2.2 kΩ grid stopper, 1.5 kΩ cathode bypassed by 35 µF, and a 500 pF cut on the plate. Its cathode is node C, shared with the tremolo follower."
- company: (none) -> Circuit Codex
- title: (none) -> 6161 — Valco 6161-style

Commit message: Fix: deterministic schematic ids and wires split at every join
- _u() is uuid5 over (amp id, emission order), so a regeneration of an
  unchanged script is byte-identical and a drift gate becomes possible
- write() splits wire segments at symbol pins, wire ends and junction dots,
  so the file connects exactly what the drawing shows under KiCad's
  endpoint-only semantics (270 pins were on a wire's interior; net
  partitions unchanged on all 38 sheets)
- all sheets regenerated; aa864-bassman title block was stale (draft) and
  now matches meta.yaml (verified)

Co-Authored-By: Claude Fable 5.1 <noreply@anthropic.com>
Claude-Session: https://claude.ai/code/session_01KBMfdh37HmCL2iWcBiL5J1
Changed lines of the file:
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@@
   (wire (pts (xy 54.51 52.1544) (xy 64.7 52.1544))
     (stroke (width 0) (type default)))
-  (wire (pts (xy 64.7 42.1544) (xy 64.7 52.1544))
+  (wire (pts (xy 64.7 42.1544) (xy 64.7 47.1544))
+    (stroke (width 0) (type default)))
+  (wire (pts (xy 64.7 47.1544) (xy 64.7 52.1544))
     (stroke (width 0) (type default)))
   (junction (at 64.7 47.1544) (diameter 0) (color 0 0 0 0))
@@
   (wire (pts (xy 54.51 110.154) (xy 64.7 110.154))
     (stroke (width 0) (type default)))
-  (wire (pts (xy 64.7 100.154) (xy 64.7 110.154))
+  (wire (pts (xy 64.7 100.154) (xy 64.7 105.154))
+    (stroke (width 0) (type default)))
+  (wire (pts (xy 64.7 105.154) (xy 64.7 110.154))
     (stroke (width 0) (type default)))
   (junction (at 64.7 105.154) (diameter 0) (color 0 0 0 0))
@@
   (wire (pts (xy 240.7 55.1544) (xy 248.89 55.1544))
     (stroke (width 0) (type default)))
-  (wire (pts (xy 256.51 55.1544) (xy 327.08 55.1544))
+  (wire (pts (xy 256.51 55.1544) (xy 274.7 55.1544))
+    (stroke (width 0) (type default)))
+  (wire (pts (xy 274.7 55.1544) (xy 292.7 55.1544))
+    (stroke (width 0) (type default)))
+  (wire (pts (xy 292.7 55.1544) (xy 327.08 55.1544))
     (stroke (width 0) (type default)))
   (junction (at 274.7 55.1544) (diameter 0) (color 0 0 0 0))
@@
   (wire (pts (xy 296.7 171.154) (xy 296.7 160.154))
     (stroke (width 0) (type default)))
-  (wire (pts (xy 292.7 160.154) (xy 327.08 160.154))
+  (wire (pts (xy 292.7 160.154) (xy 296.7 160.154))
+    (stroke (width 0) (type default)))
+  (wire (pts (xy 296.7 160.154) (xy 304.7 160.154))
+    (stroke (width 0) (type default)))
+  (wire (pts (xy 304.7 160.154) (xy 327.08 160.154))
     (stroke (width 0) (type default)))
   (junction (at 296.7 160.154) (diameter 0) (color 0 0 0 0))
@@
   (wire (pts (xy 174.7 208.774) (xy 174.7 209.154))
     (stroke (width 0) (type default)))
-  (wire (pts (xy 120.7 209.154) (xy 182.7 209.154))
+  (wire (pts (xy 120.7 209.154) (xy 132.7 209.154))
+    (stroke (width 0) (type default)))
+  (wire (pts (xy 132.7 209.154) (xy 152.7 209.154))
+    (stroke (width 0) (type default)))
+  (wire (pts (xy 152.7 209.154) (xy 174.7 209.154))
+    (stroke (width 0) (type default)))
+  (wire (pts (xy 174.7 209.154) (xy 182.7 209.154))
     (stroke (width 0) (type default)))
   (junction (at 132.7 209.154) (diameter 0) (color 0 0 0 0))
@@
   (wire (pts (xy 380.7 215.154) (xy 380.7 225.154))
     (stroke (width 0) (type default)))
-  (wire (pts (xy 364.7 225.154) (xy 380.7 225.154))
+  (wire (pts (xy 364.7 225.154) (xy 372.7 225.154))
+    (stroke (width 0) (type default)))
+  (wire (pts (xy 372.7 225.154) (xy 380.7 225.154))
     (stroke (width 0) (type default)))
   (junction (at 372.7 225.154) (diameter 0) (color 0 0 0 0))

Commit message: Fix: schematic wiring on the tweed family, jtm45 and 6161
- pot cold lugs: s.gnd() sat 3.81 mm below cx:POT pin 3 on nine sheets
  (19 pins); every flag now lands on the lug
- retyped coordinates replaced by helper returns (5e5a OT pins alone freed
  nine pins; 5d3 V3 cathode, 5f10 RKB, 5e6a CBS, 5f2a dropper, grid leaks)
- shorts only verify_schematic_nets could see: 5e3 cathode bus through V4's
  screen pin (B+2 tied to the cathodes), C7 through RG6A, PI leak through
  RGPI, C8 on the cathode not the tail; 5f10 the same RGPI/C7 pair; 5e5a
  presence feed down the tube column; 5e6a RFB loop through RL3
- three dated waivers: two-terminal rheostat far lugs (5e6a VR5, 6161 VR3/VR4)

Co-Authored-By: Claude Fable 5.1 <noreply@anthropic.com>
Claude-Session: https://claude.ai/code/session_01KBMfdh37HmCL2iWcBiL5J1
Parts:
- removed CK3: .05u, symbol cx:C
- removed CKO: 35u, symbol cx:C
- removed RTI2: 1.5M, symbol cx:R
- removed SW1: SPST, symbol cx:SWITCH
- removed V3B: 12AX7, symbol cx:TRIODE
- removed V4: 6973, symbol cx:PENTODE
- removed VR4: 500k-A, symbol cx:POT
- added CTI1: .05u, symbol cx:C
- added CTOUT: .01u, symbol cx:C
- added RGS2, RK3: 2.2k, symbol cx:R
- added RKO: 250 7W, symbol cx:R
- added RSPD: 100k, symbol cx:R
- added V5: 6973, symbol cx:PENTODE
- CK3: renamed from RK3; value 2.2k -> .05u; symbol cx:R -> cx:C
- CKO: renamed from RKO; value 250 7W -> 35u; symbol cx:R -> cx:C
- RTI2: renamed from CTI1; value .05u -> 1.5M; symbol cx:C -> cx:R
- RTOUT: renamed from CTOUT; value .01u -> 1M; symbol cx:C -> cx:R
- SW1: renamed from RTOUT; value 1M -> SPST; symbol cx:R -> cx:SWITCH
- V3B: renamed from RGS2; value 2.2k -> 12AX7; symbol cx:R -> cx:TRIODE
- VR4: renamed from RSPD; value 100k -> 500k-A; symbol cx:R -> cx:POT
- renumbered V5 to V4
Connections:
- net B1: now also V3B.1 (P)
- net BP2: now also V5.3 (G2)
- net C: now also V3B.3 (K)
- net FT SW: now also SW1.2
- net GND: now also VR4.2 (W), CTI1.2, RK3.2, RKO.2; no longer RTI2.2
- net KOUT: now also CKO.1, RKO.1, V5.4 (K)
- net at CTO1.2, RTO1.1, V3A.1 (P): now also CTOUT.1; no longer RTOUT.1
- net at CC2.2, RGL2.1: now also V4.2 (G1)
- net at CTI2.1, RTI.1: now also RTI2.2, RGS2.1; no longer V3B.1
- net at CK3.1, V2A.3 (K): now also RK3.1
- net at RTI1.2, RTI2.1: now also CTI1.1
- net at CTO1.1, CTO2.1: now also RSPD.1; no longer VR4.1
- net at V3B.2 (G): now also RGS2.2
- net at T2.3 (PRI_B): now also V4.1 (P)
- net at CC1.2: now also V5.2 (G1); no longer V4.2 (G1)
- net at T2.1 (PRI_A): now also V5.1 (P); no longer V4.1 (P)
- new net: CTOUT.2, RTOUT.1
- new net: RSPD.2, VR4.1
Other:
- moved on the sheet: V4
Changed lines of the file:
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@@
   (global_label "GND" (shape input) (at 204.7 85.1544 0)
     (effects (font (size 1.27 1.27)) (justify left)))
-  (wire (pts (xy 192.7 88.9644) (xy 192.7 91.1544))
-    (stroke (width 0) (type default)))
   (text "Tone — a rheostat: wiper to ground, far lug left free" (at 178.7 95.1544 0)
     (effects (font (size 1.2 1.2)) (justify left)))
@@
   (global_label "KOUT" (shape input) (at 280.7 194.154 180)
     (effects (font (size 1.27 1.27)) (justify right)))
-  (wire (pts (xy 284.7 194.154) (xy 292.7 194.154))
+  (wire (pts (xy 280.7 194.154) (xy 292.7 194.154))
     (stroke (width 0) (type default)))
   (symbol (lib_id "cx:R") (at 292.7 197.964 0) (unit 1)
@@
   (wire (pts (xy 120.7 201.584) (xy 120.7 209.154))
     (stroke (width 0) (type default)))
-  (wire (pts (xy 112.7 205.394) (xy 112.7 208.154))
-    (stroke (width 0) (type default)))
   (text "Speed" (at 98.7 199.154 0)

Commit message: Add: real tube pin numbers and readable valve glyphs on every schematic
Phase B of the drawing program. A factory service sheet numbers every tube
pin, because the number is what a technician puts a probe on. This corpus
printed none, and the numbers hidden in its symbols were positional
placeholders (P=1, G=2, K=3) that would have published a 6V6GT's plate as
pin 1 when it is pin 3.

1055 electrodes now carry the real number, 1027 lettered (27 are shared
filaments deduped, 1 dropped for want of clear space on the 6G2). Resolved per
instance from reference/tubes/<slug>.yaml through the same alias resolution the
layout renderer uses, so a 12AX7 section and a 6SL7 section each get their own
basing. A valve whose basing the corpus does not carry prints nothing rather
than a wrong number.

Section letters and basing units are now separate things, which cost a detour
worth recording. The RCA 12AX7-A sheet reads "Pin 1 - Plate of Unit No.2 ...
Pin 6 - Plate of Unit No.1", so unit numbering is not pin order; the 5Y3 and
GZ34 number their units in opposite pin order, so nothing positional can
express it. But the section LETTER is a designator, not a basing fact: this
corpus, like every technician, calls the first stage in signal order V1A, and
five amps' prose already did. On four amps the factory sheets put that first
stage on the other half -- the AA764's own schematic prints +200 V on pin 1 --
so those drawings now state their unit explicitly, each citing its source, and
no letter, netlist, parts list or layout comment changed. 183 layout comments
agree with the printed numbers, 0 disagree. A guard fires if two halves of one
bottle resolve to the same unit, which is exactly how this was found.

Glyphs: the cathode gains a bracket and filament hairpin so it can no longer be
confused with the plate bar, the pentode's screen sits on its own row, and a
rectifier draws as one envelope over its sections instead of two apparent
bottles. Line weights are scaled per sheet to a co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
Other:
- note added: "1"
- note added: "1,8"
- note added: "2"
- note added: "2,8"
- note added: "3"
- note added: "3,6"
- note added: "4"
- note added: "6"
- note added: "7"
- note added: "8"
- note added: "9"

Commit message: Fix: schematic sheet notes no longer name repository files
Thirty-seven committed sheets rendered footnotes and section notes such as
"Heaters and PT primary omitted — see netlist.cir and meta.yaml" or
"excluded from netlist.cir (notes.md)" to visitors through KiCanvas. The
prose sweeps never counted sheets. Rewritten in the site's own words — the
netlist, the sources list, the circuit story, the parts list, the board
drawing — in 59 strings across 33 draw scripts, keeping every technical
claim as it was; the three tone sheets (6G4, 6G5, 6G6-B) are under repair
elsewhere and keep theirs for now. The sweep touched only strings passed to
the sheet's note, text, caption and footnote calls, never a path or a value.

Gates: check_schematics 40/0, connectivity 0 isolated pins;
verify_schematic_nets 40 clean; only the regenerated sheets and their served
copies changed.

Co-Authored-By: Claude Fable 5.1 <noreply@anthropic.com>
Claude-Session: https://claude.ai/code/session_01KBMfdh37HmCL2iWcBiL5J1
Other:
- note added: "Heaters, the mains side beyond the transformer (2 A fuse, switch, mains capacitor, line-reverse arrangement), the neon pilot, the input and footswitch jacks and the two 10-inch speakers are omitted here — see the netlist, the parts list, the board drawing."
- note added: "Tremolo — a phase-shift oscillator on V3A with Speed wired as a rheostat. Its DC point alone is excluded from the netlist: a running oscillator has no static operating point (see the circuit story)."
- note removed: "Heaters, the mains side beyond the transformer (2 A fuse, switch, mains capacitor, line-reverse arrangement), the neon pilot, the input and footswitch jacks and the two 10-inch speakers are omitted here — see netlist.cir, bom.yaml, layout.yaml."
- note removed: "Tremolo — a phase-shift oscillator on V3A with Speed wired as a rheostat. Its DC point alone is excluded from netlist.cir: a running oscillator has no static operating point (notes.md)."
Changed lines of the file:
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@@
   (symbol (lib_id "cx:C") (at 264.7 171.154 90) (unit 1)
     (in_bom yes) (on_board yes)
-    (property "Reference" "CC2" (at 261.5 164.954 270) (effects (font (size 1.27 1.27)) (justify left)))
-    (property "Value" ".01u" (at 261.5 167.354 270) (effects (font (size 1.27 1.27)) (justify left))))
+    (property "Reference" "CC2" (at 266.362 170.022 270) (effects (font (size 1.27 1.27)) (justify left)))
+    (property "Value" ".01u" (at 266.362 172.422 270) (effects (font (size 1.27 1.27)) (justify left))))
   (wire (pts (xy 240.7 171.154) (xy 260.89 171.154))
     (stroke (width 0) (type default)))
@@
   (global_label "GND" (shape input) (at 410.7 109.694 0)
     (effects (font (size 1.27 1.27)) (justify left)))
-  (text "Tremolo — a phase-shift oscillator on V3A with Speed wired as a rheostat. Its DC point alone is excluded from netlist.cir: a running oscillator has no static operating point (notes.md)." (at 48.7 167.154 0)
+  (text "Tremolo — a phase-shift oscillator on V3A with Speed wired as a rheostat. Its DC point alone is excluded from the netlist: a running oscillator has no static operating point (see the circuit story)." (at 48.7 167.154 0)
     (effects (font (size 1.5 1.5)) (justify left)))
   (symbol (lib_id "cx:TRIODE") (at 174.7 190.154 0) (unit 1)
@@
   (text "Rails: BP1 reservoir · OT centre tap · 6973 plates — BP2 6973 screens, on their OWN supply node (not tapped on the transformer primary) — B1 preamp and inverter rail. The drawing prints no voltages of any kind." (at 12.7 264.585 0)
     (effects (font (size 1.2 1.2)) (justify left)))
-  (text "Heaters, the mains side beyond the transformer (2 A fuse, switch, mains capacitor, line-reverse arrangement), the neon pilot, the input and footswitch jacks and the two 10-inch speakers are omitted here — see netlist.cir, bom.yaml, layout.yaml." (at 12.7 268.985 0)
+  (text "Heaters, the mains side beyond the transformer (2 A fuse, switch, mains capacitor, line-reverse arrangement), the neon pilot, the input and footswitch jacks and the two 10-inch speakers are omitted here — see the netlist, the parts list, the board drawing." (at 12.7 268.985 0)
     (effects (font (size 1.2 1.2)) (justify left)))
   (text "The two stubs lettered A are the sheet's own markers on the two output-grid nodes; they are two separate nodes, not one, and the published redraw of the Supro-badged sibling bridges them with a silencing switch." (at 12.7 273.385 0)

Commit message: Fix: state the datasheet unit on 17 dual-triode sections whose sheets printed the other half's pin numbers
The sheet-vs-board gate reported these sockets as SECTION-SWAP; the
2026-09-10 source-read triage found the BOARD right on every one of them
(and both surfaces wrong on the 5G9 tremolo bottle). Each sheet had
lettered the section on the default map (A -> unit 1 -> pins 6/7/8) where
the factory drawing puts that stage on 1/2/3. The draw scripts now state
`unit=` on both halves, with the source cited beside the call, so the
printed socket numbers are the factory's:

- 5f4 V3: driver V3A -> 1/2/3, cathodyne V3B -> 6/7/8
  (crop 5f4-V3-layout-trace.png: +213 V driver plate -> pin 1, +270 V -> 6)
- 5f8a V3: 82k half V3A -> 1/2/3, 100k half V3B -> 6/7/8
  (crop 5f8a-V3-layout-trace.png: +225 -> 6, +19 -> 2, +28.5 -> 8)
- 6161 V1: channel 1 V1A -> 1/2/3 (crop 6161-V1-ch1.png prints 1/2/3);
  6161 V2: 1 MEG-grid half V2A -> 1/2/3, paraphase V2B -> 6/7/8
  (crop 6161-V2.png / 6161-V2-right.png)
- 6g3 V3: 82k half V3A -> 1/2/3 (crop 6g3-V3-layout-wires.png: +230 -> 1,
  +225 -> 6, +20 -> 7)
- aa1164 V3: recovery V3A -> 1/2/3, mixer V3B -> 6/7/8
  (crops aa1164-V3A-recovery-schem.png, aa1164-V3B-mixer-schem.png)
- aa864-bassman V1/V2: input stages 2/1/3, second stages 7/6/8; V4: the
  .1/500 pF-fed 82k half 2/1/3 (crops aa864-V1A-input.png,
  aa864-V1B-second.png, aa864-V2A-input.png, aa864-V2B-second.png,
  aa864-V4-PI.png)
- ab165 V1/V2/V4: same pattern (crops ab165-V1A-input.png,
  ab165-V1B-second.png, ab165-V2A-input.png, ab165-V2B-second.png,
  ab165-V4-PI.png)
- ab763-super V1/V2: slope-plate +270 V -> pin 1 (input stage), .047
  plate -> 6 (crops ab763-super-V1-layout-sh.png, ab763-super-V2-layout-sh.png)
- dr103 V2/V3: gain stages 6/7/8, cathode followers 1/2/3 (crops
  dr103-V2-huss.png, dr103-V3-huss.png — the Huss redraw, not a factory
  print; noted in the script)
- 5g9 V3: oscillator V3A -> 1/2/3, follower V3B -> 6/7/8 (crops
  5g9-V3-strap71-zoom.png, 5g9-V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
Parts:
- V1A, V2A: Basing_unit (none) -> 2
- V1B, V2B: Basing_unit (none) -> 1
Changed lines of the file:
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@@
     (in_bom yes) (on_board yes)
     (property "Reference" "V1A" (at 84.7 40.7544 0) (effects (font (size 1.27 1.27)) (justify left)))
-    (property "Value" "12AX7" (at 84.7 43.1544 0) (effects (font (size 1.27 1.27)) (justify left))))
+    (property "Value" "12AX7" (at 84.7 43.1544 0) (effects (font (size 1.27 1.27)) (justify left)))
+    (property "Basing_unit" "2" (at 84.7 45.5544 0) (effects (font (size 1.27 1.27)) hide)))
   (wire (pts (xy 64.7 47.1544) (xy 71.08 47.1544))
     (stroke (width 0) (type default)))
@@
     (in_bom yes) (on_board yes)
     (property "Reference" "V1B" (at 90.7 98.7544 0) (effects (font (size 1.27 1.27)) (justify left)))
-    (property "Value" "12AX7" (at 90.7 101.154 0) (effects (font (size 1.27 1.27)) (justify left))))
+    (property "Value" "12AX7" (at 90.7 101.154 0) (effects (font (size 1.27 1.27)) (justify left)))
+    (property "Basing_unit" "1" (at 90.7 103.554 0) (effects (font (size 1.27 1.27)) hide)))
   (symbol (lib_id "cx:R") (at 70.7 105.154 90) (unit 1)
     (in_bom yes) (on_board yes)
@@
     (in_bom yes) (on_board yes)
     (property "Reference" "V2A" (at 240.7 65.7544 0) (effects (font (size 1.27 1.27)) (justify left)))
-    (property "Value" "12AX7" (at 240.7 68.1544 0) (effects (font (size 1.27 1.27)) (justify left))))
+    (property "Value" "12AX7" (at 240.7 68.1544 0) (effects (font (size 1.27 1.27)) (justify left)))
+    (property "Basing_unit" "2" (at 240.7 70.5544 0) (effects (font (size 1.27 1.27)) hide)))
   (wire (pts (xy 216.7 72.1544) (xy 227.08 72.1544))
     (stroke (width 0) (type default)))
@@
     (in_bom yes) (on_board yes)
     (property "Reference" "V2B" (at 240.7 118.754 0) (effects (font (size 1.27 1.27)) (justify left)))
-    (property "Value" "12AX7" (at 240.7 121.154 0) (effects (font (size 1.27 1.27)) (justify left))))
+    (property "Value" "12AX7" (at 240.7 121.154 0) (effects (font (size 1.27 1.27)) (justify left)))
+    (property "Basing_unit" "1" (at 240.7 123.554 0) (effects (font (size 1.27 1.27)) hide)))
   (wire (pts (xy 234.7 117.534) (xy 234.7 114.054))
     (stroke (width 0) (type default)))
@@
   (polyline (pts (xy 362.8 209.769) (xy 364.7 208.169) (xy 372.7 210.249) (xy 380.7 208.169) (xy 382.6 209.769))
     (stroke (width 0.579) (type default) (color 197 163 255 1)) (fill (type none)))
-  (text "6" (at 79.55 40.8044 0)
-    (effects (font (size 1.1 1.1)) (justify left)))
-  (text "7" (at 71.7528 45.7544 0)
-    (effects (font (size 1.1 1.1)) (justify left)))
-  (text "8" (at 79.55 53.5044 0)
-    (effects (font (size 1.1 1.1)) (justify left)))
-  (text "1" (at 85.55 98.8044 0)
-    (effects (font (size 1.1 1.1)) (justify left)))
-  (text "2" (at 77.7528 103.754 0)
-    (effects (font (size 1.1 1.1)) (justify left)))
-  (text "3" (at 85.55 111.504 0)
-    (effects (font (size 1.1 1.1)) (justify left)))
-  (text "6" (at 235.55 65.8044 0)
-    (effects (font (size 1.1 1.1)) (justify left)))
-  (text "7" (at 227.753 70.7544 0)
-    (effects (font (size 1.1 1.1)) (justify left)))
-  (text "8" (at 235.55 78.5044 0)
-    (effects (font (size 1.1 1.1)) (justify left)))
-  (text "1" (at 235.55 118.804 0)
-    (effects (font (size 1.1 1.1)) (justify left)))
-  (text "2" (at 227.753 123.754 0)
-    (effects (font (size 1.1 1.1)) (justify left)))
-  (text "3" (at 235.55 131.504 0)
+  (text "1" (at 79.55 40.8044 0)
+    (effects (font (size 1.1 1.1)) (justify left)))
+  (text "2" (at 71.7528 45.7544 0)
+    (effects (font (size 1.1 1.1)) (justify left)))
+  (text "3" (at 79.55 53.5044 0)
+    (effects (font (size 1.1 1.1)) (justify left)))
+  (text "6" (at 85.55 98.8044 0)
+    (effects (font (size 1.1 1.1)) (justify left)))
+  (text "7" (at 77.7528 103.754 0)
+    (effects (font (size 1.1 1.1)) (justify left)))
+  (text "8" (at 85.55 111.504 0)
+    (effects (font (size 1.1 1.1)) (justify left)))
+  (text "1" (at 235.55 65.8044 0)
+    (effects (font (size 1.1 1.1)) (justify left)))
+  (text "2" (at 227.753 70.7544 0)
+    (effects (font (size 1.1 1.1)) (justify left)))
+  (text "3" (at 235.55 78.5044 0)
+    (effects (font (size 1.1 1.1)) (justify left)))
+  (text "6" (at 235.55 118.804 0)
+    (effects (font (size 1.1 1.1)) (justify left)))
+  (text "7" (at 227.753 123.754 0)
+    (effects (font (size 1.1 1.1)) (justify left)))
+  (text "8" (at 235.55 131.504 0)
     (effects (font (size 1.1 1.1)) (justify left)))
   (text "9" (at 335.55 48.1694 0)
