File: amps/6161/schematic.kicad_sch (KiCad schematic)
At the start: 80 parts, among them SW1 SPST, T1 E-3693A, T2 340-6

Commit message: Fix: the 6G5's rectifier was connected to nothing; 17 sheets shorted the mains by naming both leads alike
6G5 power supply. The sheet drew four diodes as a "silicon bridge" whose
HT_A/HT_B labels stopped 6 mm short of their wires. D1/D2's anodes sat on
the tremolo's cathode node (a tremolo wire's end touched the old diode
stub), D3/D4 ran from ground to the reservoir, and TR1's centre tap floated
under an open-pin waiver whose stated reason was the bridge itself.
A-FJ (Schematic Heaven 2153x1437, read enlarged): each HT end of TR1 runs
through a leg of three silicon diodes, every + (cathode) toward the +460 V
reservoir; the centre tap is grounded; TR1's second secondary terminal is a
bias tap feeding the 6G4's network part for part: rectifier, 8-150, 10K,
then 8-150 and a 56K bleeder at the -55 V line. Redrawn as the drawing
shows: D1-D6, TR1 with its tap pin, the centre tap to ground, the bias
network (CBIAS 25 uF -> 8 uF; RBIAS2, CBIAS2, RBIAS1 added), the waiver
deleted, and the notes, meta, netlist header and parts list no longer say
bridge. Not yet carried: the drawing's second 20-600 at the reservoir and
the standby switch (this sheet omits chassis switches by its own note);
and the tremolo ladder still runs through the transformer's corner of the
sheet, a layout clash rather than a connection, queued for its own redraw.

Mains. Two global labels with one name are one net. 16 of 24 power
transformers on the sheets carried a label named MAINS on both primary
leads, so the winding's two pins were one net: 5E4-A, 5E5-A, 5F4, 5G9,
6161, 6G2, 6G3, 6G4, AA1164, AA764, AA764-Vibro, AA964, AB763, AB763
Super, AB763 Twin, GA-40. The 6G5's loop ran from one MAINS label through
switch, fuse and winding back to the same name. No gate models the primary,
so a copy-pasted idiom did this. The second lead is now MAINS N, the AC15's
idiom; the AA1164's and AA964's second AC row, drawn under the first row's
name, is the neutral. The death and across-the-line caps stay on the le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
Connections:
- net MAINS: no longer T1.2 (PRI_2)
- new net MAINS N: T1.2 (PRI_2)
Changed lines of the file:
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@@
   (wire (pts (xy 315.81 222.234) (xy 311.81 222.234))
     (stroke (width 0) (type default)))
-  (global_label "MAINS" (shape input) (at 311.81 222.234 180)
+  (global_label "MAINS N" (shape input) (at 311.81 222.234 180)
     (effects (font (size 1.27 1.27)) (justify right)))
   (wire (pts (xy 333.59 217.154) (xy 338.59 217.154))
