File: amps/6g3/schematic.kicad_sch (KiCad schematic)
At the start: 79 parts, among them T1 125P2A, T2 125A1A

Commit message: Add: real tube pin numbers and readable valve glyphs on every schematic
Phase B of the drawing program. A factory service sheet numbers every tube
pin, because the number is what a technician puts a probe on. This corpus
printed none, and the numbers hidden in its symbols were positional
placeholders (P=1, G=2, K=3) that would have published a 6V6GT's plate as
pin 1 when it is pin 3.

1055 electrodes now carry the real number, 1027 lettered (27 are shared
filaments deduped, 1 dropped for want of clear space on the 6G2). Resolved per
instance from reference/tubes/<slug>.yaml through the same alias resolution the
layout renderer uses, so a 12AX7 section and a 6SL7 section each get their own
basing. A valve whose basing the corpus does not carry prints nothing rather
than a wrong number.

Section letters and basing units are now separate things, which cost a detour
worth recording. The RCA 12AX7-A sheet reads "Pin 1 - Plate of Unit No.2 ...
Pin 6 - Plate of Unit No.1", so unit numbering is not pin order; the 5Y3 and
GZ34 number their units in opposite pin order, so nothing positional can
express it. But the section LETTER is a designator, not a basing fact: this
corpus, like every technician, calls the first stage in signal order V1A, and
five amps' prose already did. On four amps the factory sheets put that first
stage on the other half -- the AA764's own schematic prints +200 V on pin 1 --
so those drawings now state their unit explicitly, each citing its source, and
no letter, netlist, parts list or layout comment changed. 183 layout comments
agree with the printed numbers, 0 disagree. A guard fires if two halves of one
bottle resolve to the same unit, which is exactly how this was found.

Glyphs: the cathode gains a bracket and filament hairpin so it can no longer be
confused with the plate bar, the pentode's screen sits on its own row, and a
rectifier draws as one envelope over its sections instead of two apparent
bottles. Line weights are scaled per sheet to a co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
Other:
- note added: "1"
- note added: "2"
- note added: "3"
- note added: "4"
- note added: "5"
- note added: "6"
- note added: "7"
- note added: "8"

Commit message: Fix: schematic sheet notes no longer name repository files
Thirty-seven committed sheets rendered footnotes and section notes such as
"Heaters and PT primary omitted — see netlist.cir and meta.yaml" or
"excluded from netlist.cir (notes.md)" to visitors through KiCanvas. The
prose sweeps never counted sheets. Rewritten in the site's own words — the
netlist, the sources list, the circuit story, the parts list, the board
drawing — in 59 strings across 33 draw scripts, keeping every technical
claim as it was; the three tone sheets (6G4, 6G5, 6G6-B) are under repair
elsewhere and keep theirs for now. The sweep touched only strings passed to
the sheet's note, text, caption and footnote calls, never a path or a value.

Gates: check_schematics 40/0, connectivity 0 isolated pins;
verify_schematic_nets 40 clean; only the regenerated sheets and their served
copies changed.

Co-Authored-By: Claude Fable 5.1 <noreply@anthropic.com>
Claude-Session: https://claude.ai/code/session_01KBMfdh37HmCL2iWcBiL5J1
Other:
- note added: "Heaters, PT primary/mains, pilot lamp, chassis switches and the tremolo footswitch jack are omitted here — see the netlist, the sources list and the board drawing. The drawing prints the first bottle 7025, a low-noise 12AX7."
- note added: "Its DC point alone is excluded from the netlist — a running oscillator has no static operating point (see the circuit story)"
- note removed: "Heaters, PT primary/mains, pilot lamp, chassis switches and the tremolo footswitch jack are omitted here — see netlist.cir, meta.yaml, layout.yaml. The drawing prints the first bottle 7025, a low-noise 12AX7."
- note removed: "Its DC point alone is excluded from netlist.cir — a running oscillator has no static operating point (notes.md)"
Changed lines of the file:
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@@
   (text "Bias-vary tremolo — V2B phase-shift oscillator; the Intensity control sits in the -26 V bias line itself" (at 60.7 155.738 0)
     (effects (font (size 1.5 1.5)) (justify left)))
-  (text "Its DC point alone is excluded from netlist.cir — a running oscillator has no static operating point (notes.md)" (at 60.7 160.738 0)
+  (text "Its DC point alone is excluded from the netlist — a running oscillator has no static operating point (see the circuit story)" (at 60.7 160.738 0)
     (effects (font (size 1.3 1.3)) (justify left)))
   (symbol (lib_id "cx:TRIODE") (at 134.7 196.738 0) (unit 1)
@@
   (text "Rails: B+1 +375 (reservoir · OT centre tap · tremolo oscillator) · B+2 +365 screens · B+3 +325 phase inverter · B+4 +270 preamp · bias -26 V" (at 12.7 254.516 0)
     (effects (font (size 1.2 1.2)) (justify left)))
-  (text "Heaters, PT primary/mains, pilot lamp, chassis switches and the tremolo footswitch jack are omitted here — see netlist.cir, meta.yaml, layout.yaml. The drawing prints the first bottle 7025, a low-noise 12AX7." (at 12.7 258.916 0)
+  (text "Heaters, PT primary/mains, pilot lamp, chassis switches and the tremolo footswitch jack are omitted here — see the netlist, the sources list and the board drawing. The drawing prints the first bottle 7025, a low-noise 12AX7." (at 12.7 258.916 0)
     (effects (font (size 1.2 1.2)) (justify left)))
   (sheet_instances (path "/" (page "1")))

Commit message: Fix: state the datasheet unit on 17 dual-triode sections whose sheets printed the other half's pin numbers
The sheet-vs-board gate reported these sockets as SECTION-SWAP; the
2026-09-10 source-read triage found the BOARD right on every one of them
(and both surfaces wrong on the 5G9 tremolo bottle). Each sheet had
lettered the section on the default map (A -> unit 1 -> pins 6/7/8) where
the factory drawing puts that stage on 1/2/3. The draw scripts now state
`unit=` on both halves, with the source cited beside the call, so the
printed socket numbers are the factory's:

- 5f4 V3: driver V3A -> 1/2/3, cathodyne V3B -> 6/7/8
  (crop 5f4-V3-layout-trace.png: +213 V driver plate -> pin 1, +270 V -> 6)
- 5f8a V3: 82k half V3A -> 1/2/3, 100k half V3B -> 6/7/8
  (crop 5f8a-V3-layout-trace.png: +225 -> 6, +19 -> 2, +28.5 -> 8)
- 6161 V1: channel 1 V1A -> 1/2/3 (crop 6161-V1-ch1.png prints 1/2/3);
  6161 V2: 1 MEG-grid half V2A -> 1/2/3, paraphase V2B -> 6/7/8
  (crop 6161-V2.png / 6161-V2-right.png)
- 6g3 V3: 82k half V3A -> 1/2/3 (crop 6g3-V3-layout-wires.png: +230 -> 1,
  +225 -> 6, +20 -> 7)
- aa1164 V3: recovery V3A -> 1/2/3, mixer V3B -> 6/7/8
  (crops aa1164-V3A-recovery-schem.png, aa1164-V3B-mixer-schem.png)
- aa864-bassman V1/V2: input stages 2/1/3, second stages 7/6/8; V4: the
  .1/500 pF-fed 82k half 2/1/3 (crops aa864-V1A-input.png,
  aa864-V1B-second.png, aa864-V2A-input.png, aa864-V2B-second.png,
  aa864-V4-PI.png)
- ab165 V1/V2/V4: same pattern (crops ab165-V1A-input.png,
  ab165-V1B-second.png, ab165-V2A-input.png, ab165-V2B-second.png,
  ab165-V4-PI.png)
- ab763-super V1/V2: slope-plate +270 V -> pin 1 (input stage), .047
  plate -> 6 (crops ab763-super-V1-layout-sh.png, ab763-super-V2-layout-sh.png)
- dr103 V2/V3: gain stages 6/7/8, cathode followers 1/2/3 (crops
  dr103-V2-huss.png, dr103-V3-huss.png — the Huss redraw, not a factory
  print; noted in the script)
- 5g9 V3: oscillator V3A -> 1/2/3, follower V3B -> 6/7/8 (crops
  5g9-V3-strap71-zoom.png, 5g9-V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
Parts:
- V3A: Basing_unit (none) -> 2
- V3B: Basing_unit (none) -> 1
Changed lines of the file:
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@@
     (in_bom yes) (on_board yes)
     (property "Reference" "V3A" (at 298.7 75.338 0) (effects (font (size 1.27 1.27)) (justify left)))
-    (property "Value" "12AX7" (at 298.7 77.738 0) (effects (font (size 1.27 1.27)) (justify left))))
+    (property "Value" "12AX7" (at 298.7 77.738 0) (effects (font (size 1.27 1.27)) (justify left)))
+    (property "Basing_unit" "2" (at 298.7 80.138 0) (effects (font (size 1.27 1.27)) hide)))
   (symbol (lib_id "cx:TRIODE") (at 292.7 117.738 0) (unit 1)
     (in_bom yes) (on_board yes)
     (property "Reference" "V3B" (at 298.7 111.338 0) (effects (font (size 1.27 1.27)) (justify left)))
-    (property "Value" "12AX7" (at 298.7 113.738 0) (effects (font (size 1.27 1.27)) (justify left))))
+    (property "Value" "12AX7" (at 298.7 113.738 0) (effects (font (size 1.27 1.27)) (justify left)))
+    (property "Basing_unit" "1" (at 298.7 116.138 0) (effects (font (size 1.27 1.27)) hide)))
   (wire (pts (xy 292.7 74.118) (xy 292.7 70.638))
     (stroke (width 0) (type default)))
@@
   (text "8" (at 185.55 70.088 0)
     (effects (font (size 1.1 1.1)) (justify left)))
-  (text "6" (at 293.55 75.388 0)
-    (effects (font (size 1.1 1.1)) (justify left)))
-  (text "7" (at 285.753 80.338 0)
-    (effects (font (size 1.1 1.1)) (justify left)))
-  (text "8" (at 293.55 88.088 0)
-    (effects (font (size 1.1 1.1)) (justify left)))
-  (text "1" (at 293.55 111.388 0)
-    (effects (font (size 1.1 1.1)) (justify left)))
-  (text "2" (at 285.753 116.338 0)
-    (effects (font (size 1.1 1.1)) (justify left)))
-  (text "3" (at 293.55 124.088 0)
+  (text "1" (at 293.55 75.388 0)
+    (effects (font (size 1.1 1.1)) (justify left)))
+  (text "2" (at 285.753 80.338 0)
+    (effects (font (size 1.1 1.1)) (justify left)))
+  (text "3" (at 293.55 88.088 0)
+    (effects (font (size 1.1 1.1)) (justify left)))
+  (text "6" (at 293.55 111.388 0)
+    (effects (font (size 1.1 1.1)) (justify left)))
+  (text "7" (at 285.753 116.338 0)
+    (effects (font (size 1.1 1.1)) (justify left)))
+  (text "8" (at 293.55 124.088 0)
     (effects (font (size 1.1 1.1)) (justify left)))
   (text "3" (at 355.55 54.753 0)
