File: amps/aa864-bassman/schematic.kicad_sch (KiCad schematic)
At the start: 102 parts, among them T1 125P7D, T2 125C1A, T3 125A13A

Commit message: Fix: schematic wiring on m1987, aa864-bassman, ac30, m1959, ga40, aa1164, aa964
- 58 open pins closed: leads that stopped short of their flags, pins
  missed by 0.01-0.11 mm, snubbers and bright caps with no leads
- two shorts the isolated-pin check cannot see: aa864-bassman V6 anode
  lead ran through its grounded cathode (plate rail to chassis) and its V5
  coupler drop shorted RGL1; m1987 RB1/RB2 stood on the wire they bridge
- 14 dated waivers: m1959 C29-C31 (factory sheet prints them unconnected),
  ga40 V2/V3/VR3.3 (net_map excluded tubes, free rheostat lug)
- all seven sheets pass connectivity and verify_schematic_nets

Co-Authored-By: Claude Fable 5.1 <noreply@anthropic.com>
Claude-Session: https://claude.ai/code/session_01KBMfdh37HmCL2iWcBiL5J1
Parts:
- removed D3, D6: Si, symbol cx:DIODE_SS
- removed FUSE: 2A slo-blo, symbol cx:FUSE
- removed RBL1, RBL2: 220k 1W, symbol cx:R
- removed RD1: 1k 1W, symbol cx:R
- removed RD2: 4.7k 1W, symbol cx:R
- removed V5, V6: 6L6GC, symbol cx:PENTODE
- added C10, C11: 70u 350V, symbol cx:C
- added C12, C13: 20u 525V, symbol cx:C
- added D1, D4: Si, symbol cx:DIODE_SS
- added RGS1, RGS2: 1.5k, symbol cx:R
- added T1: 125P7D, symbol cx:PT
- FUSE: renamed from T1; value 125P7D -> 2A slo-blo; symbol cx:PT -> cx:FUSE
- RBL1: renamed from C10; value 70u 350V -> 220k 1W; symbol cx:C -> cx:R
- RBL2: renamed from C11; value 70u 350V -> 220k 1W; symbol cx:C -> cx:R
- RD1: renamed from C12; value 20u 525V -> 1k 1W; symbol cx:C -> cx:R
- RD2: renamed from C13; value 20u 525V -> 4.7k 1W; symbol cx:C -> cx:R
- V5: renamed from RGS1; value 1.5k -> 6L6GC; symbol cx:R -> cx:PENTODE
- V6: renamed from RGS2; value 1.5k -> 6L6GC; symbol cx:R -> cx:PENTODE
- renumbered D1 to D3, D4 to D6
Connections:
- net -44V: no longer C1.2, RGL1.2, V5.1
- net AC LINE: now also FUSE.1, SWGND.1, T1.2 (PRI_2)
- net B+PI: now also RD1.2, C13.1
- net B+PRE: now also RD2.2
- net B+SCR: now also C12.1
- net BASS 1: now also R2b.1
- net BASS 2: now also R1b.1
- net GND: now also V5.4 (K), V6.4 (K), C11.2, C12.2, C13.2, T1.4 (HT_CT); no longer FUSE.4 (HT_CT), RD1.2, RD2.2, T3.3 (PRI_B)
- net HT-A: now also RBIAS.1, D1.1 (A), T1.3 (HT_A); no longer D3.1 (A), FUSE.3 (HT_A)
- net NORM 1: now also R2n.1
- net NORM 2: now also R1n.1
- net PIMIX: now also CPI.1
- net SPKR: now also RNFB.1
- net at RBL1.1, SWSTBY.1: now also D3.2 (K), D6.2 (K), C10.1
- net at RBL1.2, RBL2.1: now also C10.2, C11.1
- net at V5.2 (G1): now also RGS1.2
- net at RS1.1: now also V5.3 (G2)
- net at D2.1 (A): now also D1.2 (K); no longer D3.2 (K)
- net at SWAC.1: now also FUSE.2
- net at SWAC.2: now also T1.1 (PRI_1); no longer FUSE.1 (PRI_1)
- net at D6.1 (A): no longer FUSE.5 (HT_B)
- net at D5.1 (A): now also D4.2 (K); no longer D6.2 (K)
- net at C2.2, RGL2.1: now also RGS2.1; no longer V6.1
- net at T3.1 (PRI_A): now also V5.1 (P)
- net at V6.2 (G1): now also RGS2.2
- net at RS2.1: now also V6.3 (G2)
- new net: C1.2, RGL1.2, RGS1.1
- new net: D4.1 (A), T1.5 (HT_B)
- new net: T3.3 (PRI_B), V6.1 (P)
Other:
- moved on the sheet: D3, D6
Changed lines of the file:
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@@
     (property "Reference" "R1b" (at 29.2724 33.009 270) (effects (font (size 1.27 1.27)) (justify left)))
     (property "Value" "68k" (at 29.2724 35.409 270) (effects (font (size 1.27 1.27)) (justify left))))
-  (wire (pts (xy 26.4724 39.009) (xy 28.6624 39.009))
+  (wire (pts (xy 22.4724 39.009) (xy 28.6624 39.009))
     (stroke (width 0) (type default)))
   (wire (pts (xy 36.2824 39.009) (xy 50.4724 39.009))
@@
     (property "Reference" "R2b" (at 29.2724 44.009 270) (effects (font (size 1.27 1.27)) (justify left)))
     (property "Value" "68k" (at 29.2724 46.409 270) (effects (font (size 1.27 1.27)) (justify left))))
-  (wire (pts (xy 26.4724 50.009) (xy 28.6624 50.009))
+  (wire (pts (xy 22.4724 50.009) (xy 28.6624 50.009))
     (stroke (width 0) (type default)))
   (wire (pts (xy 36.2824 50.009) (xy 50.4724 50.009))
@@
     (property "Reference" "R1n" (at 29.2724 151.009 270) (effects (font (size 1.27 1.27)) (justify left)))
     (property "Value" "68k" (at 29.2724 153.409 270) (effects (font (size 1.27 1.27)) (justify left))))
-  (wire (pts (xy 26.4724 157.009) (xy 28.6624 157.009))
+  (wire (pts (xy 22.4724 157.009) (xy 28.6624 157.009))
     (stroke (width 0) (type default)))
   (wire (pts (xy 36.2824 157.009) (xy 50.4724 157.009))
@@
     (property "Reference" "R2n" (at 29.2724 162.009 270) (effects (font (size 1.27 1.27)) (justify left)))
     (property "Value" "68k" (at 29.2724 164.409 270) (effects (font (size 1.27 1.27)) (justify left))))
-  (wire (pts (xy 26.4724 168.009) (xy 28.6624 168.009))
+  (wire (pts (xy 22.4724 168.009) (xy 28.6624 168.009))
     (stroke (width 0) (type default)))
   (wire (pts (xy 36.2824 168.009) (xy 50.4724 168.009))
@@
     (property "Reference" "CPI" (at 255.272 56.309 270) (effects (font (size 1.27 1.27)) (justify left)))
     (property "Value" "500p" (at 255.272 58.709 270) (effects (font (size 1.27 1.27)) (justify left))))
-  (wire (pts (xy 240.472 62.509) (xy 254.662 62.509))
+  (wire (pts (xy 236.472 62.509) (xy 254.662 62.509))
     (stroke (width 0) (type default)))
   (wire (pts (xy 262.282 62.509) (xy 268.852 62.509))
@@
     (property "Reference" "RNFB" (at 195.272 66.509 270) (effects (font (size 1.27 1.27)) (justify left)))
     (property "Value" "820" (at 195.272 68.909 270) (effects (font (size 1.27 1.27)) (justify left))))
-  (wire (pts (xy 188.472 72.509) (xy 194.662 72.509))
+  (wire (pts (xy 184.472 72.509) (xy 194.662 72.509))
     (stroke (width 0) (type default)))
   (wire (pts (xy 202.282 72.509) (xy 214.472 72.509))
@@
   (wire (pts (xy 296.282 51.409) (xy 306.472 51.409))
     (stroke (width 0) (type default)))
-  (wire (pts (xy 306.472 51.409) (xy 306.472 44.669))
-    (stroke (width 0) (type default)))
-  (wire (pts (xy 306.472 44.669) (xy 306.472 42.129))
-    (stroke (width 0) (type default)))
-  (wire (pts (xy 306.472 42.129) (xy 306.472 34.509))
+  (wire (pts (xy 306.472 51.409) (xy 306.472 34.509))
     (stroke (width 0) (type default)))
   (wire (pts (xy 276.472 91.409) (xy 286.472 91.409))
@@
     (effects (font (size 1.4 1.4)) (justify left)))
   (junction (at 306.472 34.509) (diameter 0) (color 0 0 0 0))
-  (symbol (lib_id "cx:R") (at 306.472 38.319 0) (unit 1)
-    (in_bom yes) (on_board yes)
-    (property "Reference" "RGL1" (at 295.472 35.119 0) (effects (font (size 1.27 1.27)) (justify left)))
-    (property "Value" "220k 5%" (at 295.472 37.519 0) (effects (font (size 1.27 1.27)) (justify left))))
-  (wire (pts (xy 306.472 42.129) (xy 306.472 44.669))
-    (stroke (width 0) (type default)))
-  (global_label "-44V" (shape input) (at 306.472 44.669 270)
-    (effects (font (size 1.27 1.27)) (justify right)))
+  (symbol (lib_id "cx:R") (at 306.472 30.699 0) (unit 1)
+    (in_bom yes) (on_board yes)
+    (property "Reference" "RGL1" (at 295.472 27.499 0) (effects (font (size 1.27 1.27)) (justify left)))
+    (property "Value" "220k 5%" (at 295.472 29.899 0) (effects (font (size 1.27 1.27)) (justify left))))
+  (wire (pts (xy 306.472 26.889) (xy 306.472 24.349))
+    (stroke (width 0) (type default)))
+  (global_label "-44V" (shape input) (at 306.472 24.349 90)
+    (effects (font (size 1.27 1.27)) (justify left)))
   (symbol (lib_id "cx:R") (at 316.472 34.509 90) (unit 1)
     (in_bom yes) (on_board yes)
@@
   (wire (pts (xy 366.472 79.429) (xy 373.582 79.429))
     (stroke (width 0) (type default)))
-  (wire (pts (xy 334.472 126.254) (xy 334.472 141.494))
-    (stroke (width 0) (type default)))
-  (wire (pts (xy 334.472 141.494) (xy 334.472 150.509))
-    (stroke (width 0) (type default)))
-  (wire (pts (xy 334.472 150.509) (xy 362.472 150.509))
-    (stroke (width 0) (type default)))
-  (wire (pts (xy 362.472 150.509) (xy 362.472 89.589))
+  (wire (pts (xy 334.472 126.254) (xy 334.472 120.509))
+    (stroke (width 0) (type default)))
+  (wire (pts (xy 334.472 120.509) (xy 362.472 120.509))
+    (stroke (width 0) (type default)))
+  (wire (pts (xy 362.472 120.509) (xy 362.472 89.589))
     (stroke (width 0) (type default)))
   (wire (pts (xy 362.472 89.589) (xy 373.582 89.589))
@@
   (global_label "AC LINE" (shape input) (at 20.4724 212.429 180)
     (effects (font (size 1.27 1.27)) (justify right)))
-  (wire (pts (xy 24.4724 212.429) (xy 26.3924 212.429))
+  (wire (pts (xy 20.4724 212.429) (xy 26.3924 212.429))
     (stroke (width 0) (type default)))
   (symbol (lib_id "cx:FUSE") (at 31.4724 212.429 0) (unit 1)
@@
   (global_label "AC LINE" (shape input) (at 20.4724 222.589 180)
     (effects (font (size 1.27 1.27)) (justify right)))
-  (wire (pts (xy 24.4724 222.589) (xy 51.5824 222.589))
+  (wire (pts (xy 20.4724 222.589) (xy 51.5824 222.589))
     (stroke (width 0) (type default)))
   (wire (pts (xy 69.3624 217.509) (xy 73.4724 217.509))
@@
   (global_label "HT-A" (shape input) (at 292.472 232.509 180)
     (effects (font (size 1.27 1.27)) (justify right)))
-  (wire (pts (xy 296.472 232.509) (xy 301.662 232.509))
+  (wire (pts (xy 292.472 232.509) (xy 301.662 232.509))
     (stroke (width 0) (type default)))
   (symbol (lib_id "cx:R") (at 305.472 232.509 90) (unit 1)
@@
   (global_label "AC LINE" (shape input) (at 20.4724 254.509 180)
     (effects (font (size 1.27 1.27)) (justify right)))
-  (wire (pts (xy 24.4724 254.509) (xy 26.3924 254.509))
+  (wire (pts (xy 20.4724 254.509) (xy 26.3924 254.509))
     (stroke (width 0) (type default)))
   (symbol (lib_id "cx:SWITCH") (at 31.4724 254.509 0) (unit 1)

Commit message: Add: real tube pin numbers and readable valve glyphs on every schematic
Phase B of the drawing program. A factory service sheet numbers every tube
pin, because the number is what a technician puts a probe on. This corpus
printed none, and the numbers hidden in its symbols were positional
placeholders (P=1, G=2, K=3) that would have published a 6V6GT's plate as
pin 1 when it is pin 3.

1055 electrodes now carry the real number, 1027 lettered (27 are shared
filaments deduped, 1 dropped for want of clear space on the 6G2). Resolved per
instance from reference/tubes/<slug>.yaml through the same alias resolution the
layout renderer uses, so a 12AX7 section and a 6SL7 section each get their own
basing. A valve whose basing the corpus does not carry prints nothing rather
than a wrong number.

Section letters and basing units are now separate things, which cost a detour
worth recording. The RCA 12AX7-A sheet reads "Pin 1 - Plate of Unit No.2 ...
Pin 6 - Plate of Unit No.1", so unit numbering is not pin order; the 5Y3 and
GZ34 number their units in opposite pin order, so nothing positional can
express it. But the section LETTER is a designator, not a basing fact: this
corpus, like every technician, calls the first stage in signal order V1A, and
five amps' prose already did. On four amps the factory sheets put that first
stage on the other half -- the AA764's own schematic prints +200 V on pin 1 --
so those drawings now state their unit explicitly, each citing its source, and
no letter, netlist, parts list or layout comment changed. 183 layout comments
agree with the printed numbers, 0 disagree. A guard fires if two halves of one
bottle resolve to the same unit, which is exactly how this was found.

Glyphs: the cathode gains a bracket and filament hairpin so it can no longer be
confused with the plate bar, the pentode's screen sits on its own row, and a
rectifier draws as one envelope over its sections instead of two apparent
bottles. Line weights are scaled per sheet to a co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
Other:
- note added: "1"
- note added: "2"
- note added: "3"
- note added: "4"
- note added: "5"
- note added: "6"
- note added: "7"
- note added: "8"

Commit message: Fix: schematic sheet notes no longer name repository files
Thirty-seven committed sheets rendered footnotes and section notes such as
"Heaters and PT primary omitted — see netlist.cir and meta.yaml" or
"excluded from netlist.cir (notes.md)" to visitors through KiCanvas. The
prose sweeps never counted sheets. Rewritten in the site's own words — the
netlist, the sources list, the circuit story, the parts list, the board
drawing — in 59 strings across 33 draw scripts, keeping every technical
claim as it was; the three tone sheets (6G4, 6G5, 6G6-B) are under repair
elsewhere and keep theirs for now. The sweep touched only strings passed to
the sheet's note, text, caption and footnote calls, never a path or a value.

Gates: check_schematics 40/0, connectivity 0 isolated pins;
verify_schematic_nets 40 clean; only the regenerated sheets and their served
copies changed.

Co-Authored-By: Claude Fable 5.1 <noreply@anthropic.com>
Claude-Session: https://claude.ai/code/session_01KBMfdh37HmCL2iWcBiL5J1
Other:
- note added: "Heaters, pilot lamp and the PT's 6.3 V winding omitted here — see the netlist, the sources list and the board drawing. Rails: B+PL +422 (OT centre tap) · B+SCR +420 screens · B+PI +410 · B+PRE +380 preamp · bias −44 V"
- note removed: "Heaters, pilot lamp and the PT's 6.3 V winding omitted here — see netlist.cir, meta.yaml, layout.yaml. Rails: B+PL +422 (OT centre tap) · B+SCR +420 screens · B+PI +410 · B+PRE +380 preamp · bias −44 V"
Changed lines of the file:
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@@
   (text "8" (at 335.322 140.224 0)
     (effects (font (size 1.1 1.1)) (justify left)))
-  (text "Heaters, pilot lamp and the PT's 6.3 V winding omitted here — see netlist.cir, meta.yaml, layout.yaml. Rails: B+PL +422 (OT centre tap) · B+SCR +420 screens · B+PI +410 · B+PRE +380 preamp · bias −44 V" (at 12.7 265.667 0)
+  (text "Heaters, pilot lamp and the PT's 6.3 V winding omitted here — see the netlist, the sources list and the board drawing. Rails: B+PL +422 (OT centre tap) · B+SCR +420 screens · B+PI +410 · B+PRE +380 preamp · bias −44 V" (at 12.7 265.667 0)
     (effects (font (size 1.2 1.2)) (justify left)))
   (sheet_instances (path "/" (page "1")))

Commit message: Fix: state the datasheet unit on 17 dual-triode sections whose sheets printed the other half's pin numbers
The sheet-vs-board gate reported these sockets as SECTION-SWAP; the
2026-09-10 source-read triage found the BOARD right on every one of them
(and both surfaces wrong on the 5G9 tremolo bottle). Each sheet had
lettered the section on the default map (A -> unit 1 -> pins 6/7/8) where
the factory drawing puts that stage on 1/2/3. The draw scripts now state
`unit=` on both halves, with the source cited beside the call, so the
printed socket numbers are the factory's:

- 5f4 V3: driver V3A -> 1/2/3, cathodyne V3B -> 6/7/8
  (crop 5f4-V3-layout-trace.png: +213 V driver plate -> pin 1, +270 V -> 6)
- 5f8a V3: 82k half V3A -> 1/2/3, 100k half V3B -> 6/7/8
  (crop 5f8a-V3-layout-trace.png: +225 -> 6, +19 -> 2, +28.5 -> 8)
- 6161 V1: channel 1 V1A -> 1/2/3 (crop 6161-V1-ch1.png prints 1/2/3);
  6161 V2: 1 MEG-grid half V2A -> 1/2/3, paraphase V2B -> 6/7/8
  (crop 6161-V2.png / 6161-V2-right.png)
- 6g3 V3: 82k half V3A -> 1/2/3 (crop 6g3-V3-layout-wires.png: +230 -> 1,
  +225 -> 6, +20 -> 7)
- aa1164 V3: recovery V3A -> 1/2/3, mixer V3B -> 6/7/8
  (crops aa1164-V3A-recovery-schem.png, aa1164-V3B-mixer-schem.png)
- aa864-bassman V1/V2: input stages 2/1/3, second stages 7/6/8; V4: the
  .1/500 pF-fed 82k half 2/1/3 (crops aa864-V1A-input.png,
  aa864-V1B-second.png, aa864-V2A-input.png, aa864-V2B-second.png,
  aa864-V4-PI.png)
- ab165 V1/V2/V4: same pattern (crops ab165-V1A-input.png,
  ab165-V1B-second.png, ab165-V2A-input.png, ab165-V2B-second.png,
  ab165-V4-PI.png)
- ab763-super V1/V2: slope-plate +270 V -> pin 1 (input stage), .047
  plate -> 6 (crops ab763-super-V1-layout-sh.png, ab763-super-V2-layout-sh.png)
- dr103 V2/V3: gain stages 6/7/8, cathode followers 1/2/3 (crops
  dr103-V2-huss.png, dr103-V3-huss.png — the Huss redraw, not a factory
  print; noted in the script)
- 5g9 V3: oscillator V3A -> 1/2/3, follower V3B -> 6/7/8 (crops
  5g9-V3-strap71-zoom.png, 5g9-V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
Parts:
- V1A, V2A, V4A: Basing_unit (none) -> 2
- V1B, V2B, V4B: Basing_unit (none) -> 1
Changed lines of the file:
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@@
     (in_bom yes) (on_board yes)
     (property "Reference" "V1A" (at 68.4724 38.109 0) (effects (font (size 1.27 1.27)) (justify left)))
-    (property "Value" "7025" (at 68.4724 40.509 0) (effects (font (size 1.27 1.27)) (justify left))))
+    (property "Value" "7025" (at 68.4724 40.509 0) (effects (font (size 1.27 1.27)) (justify left)))
+    (property "Basing_unit" "2" (at 68.4724 42.909 0) (effects (font (size 1.27 1.27)) hide)))
   (wire (pts (xy 50.4724 44.509) (xy 54.8524 44.509))
     (stroke (width 0) (type default)))
@@
     (in_bom yes) (on_board yes)
     (property "Reference" "V1B" (at 174.472 38.109 0) (effects (font (size 1.27 1.27)) (justify left)))
-    (property "Value" "7025" (at 174.472 40.509 0) (effects (font (size 1.27 1.27)) (justify left))))
+    (property "Value" "7025" (at 174.472 40.509 0) (effects (font (size 1.27 1.27)) (justify left)))
+    (property "Basing_unit" "1" (at 174.472 42.909 0) (effects (font (size 1.27 1.27)) hide)))
   (wire (pts (xy 145.472 44.509) (xy 160.852 44.509))
     (stroke (width 0) (type default)))
@@
     (in_bom yes) (on_board yes)
     (property "Reference" "V2A" (at 68.4724 156.109 0) (effects (font (size 1.27 1.27)) (justify left)))
-    (property "Value" "7025" (at 68.4724 158.509 0) (effects (font (size 1.27 1.27)) (justify left))))
+    (property "Value" "7025" (at 68.4724 158.509 0) (effects (font (size 1.27 1.27)) (justify left)))
+    (property "Basing_unit" "2" (at 68.4724 160.909 0) (effects (font (size 1.27 1.27)) hide)))
   (wire (pts (xy 50.4724 162.509) (xy 54.8524 162.509))
     (stroke (width 0) (type default)))
@@
     (in_bom yes) (on_board yes)
     (property "Reference" "V2B" (at 174.472 156.109 0) (effects (font (size 1.27 1.27)) (justify left)))
-    (property "Value" "7025" (at 174.472 158.509 0) (effects (font (size 1.27 1.27)) (justify left))))
+    (property "Value" "7025" (at 174.472 158.509 0) (effects (font (size 1.27 1.27)) (justify left)))
+    (property "Basing_unit" "1" (at 174.472 160.909 0) (effects (font (size 1.27 1.27)) hide)))
   (wire (pts (xy 145.472 162.509) (xy 160.852 162.509))
     (stroke (width 0) (type default)))
@@
     (in_bom yes) (on_board yes)
     (property "Reference" "V4A" (at 282.472 56.109 0) (effects (font (size 1.27 1.27)) (justify left)))
-    (property "Value" "12AT7" (at 282.472 58.509 0) (effects (font (size 1.27 1.27)) (justify left))))
+    (property "Value" "12AT7" (at 282.472 58.509 0) (effects (font (size 1.27 1.27)) (justify left)))
+    (property "Basing_unit" "2" (at 282.472 60.909 0) (effects (font (size 1.27 1.27)) hide)))
   (symbol (lib_id "cx:TRIODE") (at 276.472 102.509 0) (unit 1)
     (in_bom yes) (on_board yes)
     (property "Reference" "V4B" (at 282.472 96.109 0) (effects (font (size 1.27 1.27)) (justify left)))
-    (property "Value" "12AT7" (at 282.472 98.509 0) (effects (font (size 1.27 1.27)) (justify left))))
+    (property "Value" "12AT7" (at 282.472 98.509 0) (effects (font (size 1.27 1.27)) (justify left)))
+    (property "Basing_unit" "1" (at 282.472 100.909 0) (effects (font (size 1.27 1.27)) hide)))
   (wire (pts (xy 276.472 54.889) (xy 276.472 51.409))
     (stroke (width 0) (type default)))
@@
   (global_label "GND" (shape input) (at 52.4724 254.509 270)
     (effects (font (size 1.27 1.27)) (justify right)))
-  (text "6" (at 63.3224 38.159 0)
-    (effects (font (size 1.1 1.1)) (justify left)))
-  (text "7" (at 55.5252 43.109 0)
-    (effects (font (size 1.1 1.1)) (justify left)))
-  (text "8" (at 63.3224 50.859 0)
-    (effects (font (size 1.1 1.1)) (justify left)))
-  (text "1" (at 169.322 38.159 0)
-    (effects (font (size 1.1 1.1)) (justify left)))
-  (text "2" (at 161.525 43.109 0)
-    (effects (font (size 1.1 1.1)) (justify left)))
-  (text "3" (at 169.322 50.859 0)
+  (text "1" (at 63.3224 38.159 0)
+    (effects (font (size 1.1 1.1)) (justify left)))
+  (text "2" (at 55.5252 43.109 0)
+    (effects (font (size 1.1 1.1)) (justify left)))
+  (text "3" (at 63.3224 50.859 0)
+    (effects (font (size 1.1 1.1)) (justify left)))
+  (text "6" (at 169.322 38.159 0)
+    (effects (font (size 1.1 1.1)) (justify left)))
+  (text "7" (at 161.525 43.109 0)
+    (effects (font (size 1.1 1.1)) (justify left)))
+  (text "8" (at 169.322 50.859 0)
     (effects (font (size 1.1 1.1)) (justify left)))
   (text "1" (at 223.322 38.159 0)
@@
   (text "3" (at 223.322 50.859 0)
     (effects (font (size 1.1 1.1)) (justify left)))
-  (text "6" (at 63.3224 156.159 0)
-    (effects (font (size 1.1 1.1)) (justify left)))
-  (text "7" (at 55.5252 161.109 0)
-    (effects (font (size 1.1 1.1)) (justify left)))
-  (text "8" (at 63.3224 168.859 0)
-    (effects (font (size 1.1 1.1)) (justify left)))
-  (text "1" (at 169.322 156.159 0)
-    (effects (font (size 1.1 1.1)) (justify left)))
-  (text "2" (at 161.525 161.109 0)
-    (effects (font (size 1.1 1.1)) (justify left)))
-  (text "3" (at 169.322 168.859 0)
-    (effects (font (size 1.1 1.1)) (justify left)))
-  (text "6" (at 277.322 56.159 0)
-    (effects (font (size 1.1 1.1)) (justify left)))
-  (text "7" (at 269.525 61.109 0)
-    (effects (font (size 1.1 1.1)) (justify left)))
-  (text "8" (at 277.322 68.859 0)
-    (effects (font (size 1.1 1.1)) (justify left)))
-  (text "1" (at 277.322 96.159 0)
-    (effects (font (size 1.1 1.1)) (justify left)))
-  (text "2" (at 269.525 101.109 0)
-    (effects (font (size 1.1 1.1)) (justify left)))
-  (text "3" (at 277.322 108.859 0)
+  (text "1" (at 63.3224 156.159 0)
+    (effects (font (size 1.1 1.1)) (justify left)))
+  (text "2" (at 55.5252 161.109 0)
+    (effects (font (size 1.1 1.1)) (justify left)))
+  (text "3" (at 63.3224 168.859 0)
+    (effects (font (size 1.1 1.1)) (justify left)))
+  (text "6" (at 169.322 156.159 0)
+    (effects (font (size 1.1 1.1)) (justify left)))
+  (text "7" (at 161.525 161.109 0)
+    (effects (font (size 1.1 1.1)) (justify left)))
+  (text "8" (at 169.322 168.859 0)
+    (effects (font (size 1.1 1.1)) (justify left)))
+  (text "1" (at 277.322 56.159 0)
+    (effects (font (size 1.1 1.1)) (justify left)))
+  (text "2" (at 269.525 61.109 0)
+    (effects (font (size 1.1 1.1)) (justify left)))
+  (text "3" (at 277.322 68.859 0)
+    (effects (font (size 1.1 1.1)) (justify left)))
+  (text "6" (at 277.322 96.159 0)
+    (effects (font (size 1.1 1.1)) (justify left)))
+  (text "7" (at 269.525 101.109 0)
+    (effects (font (size 1.1 1.1)) (justify left)))
+  (text "8" (at 277.322 108.859 0)
     (effects (font (size 1.1 1.1)) (justify left)))
   (text "3" (at 335.322 27.524 0)
