File: amps/aa764/schematic.kicad_sch (KiCad schematic)
At the start: 36 parts, among them T1 125P1B, T2 125A35A

Commit message: Add: real tube pin numbers and readable valve glyphs on every schematic
Phase B of the drawing program. A factory service sheet numbers every tube
pin, because the number is what a technician puts a probe on. This corpus
printed none, and the numbers hidden in its symbols were positional
placeholders (P=1, G=2, K=3) that would have published a 6V6GT's plate as
pin 1 when it is pin 3.

1055 electrodes now carry the real number, 1027 lettered (27 are shared
filaments deduped, 1 dropped for want of clear space on the 6G2). Resolved per
instance from reference/tubes/<slug>.yaml through the same alias resolution the
layout renderer uses, so a 12AX7 section and a 6SL7 section each get their own
basing. A valve whose basing the corpus does not carry prints nothing rather
than a wrong number.

Section letters and basing units are now separate things, which cost a detour
worth recording. The RCA 12AX7-A sheet reads "Pin 1 - Plate of Unit No.2 ...
Pin 6 - Plate of Unit No.1", so unit numbering is not pin order; the 5Y3 and
GZ34 number their units in opposite pin order, so nothing positional can
express it. But the section LETTER is a designator, not a basing fact: this
corpus, like every technician, calls the first stage in signal order V1A, and
five amps' prose already did. On four amps the factory sheets put that first
stage on the other half -- the AA764's own schematic prints +200 V on pin 1 --
so those drawings now state their unit explicitly, each citing its source, and
no letter, netlist, parts list or layout comment changed. 183 layout comments
agree with the printed numbers, 0 disagree. A guard fires if two halves of one
bottle resolve to the same unit, which is exactly how this was found.

Glyphs: the cathode gains a bracket and filament hairpin so it can no longer be
confused with the plate bar, the pentode's screen sits on its own row, and a
rectifier draws as one envelope over its sections instead of two apparent
bottles. Line weights are scaled per sheet to a co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
Other:
- note added: "1"
- note added: "2"
- note added: "2,8"
- note added: "3"
- note added: "4"
- note added: "5"
- note added: "6"
- note added: "7"
- note added: "8"
Changed lines of the file:
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@@
   (wire (pts (xy 43.8816 38.278) (xy 43.8816 42.278))
     (stroke (width 0) (type default)))
-  (junction (at 43.8816 38.278) (diameter 0) (color 0 0 0 0))
+  (junction (at 43.8816 38.278) (diameter 1) (color 0 0 0 0))
   (symbol (lib_id "cx:R") (at 43.8816 46.088 0) (unit 1)
     (in_bom yes) (on_board yes)
@@
   (global_label "GND" (shape input) (at 55.8816 54.898 270)
     (effects (font (size 1.27 1.27)) (justify right)))
-  (junction (at 55.8816 27.178) (diameter 0) (color 0 0 0 0))
+  (junction (at 55.8816 27.178) (diameter 1) (color 0 0 0 0))
   (wire (pts (xy 55.8816 27.178) (xy 67.8816 27.178))
     (stroke (width 0) (type default)))
@@
   (wire (pts (xy 67.8816 27.178) (xy 67.8816 32.278))
     (stroke (width 0) (type default)))
-  (junction (at 67.8816 27.178) (diameter 0) (color 0 0 0 0))
+  (junction (at 67.8816 27.178) (diameter 1) (color 0 0 0 0))
   (symbol (lib_id "cx:C") (at 79.8816 24.658 90) (unit 1)
     (in_bom yes) (on_board yes)
@@
   (wire (pts (xy 77.6916 32.278) (xy 81.8816 32.278))
     (stroke (width 0) (type default)))
-  (junction (at 81.8816 32.278) (diameter 0) (color 0 0 0 0))
+  (junction (at 81.8816 32.278) (diameter 1) (color 0 0 0 0))
   (symbol (lib_id "cx:C") (at 88.8816 32.278 90) (unit 1)
     (in_bom yes) (on_board yes)
@@
     (property "Reference" "VR3" (at 100.282 32.888 0) (effects (font (size 1.27 1.27)) (justify left)))
     (property "Value" "250k bass" (at 100.282 35.288 0) (effects (font (size 1.27 1.27)) (justify left))))
-  (junction (at 95.8816 32.278) (diameter 0) (color 0 0 0 0))
+  (junction (at 95.8816 32.278) (diameter 1) (color 0 0 0 0))
   (wire (pts (xy 100.962 36.088) (xy 103.882 36.088))
     (stroke (width 0) (type default)))
@@
   (wire (pts (xy 133.882 63.898) (xy 141.882 63.898))
     (stroke (width 0) (type default)))
-  (junction (at 133.882 63.898) (diameter 0) (color 0 0 0 0))
+  (junction (at 133.882 63.898) (diameter 1) (color 0 0 0 0))
   (symbol (lib_id "cx:R") (at 133.882 67.708 0) (unit 1)
     (in_bom yes) (on_board yes)
@@
   (global_label "SPKR" (shape input) (at 121.882 71.518 270)
     (effects (font (size 1.27 1.27)) (justify right)))
-  (junction (at 133.882 35.178) (diameter 0) (color 0 0 0 0))
+  (junction (at 133.882 35.178) (diameter 1) (color 0 0 0 0))
   (wire (pts (xy 133.882 35.178) (xy 141.882 35.178))
     (stroke (width 0) (type default)))
@@
   (wire (pts (xy 159.882 35.178) (xy 159.882 46.278))
     (stroke (width 0) (type default)))
-  (junction (at 159.882 46.278) (diameter 0) (color 0 0 0 0))
+  (junction (at 159.882 46.278) (diameter 1) (color 0 0 0 0))
   (symbol (lib_id "cx:R") (at 159.882 50.088 0) (unit 1)
     (in_bom yes) (on_board yes)
@@
   (symbol (lib_id "cx:DIODE_TUBE") (at 79.8816 124.398 0) (unit 1)
     (in_bom yes) (on_board yes)
-    (property "Reference" "V3A" (at 68.1574 124.678 0) (effects (font (size 1.27 1.27)) (justify left)))
-    (property "Value" "5Y3GT" (at 68.1574 127.078 0) (effects (font (size 1.27 1.27)) (justify left))))
+    (property "Reference" "V3A" (at 77.0876 131.278 0) (effects (font (size 1.27 1.27)) (justify left)))
+    (property "Value" "5Y3GT" (at 77.0876 133.678 0) (effects (font (size 1.27 1.27)) (justify left))))
   (global_label "HT_B" (shape input) (at 91.8816 114.278 90)
     (effects (font (size 1.27 1.27)) (justify left)))
@@
   (wire (pts (xy 97.8816 134.278) (xy 105.882 134.278))
     (stroke (width 0) (type default)))
-  (junction (at 91.8816 134.278) (diameter 0) (color 0 0 0 0))
-  (junction (at 97.8816 134.278) (diameter 0) (color 0 0 0 0))
+  (junction (at 91.8816 134.278) (diameter 1) (color 0 0 0 0))
+  (junction (at 97.8816 134.278) (diameter 1) (color 0 0 0 0))
   (symbol (lib_id "cx:C") (at 97.8816 138.088 0) (unit 1)
     (in_bom yes) (on_board yes)
@@
   (wire (pts (xy 125.882 134.278) (xy 127.882 134.278))
     (stroke (width 0) (type default)))
-  (junction (at 121.882 134.278) (diameter 0) (color 0 0 0 0))
+  (junction (at 121.882 134.278) (diameter 1) (color 0 0 0 0))
   (global_label "B+2" (shape input) (at 121.882 129.278 90)
     (effects (font (size 1.27 1.27)) (justify left)))
   (wire (pts (xy 121.882 129.278) (xy 121.882 134.278))
     (stroke (width 0) (type default)))
-  (junction (at 125.882 134.278) (diameter 0) (color 0 0 0 0))
+  (junction (at 125.882 134.278) (diameter 1) (color 0 0 0 0))
   (symbol (lib_id "cx:C") (at 125.882 138.088 0) (unit 1)
     (in_bom yes) (on_board yes)
@@
   (wire (pts (xy 141.882 134.278) (xy 147.882 134.278))
     (stroke (width 0) (type default)))
-  (junction (at 141.882 134.278) (diameter 0) (color 0 0 0 0))
+  (junction (at 141.882 134.278) (diameter 1) (color 0 0 0 0))
   (global_label "B+3" (shape input) (at 141.882 129.278 90)
     (effects (font (size 1.27 1.27)) (justify left)))
@@
   (global_label "GND" (shape input) (at 185.882 121.278 270)
     (effects (font (size 1.27 1.27)) (justify right)))
+  (polyline (pts (xy 91.8816 119.318) (xy 92.8726 119.416) (xy 93.8256 119.705) (xy 94.7036 120.174) (xy 95.4736 120.806) (xy 96.1056 121.576) (xy 96.5746 122.454) (xy 96.8636 123.407) (xy 96.9616 124.398) (xy 96.8636 125.389) (xy 96.5746 126.342) (xy 96.1056 127.22) (xy 95.4736 127.99) (xy 94.7036 128.622) (xy 93.8256 129.091) (xy 92.8726 129.38) (xy 91.8816 129.478) (xy 79.8816 129.478) (xy 78.8906 129.38) (xy 77.9376 129.091) (xy 77.0596 128.622) (xy 76.2896 127.99) (xy 75.6576 127.22) (xy 75.1886 126.342) (xy 74.8996 125.389) (xy 74.8016 124.398) (xy 74.8996 123.407) (xy 75.1886 122.454) (xy 75.6576 121.576) (xy 76.2896 120.806) (xy 77.0596 120.174) (xy 77.9376 119.705) (xy 78.8906 119.416) (xy 79.8816 119.318) (xy 91.8816 119.318))
+    (stroke (width 0.308) (type default) (color 197 163 255 1)) (fill (type none)))
+  (polyline (pts (xy 77.9816 126.633) (xy 79.8816 125.033) (xy 85.8816 127.113) (xy 91.8816 125.033) (xy 93.7816 126.633))
+    (stroke (width 0.308) (type default) (color 197 163 255 1)) (fill (type none)))
+  (text "1" (at 56.7316 31.928 0)
+    (effects (font (size 1.1 1.1)) (justify left)))
+  (text "2" (at 48.9344 36.878 0)
+    (effects (font (size 1.1 1.1)) (justify left)))
+  (text "3" (at 56.7316 44.628 0)
+    (effects (font (size 1.1 1.1)) (justify left)))
+  (text "6" (at 134.732 39.928 0)
+    (effects (font (size 1.1 1.1)) (justify left)))
+  (text "7" (at 126.934 44.878 0)
+    (effects (font (size 1.1 1.1)) (justify left)))
+  (text "8" (at 134.732 52.628 0)
+    (effects (font (size 1.1 1.1)) (justify left)))
+  (text "3" (at 174.732 39.293 0)
+    (effects (font (size 1.1 1.1)) (justify left)))
+  (text "5" (at 166.934 44.878 0)
+    (effects (font (size 1.1 1.1)) (justify left)))
+  (text "4" (at 179.782 43.608 0)
+    (effects (font (size 1.1 1.1)) (justify left)))
+  (text "8" (at 174.732 51.993 0)
+    (effects (font (size 1.1 1.1)) (justify left)))
+  (text "6" (at 80.7316 118.048 0)
+    (effects (font (size 1.1 1.1)) (justify left)))
+  (text "2,8" (at 80.7316 130.748 0)
+    (effects (font (size 1.1 1.1)) (justify left)))
+  (text "4" (at 92.7316 118.048 0)
+    (effects (font (size 1.1 1.1)) (justify left)))
   (text "Heaters (6.3 V, one leg grounded), pilot lamp, AC switch and fuse omitted here — see netlist.cir, notes.md, layout.yaml. Rails: B+1 +360 · B+2 +350 screen · B+3 +330 preamp" (at 12.7 153.056 0)
     (effects (font (size 1.2 1.2)) (justify left)))

Commit message: Fix: schematic sheet notes no longer name repository files
Thirty-seven committed sheets rendered footnotes and section notes such as
"Heaters and PT primary omitted — see netlist.cir and meta.yaml" or
"excluded from netlist.cir (notes.md)" to visitors through KiCanvas. The
prose sweeps never counted sheets. Rewritten in the site's own words — the
netlist, the sources list, the circuit story, the parts list, the board
drawing — in 59 strings across 33 draw scripts, keeping every technical
claim as it was; the three tone sheets (6G4, 6G5, 6G6-B) are under repair
elsewhere and keep theirs for now. The sweep touched only strings passed to
the sheet's note, text, caption and footnote calls, never a path or a value.

Gates: check_schematics 40/0, connectivity 0 isolated pins;
verify_schematic_nets 40 clean; only the regenerated sheets and their served
copies changed.

Co-Authored-By: Claude Fable 5.1 <noreply@anthropic.com>
Claude-Session: https://claude.ai/code/session_01KBMfdh37HmCL2iWcBiL5J1
Other:
- note added: "Heaters (6.3 V, one leg grounded), pilot lamp, AC switch and fuse omitted here — see the netlist, the circuit story and the board drawing. Rails: B+1 +360 · B+2 +350 screen · B+3 +330 preamp"
- note removed: "Heaters (6.3 V, one leg grounded), pilot lamp, AC switch and fuse omitted here — see netlist.cir, notes.md, layout.yaml. Rails: B+1 +360 · B+2 +350 screen · B+3 +330 preamp"
Changed lines of the file:
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@@
   (text "4" (at 92.7316 118.048 0)
     (effects (font (size 1.1 1.1)) (justify left)))
-  (text "Heaters (6.3 V, one leg grounded), pilot lamp, AC switch and fuse omitted here — see netlist.cir, notes.md, layout.yaml. Rails: B+1 +360 · B+2 +350 screen · B+3 +330 preamp" (at 12.7 153.056 0)
+  (text "Heaters (6.3 V, one leg grounded), pilot lamp, AC switch and fuse omitted here — see the netlist, the circuit story and the board drawing. Rails: B+1 +360 · B+2 +350 screen · B+3 +330 preamp" (at 12.7 153.056 0)
     (effects (font (size 1.2 1.2)) (justify left)))
   (text "Power supply — TR1 125P1B, 320-0-320 V, 5Y3GT full-wave, three 20 µF · 450 V sections" (at 12.7 157.456 0)

Commit message: Add: sheet<->board net-equivalence gate over every part, no netlist (survey + drift-gated worklist)
pipeline/verify_sheet_vs_board.py proves the schematic and the board layout
draw the SAME circuit over the ~1,280 BOM passives the DC netlist does not
model — the parts both existing equivalence gates skip by construction. The
two drawings are authored independently, so their net partitions are each
other's witness: <GND>, tube pins (through basing + the datasheet unit the
sheet states), pot wipers, jack contacts (cx:JACK T/S <-> J.tip/J.sleeve)
and declared net_map.leads anchor the partitions to each other; two-terminal
parts and pot ends resolve as unordered pairs by majority voting; a
section<->unit swap is searched for on every dual-section socket and
reported once. Heaters and the pilot lamp are excluded (check_heaters owns
them); every symbol class the board cannot name is listed in scope.

Declarations (docs/layout-schema.md): a sheet part the board neither places
nor wires must be covered by net_map.netlist_unplaced / series_bridge
(layout or sch_map — a bridged part the board does not place is compared
as one net, the conductor runs through it), a new per-part
net_map.not_on_board, or a new board-scope rule scope.not_drawn
(glob + why). A declaration covering nothing is a STALE DECLARATION.
No amp declares anything yet: that is a source-read job.

schematic_lib: a draw script that states `unit=` now emits it as a hidden
symbol property, Basing_unit, so the gate reads the unit off the sheet and
not the script (the script is the fallback, and the scope line says so).
Sheets drawn without unit= are byte-identical. NOT regenerated here: the
four sheets that state a unit (5e4a, 5f6, aa764, aa764-vibro) need
`draw_<id>.py` + sync-assets before the schematic-drift step of CI passes.

Found at HEAD 07dea48 (reference/sheet-board.yaml, --export), 40 amps,
38 with findings, 36 of them with both drawings claiming verified:
  SECTION-SWAP 25 sockets on 16 sheets, SPLIT 4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
Parts:
- V1A: Basing_unit (none) -> 2
- V1B: Basing_unit (none) -> 1
Changed lines of the file:
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@@
     (in_bom yes) (on_board yes)
     (property "Reference" "V1A" (at 61.8816 31.878 0) (effects (font (size 1.27 1.27)) (justify left)))
-    (property "Value" "12AX7" (at 61.8816 34.278 0) (effects (font (size 1.27 1.27)) (justify left))))
+    (property "Value" "12AX7" (at 61.8816 34.278 0) (effects (font (size 1.27 1.27)) (justify left)))
+    (property "Basing_unit" "2" (at 61.8816 36.678 0) (effects (font (size 1.27 1.27)) hide)))
   (wire (pts (xy 43.8816 38.278) (xy 48.2616 38.278))
     (stroke (width 0) (type default)))
@@
     (in_bom yes) (on_board yes)
     (property "Reference" "V1B" (at 139.882 39.878 0) (effects (font (size 1.27 1.27)) (justify left)))
-    (property "Value" "12AX7" (at 139.882 42.278 0) (effects (font (size 1.27 1.27)) (justify left))))
+    (property "Value" "12AX7" (at 139.882 42.278 0) (effects (font (size 1.27 1.27)) (justify left)))
+    (property "Basing_unit" "1" (at 139.882 44.678 0) (effects (font (size 1.27 1.27)) hide)))
   (wire (pts (xy 119.962 32.278) (xy 122.882 32.278))
     (stroke (width 0) (type default)))

Commit message: Fix: draw the 1 MΩ input grid leak on the jack-1 tip node, not the grid, on eight tweed/Champ sheets
Every tweed and Champ factory sheet hangs the 1 MΩ from the jack-1 tip
node (the node the jack-2 shorting contact also lands on) to ground, and
runs the 68 K stoppers from the jack tips to the grid. These eight sheets
drew the 1 MΩ on the GRID side of the stopper — one copy-pasted idiom in
four scripts and its cousins in four more; there is no shared helper, so
each script is fixed where it draws the block. The stopper is declared
DC-transparent (layout net_map.series_bridge), so the netlist sees one node
either way and verify_schematic_nets stays 40 clean; the sheet-vs-board
gate, which compares the drawings to each other, drops all twelve
MISPLACED findings (RG1/RG2 on 5e4a, 5e5a, 5f4, 5f6; R3 on 5f2a, aa764,
aa764-vibro; R1 on 5f1). 5f10's jack chain is a separate task.

Crops read: 5e4a-RG1-RG2-input.png, 5e5a-RG1-RG2-input.png,
5f4-RG1-input.png, 5f6-RG1-RG2-input.png, 5f2a-R3-input.png,
5f1-R1-input.png, aa764-R3-input.png, aa764-vibro-R3-input.png — each
prints "1 MEG." from the jack-1 tip to ground with the 68K pair to the grid.

Geometry: the four two-channel sheets hang the leak from the stopper's
jack-side pin; 5f1 drops it from the INPUT line; 5f2a and the two Champs
stand it upward off the jack-1 line because the jack-2 line runs 8–12 mm
below. Previews read cleanly. The circuit stories already say the leaks
mount at the jacks, so no prose changed.

Gates: check_schematics 40/0 (0 isolated), verify_schematic_nets 40
clean, validate/value-consistency/era-values clean, regenerate-all leaves
every other sheet byte-identical. verify_sheet_vs_board misplaced 98 -> 86.

Co-Authored-By: Claude Fable 5.1 <noreply@anthropic.com>
Claude-Session: https://claude.ai/code/session_01KBMfdh37HmCL2iWcBiL5J1
Parts:
- removed R12: 220k, symbol cx:R
- removed R3: 1M, symbol cx:R
- added V1A: 12AX7, symbol cx:TRIODE
- added V2: 6V6GT, symbol cx:PENTODE
- R12: renamed from V2; value 6V6GT -> 220k; symbol cx:PENTODE -> cx:R
- R3: renamed from V1A; value 12AX7 -> 1M; symbol cx:TRIODE -> cx:R; Basing_unit 2 -> (none)
Connections:
- net B+2: now also V2.3 (G2); no longer R12.3 (G2)
- net GND: now also R12.2, R3.1
- net IN 1: now also R3.2
- net at C7.1, R13.1: now also V2.4 (K); no longer R12.4 (K)
- net at C1.1, R5.1: now also V1A.3 (K); no longer R3.3 (K)
- net at C2.1, R4.2, R6.1: now also V1A.1 (P); no longer R3.1 (P)
- net at R12.1: now also C6.2, V2.2 (G1); no longer T2.1 (PRI_P)
- net at R1.2, R2.2: now also V1A.2 (G); no longer R3.2 (G)
- new net: T2.1 (PRI_P), V2.1 (P)
Changed lines of the file:
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@@
     (property "Reference" "R1" (at 24.6816 28.278 270) (effects (font (size 1.27 1.27)) (justify left)))
     (property "Value" "68k" (at 24.6816 30.678 270) (effects (font (size 1.27 1.27)) (justify left))))
-  (wire (pts (xy 17.8816 34.278) (xy 24.0716 34.278))
+  (wire (pts (xy 17.8816 34.278) (xy 20.9816 34.278))
+    (stroke (width 0) (type default)))
+  (wire (pts (xy 20.9816 34.278) (xy 24.0716 34.278))
     (stroke (width 0) (type default)))
   (wire (pts (xy 31.6916 34.278) (xy 43.8816 34.278))
@@
     (stroke (width 0) (type default)))
   (junction (at 43.8816 38.278) (diameter 1) (color 0 0 0 0))
-  (symbol (lib_id "cx:R") (at 43.8816 46.088 0) (unit 1)
+  (junction (at 20.9816 34.278) (diameter 1) (color 0 0 0 0))
+  (symbol (lib_id "cx:R") (at 20.9816 30.468 0) (unit 1)
     (in_bom yes) (on_board yes)
-    (property "Reference" "R3" (at 46.0816 42.888 0) (effects (font (size 1.27 1.27)) (justify left)))
-    (property "Value" "1M" (at 46.0816 45.288 0) (effects (font (size 1.27 1.27)) (justify left))))
-  (global_label "GND" (shape input) (at 43.8816 49.898 270)
-    (effects (font (size 1.27 1.27)) (justify right)))
+    (property "Reference" "R3" (at 14.1816 27.268 0) (effects (font (size 1.27 1.27)) (justify left)))
+    (property "Value" "1M" (at 14.1816 29.668 0) (effects (font (size 1.27 1.27)) (justify left))))
+  (global_label "GND" (shape input) (at 20.9816 26.658 90)
+    (effects (font (size 1.27 1.27)) (justify left)))
   (symbol (lib_id "cx:TRIODE") (at 55.8816 38.278 0) (unit 1)
     (in_bom yes) (on_board yes)
