File: amps/6g6b/schematic.kicad_sch (KiCad schematic)
At the start: 88 parts, among them T1 125P7A, T3 125A13A

Commit message: Fix: one lettering convention per surface, engine-enforced; legend inside the viewBox
WS3 — layout pipeline + cross-surface value-consistency engine.

## One convention per surface (docs/lettering-conventions.md, new)

The same part stated its value in several notations at once. 5E3 C6 and 5D3 C6
rendered "5n" on the schematic, "0.005 µF · 600 V" in the parts list and
"0.005 µF" on the board. 5F6-A RD1 printed "4,700 Ω" beside neighbours printing
"15 kΩ". check_value_consistency proves the surfaces name the same QUANTITY; it
cannot see that they name it three ways. So each surface now has exactly one
convention and every one of them is gated:

* house units in bom.yaml/prose — engineering prefix with the mantissa 1…999,
  pF below 1000 pF and µF at and above it, no comma-grouped thousands. 19 values
  normalised (5E6-A, 5F6-A, 5F10, 6161, 6G2, 6G5, 6G6-B).
* schematic drafting shorthand — the unit letter is the SI prefix of the house
  unit, in the amp's declared idiom (meta.yaml conventions.notation: us|uk).
  British RKM/nanofarad practice on the Hiwatt and the 2204 is DECLARED, not
  normalised away; it is what those source drawings letter. Secondary ratings
  are space-separated fields with their own unit ("20u 600V"), never the era's
  dashed shorthand and never the house middot. 30 symbol values corrected across
  ten draw scripts.
* era sheet lettering — generated only, by era_pair(); documented cases and a
  corpus round-trip sweep in test_era_values.py, now 57 cases.

## Era-lettering fall-throughs closed

A value era_pair() refuses came back as the house string, and a house string can
be a whole sentence. Fixed at the source rather than per case:

* body_value() — a parenthetical GLOSS is never lettered on a component body.
  "selenium (silicon diode in modern builds)" was lettered in full on the 5E4-A
  and ran off the left edge of the page.
* twin cans letter as the era sheets did: 25 µF + 25 µF -> "25/25MFD".
* a repeat count is not a rating: "(×2)" com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
Parts:
- C10, C11: value 20u·600V -> 20u 600V
- C12: value 20u·600V (dual) -> 20u 600V
- RB1: value 1k·1W·5% -> 1k 1W 5%
- RB2: value 27k·1W·5% -> 27k 1W 5%
- RD1: value 4700·1W -> 4.7k 1W
- RD2: value 27k·1W -> 27k 1W
- RK1A, RK2B: value 2700 -> 2.7k
- RK2A, RK3B: value 1500 -> 1.5k
- RK3A: value 1500 (est) -> 1.5k (est)
- RL4A: value 82k · 5% -> 82k 5%
- RL4B: value 100k · 5% -> 100k 5%
- RS5, RS6: value 470 · 1W -> 470 1W
- RTN4: value 6800 -> 6.8k
Changed lines of the file:
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@@
     (in_bom yes) (on_board yes)
     (property "Reference" "RK1A" (at 62.2 50.61 0) (effects (font (size 1.27 1.27)) (justify left)))
-    (property "Value" "2700" (at 62.2 53.01 0) (effects (font (size 1.27 1.27)) (justify left))))
+    (property "Value" "2.7k" (at 62.2 53.01 0) (effects (font (size 1.27 1.27)) (justify left))))
   (symbol (lib_id "cx:C") (at 67.62 53.81 0) (unit 1)
     (in_bom yes) (on_board yes)
@@
     (in_bom yes) (on_board yes)
     (property "Reference" "RK2A" (at 62.2 140.61 0) (effects (font (size 1.27 1.27)) (justify left)))
-    (property "Value" "1500" (at 62.2 143.01 0) (effects (font (size 1.27 1.27)) (justify left))))
+    (property "Value" "1.5k" (at 62.2 143.01 0) (effects (font (size 1.27 1.27)) (justify left))))
   (symbol (lib_id "cx:C") (at 67.62 143.81 0) (unit 1)
     (in_bom yes) (on_board yes)
@@
     (in_bom yes) (on_board yes)
     (property "Reference" "RTN4" (at 130.2 142.89 0) (effects (font (size 1.27 1.27)) (justify left)))
-    (property "Value" "6800" (at 130.2 145.29 0) (effects (font (size 1.27 1.27)) (justify left))))
+    (property "Value" "6.8k" (at 130.2 145.29 0) (effects (font (size 1.27 1.27)) (justify left))))
   (global_label "GND" (shape input) (at 128 149.9 270)
     (effects (font (size 1.27 1.27)) (justify left)))
@@
     (in_bom yes) (on_board yes)
     (property "Reference" "RK2B" (at 198.2 140.61 0) (effects (font (size 1.27 1.27)) (justify left)))
-    (property "Value" "2700" (at 198.2 143.01 0) (effects (font (size 1.27 1.27)) (justify left))))
+    (property "Value" "2.7k" (at 198.2 143.01 0) (effects (font (size 1.27 1.27)) (justify left))))
   (symbol (lib_id "cx:C") (at 203.62 143.81 0) (unit 1)
     (in_bom yes) (on_board yes)
@@
     (in_bom yes) (on_board yes)
     (property "Reference" "RK3A" (at 248.2 162.61 0) (effects (font (size 1.27 1.27)) (justify left)))
-    (property "Value" "1500 (est)" (at 248.2 165.01 0) (effects (font (size 1.27 1.27)) (justify left))))
+    (property "Value" "1.5k (est)" (at 248.2 165.01 0) (effects (font (size 1.27 1.27)) (justify left))))
   (global_label "GND" (shape input) (at 246 169.62 270)
     (effects (font (size 1.27 1.27)) (justify left)))
@@
     (in_bom yes) (on_board yes)
     (property "Reference" "RK3B" (at 304.2 162.61 0) (effects (font (size 1.27 1.27)) (justify left)))
-    (property "Value" "1500" (at 304.2 165.01 0) (effects (font (size 1.27 1.27)) (justify left))))
+    (property "Value" "1.5k" (at 304.2 165.01 0) (effects (font (size 1.27 1.27)) (justify left))))
   (global_label "GND" (shape input) (at 302 169.62 270)
     (effects (font (size 1.27 1.27)) (justify left)))
@@
     (in_bom yes) (on_board yes)
     (property "Reference" "RL4A" (at 350.2 181.89 0) (effects (font (size 1.27 1.27)) (justify left)))
-    (property "Value" "82k · 5%" (at 350.2 184.29 0) (effects (font (size 1.27 1.27)) (justify left))))
+    (property "Value" "82k 5%" (at 350.2 184.29 0) (effects (font (size 1.27 1.27)) (justify left))))
   (wire (pts (xy 348 181.28) (xy 348 178.74))
     (stroke (width 0) (type default)))
@@
     (in_bom yes) (on_board yes)
     (property "Reference" "RL4B" (at 350.2 217.89 0) (effects (font (size 1.27 1.27)) (justify left)))
-    (property "Value" "100k · 5%" (at 350.2 220.29 0) (effects (font (size 1.27 1.27)) (justify left))))
+    (property "Value" "100k 5%" (at 350.2 220.29 0) (effects (font (size 1.27 1.27)) (justify left))))
   (wire (pts (xy 348 217.28) (xy 348 214.74))
     (stroke (width 0) (type default)))
@@
     (in_bom yes) (on_board yes)
     (property "Reference" "RS5" (at 431.23 192.73 270) (effects (font (size 1.27 1.27)) (justify left)))
-    (property "Value" "470 · 1W" (at 431.23 195.13 270) (effects (font (size 1.27 1.27)) (justify left))))
+    (property "Value" "470 1W" (at 431.23 195.13 270) (effects (font (size 1.27 1.27)) (justify left))))
   (wire (pts (xy 438.24 198.73) (xy 439.62 198.73))
     (stroke (width 0) (type default)))
@@
     (in_bom yes) (on_board yes)
     (property "Reference" "RS6" (at 431.23 228.73 270) (effects (font (size 1.27 1.27)) (justify left)))
-    (property "Value" "470 · 1W" (at 431.23 231.13 270) (effects (font (size 1.27 1.27)) (justify left))))
+    (property "Value" "470 1W" (at 431.23 231.13 270) (effects (font (size 1.27 1.27)) (justify left))))
   (wire (pts (xy 438.24 234.73) (xy 439.62 234.73))
     (stroke (width 0) (type default)))
@@
     (in_bom yes) (on_board yes)
     (property "Reference" "C10" (at 98.2 360.61 0) (effects (font (size 1.27 1.27)) (justify left)))
-    (property "Value" "20u·600V" (at 98.2 363.01 0) (effects (font (size 1.27 1.27)) (justify left))))
+    (property "Value" "20u 600V" (at 98.2 363.01 0) (effects (font (size 1.27 1.27)) (justify left))))
   (global_label "GND" (shape input) (at 96 367.62 270)
     (effects (font (size 1.27 1.27)) (justify left)))
@@
     (in_bom yes) (on_board yes)
     (property "Reference" "RD1" (at 102.8 354 270) (effects (font (size 1.27 1.27)) (justify left)))
-    (property "Value" "4700·1W" (at 102.8 356.4 270) (effects (font (size 1.27 1.27)) (justify left))))
+    (property "Value" "4.7k 1W" (at 102.8 356.4 270) (effects (font (size 1.27 1.27)) (justify left))))
   (wire (pts (xy 96 360) (xy 102.19 360))
     (stroke (width 0) (type default)))
@@
     (in_bom yes) (on_board yes)
     (property "Reference" "C11" (at 152.2 360.61 0) (effects (font (size 1.27 1.27)) (justify left)))
-    (property "Value" "20u·600V" (at 152.2 363.01 0) (effects (font (size 1.27 1.27)) (justify left))))
+    (property "Value" "20u 600V" (at 152.2 363.01 0) (effects (font (size 1.27 1.27)) (justify left))))
   (global_label "GND" (shape input) (at 150 367.62 270)
     (effects (font (size 1.27 1.27)) (justify left)))
@@
     (in_bom yes) (on_board yes)
     (property "Reference" "RD2" (at 160.8 354 270) (effects (font (size 1.27 1.27)) (justify left)))
-    (property "Value" "27k·1W" (at 160.8 356.4 270) (effects (font (size 1.27 1.27)) (justify left))))
+    (property "Value" "27k 1W" (at 160.8 356.4 270) (effects (font (size 1.27 1.27)) (justify left))))
   (wire (pts (xy 156 360) (xy 160.19 360))
     (stroke (width 0) (type default)))
@@
     (in_bom yes) (on_board yes)
     (property "Reference" "C12" (at 184.2 360.61 0) (effects (font (size 1.27 1.27)) (justify left)))
-    (property "Value" "20u·600V (dual)" (at 184.2 363.01 0) (effects (font (size 1.27 1.27)) (justify left))))
+    (property "Value" "20u 600V" (at 184.2 363.01 0) (effects (font (size 1.27 1.27)) (justify left))))
   (global_label "GND" (shape input) (at 182 367.62 270)
     (effects (font (size 1.27 1.27)) (justify left)))
@@
     (in_bom yes) (on_board yes)
     (property "Reference" "RB1" (at 254.8 294 270) (effects (font (size 1.27 1.27)) (justify left)))
-    (property "Value" "1k·1W·5%" (at 254.8 296.4 270) (effects (font (size 1.27 1.27)) (justify left))))
+    (property "Value" "1k 1W 5%" (at 254.8 296.4 270) (effects (font (size 1.27 1.27)) (justify left))))
   (wire (pts (xy 250 300) (xy 254.19 300))
     (stroke (width 0) (type default)))
@@
     (in_bom yes) (on_board yes)
     (property "Reference" "RB2" (at 276.8 294 270) (effects (font (size 1.27 1.27)) (justify left)))
-    (property "Value" "27k·1W·5%" (at 276.8 296.4 270) (effects (font (size 1.27 1.27)) (justify left))))
+    (property "Value" "27k 1W 5%" (at 276.8 296.4 270) (effects (font (size 1.27 1.27)) (justify left))))
   (wire (pts (xy 270 300) (xy 276.19 300))
     (stroke (width 0) (type default)))

Commit message: Update: regenerate every drawing the four merged units changed
The four parallel units all rewrote generators, so their committed artifacts
were each generated against only their own third of the merged pipeline. Every
schematic, both layout styles, the social cards and the manifest are rebuilt
here from the merged sources, so what ships is what the merged generators draw.

One integration fault the rebuild exposed, invisible to any single unit:

- 5E5-A: the note explaining that the Presence wiper and the 100k feedback
  resistor land on V3A's GRID (not its cathode, as on the 5F4) was added as a
  hand-placed `s.text()` at a coordinate chosen before the sheet gained a
  reserved notes band. Merged, it printed through the -32V bias label. Moved to
  `note()`, which wraps prose into that band — the exact failure mode the band
  was built to end.

Three conflicts resolved against docs/lettering-conventions.md rather than by
picking a side, since two units had corrected the same lines for different
reasons:

- 5E5-A tone/feedback caps take the corrected designators (C7, C8, C9, RNF —
  `C_tr1`/`C_NFB` were generator identifiers that had leaked onto a published
  board) with the house-derived lettering (`.01u 400V`, `500p`, `.1u 200V`).
  Dropping the working voltage or writing `.0005u` would have lost a rating the
  source prints and re-broken the pF/µF decade rule.
- 5D3 C6 and 6G6-B's three cathode resistors take the SI-prefix form the
  convention binds (`.005u`, `2.7k`, `1.5k`), keeping the ground-flag direction
  fix and the removal of the second `gnd()` that shorted each cathode it biased.
- 5F6-A's bias supply keeps both 8 µF cans drawn — the second was previously a
  parenthetical claiming one of two was shown — at the coordinates that clear
  the title-block strip.

All gates green, including check_value_consistency at zero disagreements.

🤖 Generated with [Claude Code](https://claude.com/claude-code)

Co-Authored-By: Claude Fable 5 <noreply@anthropic.com>
Connections:
- net GND: no longer CK1A.1, CK2A.1, CK2B.1, RK1A.1, RK2A.1, RK2B.1, V1A.3 (K), V2A.3 (K), V2B.3 (K)
- new net: CK2B.1, RK2B.1, V2B.3 (K)
- new net: CK1A.1, RK1A.1, V1A.3 (K)
- new net: CK2A.1, RK2A.1, V2A.3 (K)
Other:
- note removed: "Model 6G6-B — Blonde Bassman-style · Circuit Codex · CC-BY-SA 4.0 · redrawn from circuit facts"
- company: (none) -> Circuit Codex
- title: (none) -> 6G6-B — Blonde Bassman-style

Commit message: Fix: the 6G6-B's V1B is a cathode follower, and "+13.6 V" is "+136 V"
Both chart disagreements that held this entry open were our reading of the
sheet, not the sheet. A lug-level re-read of the E-FB schematic page at 750 dpi
shows:

- V1B is a CATHODE FOLLOWER. Its plate lead runs straight to the Bass row's
  +230 V lane with no plate-load resistor, its grid takes V1A's plate directly
  (no coupling cap, no grid leak), and the 100k cathode load is the output. The
  printed figure is +136 V, not +13.6 V — the mark between the 3 and the 6 is
  the +230 V lane's own wire crossing the lettering. The earlier pass invented
  a coupling cap, a grid leak and a 220k plate load; none is on the sheet.
- The sheet letters "+230 V." three times. Twice it is the Bass row's B+ lane;
  the third is V2A's PLATE, whose 100k load climbs to the +355 V lane. Reading
  it as a shared preamp rail is what missed V2A's printed cathode by a third.
- The phase-inverter foot is fully lettered after all: 6800 from the tail
  junction to the feedback node, 4700 from there to ground, with the 56k
  speaker feedback returning to the same node. The 10k estimate is gone.
- K3A and P1B were carried as chart: null estimates; K3A (+1.2 V) is printed
  beside the stage, and P1B does not exist on a follower.

The drawing corroborates itself twice: 136 V over 100k is the 1.36 mA that
makes the 56k rail dropper arrive at +230 V, and 125 V over V2A's 100k is the
1.25 mA its printed 1.9 V over 1500 implies. Every gated node now lands, worst
17.3% against the chart's own +/-20%. Schematic, both layout styles and the
social card are regenerated. Still draft — the remaining blocker is maintainer
sign-off, which is not ours to grant.

Co-Authored-By: Claude Fable 5 <noreply@anthropic.com>
Parts:
- removed C0: .1u (est), symbol cx:C
- removed RFOOT: 10k (est), symbol cx:R
- removed RG1B: 1M, symbol cx:R
- removed RL1B: 220k (est), symbol cx:R
- added C14: 20u 600V, symbol cx:C
- added RD3, RNFB: 56k 1W, symbol cx:R
- added RPF: 4.7k, symbol cx:R
- added RT2: 6.8k, symbol cx:R
Connections:
- net GND is gone; now on net BP428: C10.2, C11.2, C12.2, C13.2, CK1A.2, CK2A.2, CK2B.2, RB2.2, RBF.2, RG1A.2, RG2A.2, RG2B.2, RG3A.2, RG3B.2, RGL5.2, RGL6.2, RK1A.2, RK1B.2, RK2A.2, RK2B.2, RK3A.2, RK3B.2, RTN4.2, T1.4 (HT_CT), V5.4 (K), V6.4 (K), VR2.3, VR3.3, VR4.2 (W), VR5.3, VR6.3, VR7.3
- net BP230: now also V1B.1 (P)
- net BP428: now also C14.2, RD3.1, RPF.2
- net SPKR: now also VR7.1, RNFB.1, RNFB.2, RPF.1, RT2.2
- net at RG4A.2, RG4B.1, RG4B.2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: now also RT2.1; no longer VR7.1
- net at RL1A.2, V1A.1 (P): now also V1B.2 (G)
- net at RTN2.1: now also V1B.3 (K); no longer V1B.1 (P)
- net at RK1B.1: no longer V1B.3 (K)
- new net: C14.1, RD3.2
Other:
- note added: "Bass ch. tone network: redrawn from the E-FB"
- note added: "Presence control: front-panel 25 kΩ-L pot bridging the 4.7 kΩ foot resistor end to end, its wiper on a 0.1 µF · 200 V cap to the foot."
- note added: "The 56 kΩ speaker feedback returns to the same foot node, so it is a second DC path to ground through the output transformer's secondary."
- note added: "modelled in netlist.cir (control island)."
- note added: "schematic page, driven by V1B's cathode. Not"
- note removed: "Bass ch. tone network: redrawn from the E-FB schematic page. NW/NY bridging exactly as the source drawing wires it (best-effort read of a"
- note removed: "Presence control: front-panel 25 kΩ-L pot at the phase-inverter tail junction; exact internal tap not traced from the available scan —"
- note removed: "drawn as a DC-neutral shunt at the tail, matching the corpus's other long-tailed-pair designs."
- note removed: "hand-drawn print — not a trace); the network is not modelled in netlist.cir (abstracted control island, same convention corpus-wide)."

Commit message: Fix: deterministic schematic ids and wires split at every join
- _u() is uuid5 over (amp id, emission order), so a regeneration of an
  unchanged script is byte-identical and a drift gate becomes possible
- write() splits wire segments at symbol pins, wire ends and junction dots,
  so the file connects exactly what the drawing shows under KiCad's
  endpoint-only semantics (270 pins were on a wire's interior; net
  partitions unchanged on all 38 sheets)
- all sheets regenerated; aa864-bassman title block was stale (draft) and
  now matches meta.yaml (verified)

Co-Authored-By: Claude Fable 5.1 <noreply@anthropic.com>
Claude-Session: https://claude.ai/code/session_01KBMfdh37HmCL2iWcBiL5J1
Connections:
- net BP428: now also CTN4.2, CTN5.2, V5.1 (P), V6.1 (P), VR3.1
- net HT_A: now also DR1.2 (K)
- net HT_B: now also DR4.2 (K)
- net at R3s.2, R4s.2, V2A.2 (G): now also RG2A.1
- net at C10.1, RD1.1: now also DR3.1 (A), DR6.1 (A)
- net at R1s.2, R2s.2, V1A.2 (G): now also RG1A.1
- net at DR3.2 (K): now also DR2.1 (A)
- net at DR1.1 (A): now also DR2.2 (K)
- net at DR5.1 (A): now also DR6.2 (K)
- net at DR5.2 (K): now also DR4.1 (A)
- net at CTN1.2, RTN2.2, VR2.1: now also RTN1.1, RTN1.2

Commit message: Fix: schematic wiring on 6g3, 6g4, 6g5, 6g6b
- long-tailed pair tail moved off section B's plate to its cathode (6g3,
  6g4, 6g5); 6g4 V8 plate lead was drawn under its grounded cathode
- 6g6b: all five OT leads on bare coordinates with the secondary drawn on
  the primary side; bias line taken off the bleeder's grounded end (NBIAS
  and GND one net); both tone networks rebuilt; mixing bus ran through
  V3A's bottle
- eight parts shorted end to end, invisible to the pin check: 6g4 RGL1;
  6g5 RG5 (mixing node on ground); 6g6b C11, RG4B, RNFB, RTAIL, RTN1, VR3
- 6g5: treble pot runs off each other's lug, driver run 12 mm short of
  V6A grid, CFB1 rotated but wired upright, choke leads short both ends
- five dated waivers (bridge rectifier centre tap, footswitch terminal
  not lettered on the source, mains side outside the drawing, VR7's
  undesignated cap)
- OPEN, not guessed: 6g5 presence network is drawn as a DC path to ground
  (RPRES + pot in series) while netlist.cir has RT2 to ground and calls the
  network DC-neutral; sources do not settle it — sheet stays unclaimed

Co-Authored-By: Claude Fable 5.1 <noreply@anthropic.com>
Claude-Session: https://claude.ai/code/session_01KBMfdh37HmCL2iWcBiL5J1
Parts:
- removed CTN3: .25u, symbol cx:C
- removed CTN4: 250p, symbol cx:C
- removed RBF, RTAIL: 820, symbol cx:R
- removed RG3B: 1M (est), symbol cx:R
- removed RK3B: 1.5k, symbol cx:R
- removed RM1, RM2: 470k, symbol cx:R
- removed RTN4: 6.8k, symbol cx:R
- removed V2A: 7025, symbol cx:TRIODE
- removed VR5: 1M-A, symbol cx:POT
- removed VR7: 25k-L · Presence, symbol cx:POT
- added C2: .1u, symbol cx:C
- added CTN6: .005u, symbol cx:C
- added R3s: 68k, symbol cx:R
- added RG2B, RG3A: 1M (est), symbol cx:R
- added RL4A: 82k 5%, symbol cx:R
- added RPF: 4.7k, symbol cx:R
- added V4A, V4B: 7025, symbol cx:TRIODE
- added VR1: 25k-L, symbol cx:POT
- added VR2: 250k-L, symbol cx:POT
- added VR3: 350k-70k, symbol cx:POT
- C1: renamed from RL4A; value 82k 5% -> 500p; symbol cx:R -> cx:C
- CTN3: renamed from RTN3; value 10k -> .25u; symbol cx:R -> cx:C
- CTN4: renamed from VR3; value 350k-70k -> 250p; symbol cx:POT -> cx:C
- RBF: renamed from VR2; value 250k-L -> 820; symbol cx:POT -> cx:R
- RG3B: renamed from RL3B; value 100k -> 1M (est)
- RK3B: renamed from C1; value 500p -> 1.5k; symbol cx:C -> cx:R
- RL3B: renamed from V4A; value 7025 -> 100k; symbol cx:TRIODE -> cx:R
- RM1: renamed from RG3A; value 1M (est) -> 470k
- RM2: renamed from V4B; value 7025 -> 470k; symbol cx:TRIODE -> cx:R
- RTAIL: renamed from RPF; value 4.7k -> 820
- RTN3: renamed from VR1; value 25k-L -> 10k; symbol cx:POT -> cx:R
- RTN4: renamed from CTN6; value .005u -> 6.8k; symbol cx:C -> cx:R
- V2A: renamed from R3s; value 68k -> 7025; symbol cx:R -> cx:TRIODE
- VR5: renamed from RG2B; value 1M (est) -> 1M-A; symbol cx:R -> cx:POT
- VR7: renamed from C2; value .1u -> 25k-L · Presence; symbol cx:C -> cx:POT
Connections:
- net BP230: now also RL3B.1; no longer RG3B.1, RL2A.1
- net BP355: now also RL2A.1
- net BP410: now also RL4A.1; no longer C1.1
- net BP428: now also T3.2 (CT); no longer C10.2, C11.2, C12.2, C13.2, C14.2, CK1A.2, CK2A.2, CK2B.2, CTN4.1, CTN4.3, CTN5.2, RB2.2, RBF.3, RG1A.2, RG2A.2, RGL5.2, RGL6.2, RK1A.2, RK1B.2, RK2A.2, RK2B.2, RK3A.2, RM1.2, RTAIL.2, T1.4 (HT_CT), V5.1 (P), V5.4 (K), V6.1 (P), V6.4 (K), VR4.2 (W), VR5.2, VR6.3
- net NORM2: now also R3s.1; no longer V2A.1
- net SPKR: now also T3.4 (SEC_H); no longer RNFB.2, RT2.2, RTAIL.1
- net at VR7.2 (W): no longer V5.2 (G1)
- net at RTN3.1: now also CTN2.2, RTN1.2, RTN2.2, VR1.1, VR1.2 (W), VR2.1; no longer RTN3.2 (W)
- net at RGL6.1: now also C3.2, V6.2 (G1)
- net at CK2A.1, RK2A.1: now also V2A.3 (K)
- net at V3B.1 (P): now also RL3B.2, RM2.1; no longer RG3B.2
- net at RK3B.1: now also V3B.3 (K)
- net at CTN3.1: now also CTN1.1, CTN2.1, RK1B.1, RTN2.1, V1B.3 (K)
- net at CTN3.2: now also RTN3.2, VR1.3
- net at RL2B.2, V2B.1 (P): now also RM1.1
- net NBIAS: now reaches C13.1, RB1.2, RB2.1
- net NBIAS: now also RGL5.2, RGL6.2
- net at T3.1 (PRI_A): now also V5.1 (P)
- net at T3.3 (PRI_B): now also V6.1 (P)
- net GND: now reaches T3.5 (SEC_C)
- net GND: now also C10.2, C11.2, C12.2, C13.2, C14.2, CK1A.2, CK2A.2, CK2B.2, RB2.2, RBF.2, RG1A.2, RG2A.2, RG3B.2, RK1A.2, RK1B.2, RK2A.2, RK2B.2, RK3A.2, RK3B.2, RTN4.2, T1.4 (HT_CT), V5.4 (K), V6.4 (K), VR4.2 (W), VR4.3, VR5.3, VR6.3, VR7.3, CTN6.2, RG2B.2, RG3A.2, RPF.2, VR2.3
- net at VR5.1: now also VR3.2 (W)
- net at V2B.2 (G): now also VR5.2 (W), RG2B.1
- net at V3A.2 (G): now also RM1.2, RG3A.1, VR2.2 (W)
- net at CTN4.2: now also VR3.1
- net at RTN4.1: now also CTN5.2, VR4.1, CTN6.1, VR3.3
- net at R4s.2, RG2A.1, V2A.2 (G): now also R3s.2
- net at CTN5.1, RL2A.2: now also CTN4.1, V2A.1 (P)
- net at C3.1, RL4B.2: now also V4B.1 (P); no longer RM2.1 (P)
- net at V3B.2 (G), VR6.2 (W): now also RG3B.1
- net at RGL5.1: now also V5.2 (G1), C2.2
- new net: RNFB.2, RPF.1, RT2.2, VR7.1
- new net: CTN1.2, RTN1.1
- new net: C1.1, RM2.2
- new net: C1.2, RG4A.1, V4A.2 (G)
- new net: RG4A.2, RG4B.2, RT2.1, RTAIL.2
- new net: RTAIL.1, V4A.3 (K), V4B.3 (K)
- new net: C2.1, RL4A.2, V4A.1 (P)
- new net: RG4B.1, V4B.2 (G)
- now unconnected: RBF.1
Other:
- moved on the sheet: RD3, RG3B, RM1, RTAIL
