File: amps/6g6b/schematic.kicad_sch (KiCad schematic)
At the start: 89 parts, among them T1 125P7A, T3 125A13A

Commit message: Add: real tube pin numbers and readable valve glyphs on every schematic
Phase B of the drawing program. A factory service sheet numbers every tube
pin, because the number is what a technician puts a probe on. This corpus
printed none, and the numbers hidden in its symbols were positional
placeholders (P=1, G=2, K=3) that would have published a 6V6GT's plate as
pin 1 when it is pin 3.

1055 electrodes now carry the real number, 1027 lettered (27 are shared
filaments deduped, 1 dropped for want of clear space on the 6G2). Resolved per
instance from reference/tubes/<slug>.yaml through the same alias resolution the
layout renderer uses, so a 12AX7 section and a 6SL7 section each get their own
basing. A valve whose basing the corpus does not carry prints nothing rather
than a wrong number.

Section letters and basing units are now separate things, which cost a detour
worth recording. The RCA 12AX7-A sheet reads "Pin 1 - Plate of Unit No.2 ...
Pin 6 - Plate of Unit No.1", so unit numbering is not pin order; the 5Y3 and
GZ34 number their units in opposite pin order, so nothing positional can
express it. But the section LETTER is a designator, not a basing fact: this
corpus, like every technician, calls the first stage in signal order V1A, and
five amps' prose already did. On four amps the factory sheets put that first
stage on the other half -- the AA764's own schematic prints +200 V on pin 1 --
so those drawings now state their unit explicitly, each citing its source, and
no letter, netlist, parts list or layout comment changed. 183 layout comments
agree with the printed numbers, 0 disagree. A guard fires if two halves of one
bottle resolve to the same unit, which is exactly how this was found.

Glyphs: the cathode gains a bracket and filament hairpin so it can no longer be
confused with the plate bar, the pentode's screen sits on its own row, and a
rectifier draws as one envelope over its sections instead of two apparent
bottles. Line weights are scaled per sheet to a co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
Other:
- note added: "1"
- note added: "2"
- note added: "3"
- note added: "4"
- note added: "5"
- note added: "6"
- note added: "7"
- note added: "8"

Commit message: Fix: 6G6-B Normal-channel tone network redrawn from the E-FB sheet — the blackface ladder on a tapped Treble pot
- The sheet draws: 100K slope off the V2A plate to a slope foot; .00025 from the
  plate to the Treble pot's hot lug; .1 from the slope foot to the pot's 70K TAP,
  where the 250K-A Bass rheostat hangs; .05 from the slope foot to the Bass foot;
  6800 from there to ground; the Treble pot's cold lug bled to ground through
  .005. Six parts and a four-terminal pot.
- The drawing had no slope resistor and no .1, ran the .05 from the plate, and
  collapsed the slope foot, the tap and the Bass foot into one node; the parts
  list was missing the 100K and the .1. Under the layout's verified wiring badge,
  which is true of the netlist-modelled parts and says nothing about this island.
- Sheet: RTN5 100k and CTN7 .1u added, VR3 drawn on cx:POT_TAP with the .1 on pin
  4 and CTN6 on pin 3, network rebuilt node by node. Parts list: RTN5, CTN7, roles
  of VR3/VR4/CTN5/CTN6/RTN4 rewritten to what they connect. Source description in
  meta.yaml names all six parts.
- Board: the three capacitors stand at cols 97/99/101 over the 100K slope on the
  bottom row (the .00025's foot on the plate eyelet, the .05's foot sharing the
  slope-foot eyelet, the .1's foot led to it) — the E-FB layout page's own
  arrangement — and the 6800 and .005 move OFF the board to the Bass and Treble
  pots, where that page mounts them. VR3 declares `tap: true`; CTN7.a lands on
  VR3.lug4. verify_layout_nets still PASS (claimed), islands as intended.
- Circuit story: the network described as the sheet draws it, with the correction
  recorded where a reader meets it.
- The gate's DEFECT entry for 6g6b:normal comes off, and the network is declared
  and walked, in the gate commit that follows.

Co-Authored-By: Claude Fable 5.1 <noreply@anthropic.com>
Claude-Session: https://claude.ai/code/session_01KBMfdh37HmCL2iWcBiL5J1
Parts:
- removed C13: 25/50u, symbol cx:C
- removed C2, C3, CDR1: .1u, symbol cx:C
- removed CTN6: .005u, symbol cx:C
- removed RD1: 4.7k 1W, symbol cx:R
- removed RL4B: 100k 5%, symbol cx:R
- removed RM2: 470k, symbol cx:R
- removed RNFB: 56k 1W, symbol cx:R
- removed T3: 125A13A, symbol cx:OT_PP
- removed V3A, V3B, V4B: 7025, symbol cx:TRIODE
- removed VR3: 350k-70k, symbol cx:POT
- added C10: 20u 600V, symbol cx:C
- added CTN5: .05u, symbol cx:C
- added RB1: 1k 1W 5%, symbol cx:R
- added RL3A, RL3B: 100k, symbol cx:R
- added RL4A: 82k 5%, symbol cx:R
- added RM1: 470k, symbol cx:R
- added RPF: 4.7k, symbol cx:R
- added RS5, RS6: 470 1W, symbol cx:R
- added RTN4: 6.8k, symbol cx:R
- added V4A: 7025, symbol cx:TRIODE
- added VR3: 350k-70k tap, symbol cx:POT_TAP
- added VR5: 1M-A, symbol cx:POT
- added VR6: 250k-A · Bass Treble, symbol cx:POT
- added VR7: 25k-L · Presence, symbol cx:POT
- C13: renamed from RB1; value 1k 1W 5% -> 25/50u; symbol cx:R -> cx:C
- C2: renamed from VR7; value 25k-L · Presence -> .1u; symbol cx:POT -> cx:C
- C3: renamed from RS5; value 470 1W -> .1u; symbol cx:R -> cx:C
- CDR1: renamed from RL3A; value 100k -> .1u; symbol cx:R -> cx:C
- CTN6: renamed from V2B; value 7025 -> .005u; symbol cx:TRIODE -> cx:C
- CTN7: renamed from RTN4; value 6.8k -> .1u; symbol cx:R -> cx:C
- RD1: renamed from C10; value 20u 600V -> 4.7k 1W; symbol cx:C -> cx:R
- RL4B: renamed from RL4A; value 82k 5% -> 100k 5%
- RM2: renamed from RL3B; value 100k -> 470k
- RNFB: renamed from RPF; value 4.7k -> 56k 1W
- RTN5: renamed from CTN5; value .05u -> 100k; symbol cx:C -> cx:R
- T3: renamed from RS6; value 470 1W -> 125A13A; symbol cx:R -> cx:OT_PP
- V2B: renamed from VR5; value 1M-A -> 7025; symbol cx:POT -> cx:TRIODE
- V3A: renamed from RM1; value 470k -> 7025; symbol cx:R -> cx:TRIODE
- V3B: renamed from VR6; value 250k-A · Bass Treble -> 7025; symbol cx:POT -> cx:TRIODE
- renumbered V4A to V4B
Connections:
- net BP230: now also RL3A.1, RL3B.1; no longer CDR1.1, RM2.1
- net BP410: now also RL4A.1
- net BP428: now also T3.2 (CT)
- net BP430: now also RS5.2, RS6.2; no longer C3.2, T3.2
- net GND: now also C13.2, CTN6.2, T3.5 (SEC_C), C10.2, RPF.2, RTN4.2, VR5.3, VR6.3, VR7.3; no longer C2.3, CTN7.2, RD1.2, RNFB.2, V2B.3, V3B.3, VR4.2 (W), VR4.3
- net NBIAS: now also C13.1, RB1.2; no longer C13.2
- net SPKR: now also RNFB.1, T3.4 (SEC_H)
- net at RG3A.1, V3A.2 (G), VR2.2 (W): now also RM1.2
- net at C2.2: now also RGL5.1, V5.2 (G1)
- net at CDR1.2: now also VR6.1
- net at V3B.1 (P): now also RM2.1, RL3B.2
- net at RGL6.1, V6.2 (G1): now also C3.2
- net at CTN7.1, RTN5.2: now also CTN5.1; no longer VR4.1
- net at DR3.1 (A), DR6.1 (A), RD1.1: now also C10.1
- net at V5.1 (P): now also T3.1 (PRI_A)
- net at V6.1 (P): now also T3.3 (PRI_B)
- net at CTN4.2: now also VR3.1
- net at V2B.1 (P): now also RL2B.2, RM1.1
- net at RK3A.1: now also V3A.3 (K)
- net at CK2B.1, RK2B.1: now also V2B.3 (K); no longer CTN6.3 (K)
- net at RG2B.1, V2B.2 (G): now also VR5.2 (W); no longer CTN6.2 (G)
- net at RM2.2: now also C1.1
- net at RG3B.1, V3B.2 (G): now also VR6.2 (W)
- net at L1.1: now also RD1.2
- net at C1.2, RG4A.1: now also V4A.2 (G); no longer V4B.2 (G)
- net at RTAIL.1, V4B.3 (K): now also V4A.3 (K)
- net at V6.3 (G2): now also RS6.1; no longer T3.1
- net at RL4B.2, V4B.1 (P): now also C3.1
- net at V5.3 (G2): now also RS5.1; no longer C3.1
- net at RK3B.1: now also V3B.3 (K)
- net at DB1.1 (A): now also RB1.1; no longer C13.1
- net at RG4B.1: now also V4B.2 (G)
- new net: CTN5.2, RTN4.1, VR4.2 (W), VR4.3
- new net: C2.1, RL4A.2, V4A.1 (P)
- new net: RNFB.2, RPF.1, RT2.2, VR7.1
- new net: CDR1.1, RL3A.2, V3A.1 (P)
- new net: VR3.2 (W), VR5.1
- new net: CTN7.2, VR3.4 (T), VR4.1
- new net: CTN6.1, VR3.3
Other:
- note added: "Normal ch. tone network: 100 kΩ slope; 250 pF into the hot lug of a 350 kΩ Treble pot with a 70 kΩ tap; 0.1 µF from the slope foot to that tap, where the 250 kΩ-A Bass rheostat hangs; 0.05 µF from the slope foot to the Bass foot and 6.8 kΩ from there to ground; the Treble pot's cold lug bled to ground through 0.005 µF. Wiper into a 1 MΩ-A Volume pot ahead of V2B. Not modelled in the netlist (cont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"
- note added: "are driven directly as ideal sources in the netlist, printed at their own chart values (see the sources list)."
- note added: "modelled in the netlist (control island)."
- note removed: "Normal ch. tone network: redrawn from the E-FB schematic page — a treble-bleed + bass-leg network feeding a Volume pot ahead of V2B."
- note removed: "are driven directly as ideal sources in netlist.cir, printed at their own chart values (see meta.yaml)."
- note removed: "modelled in netlist.cir (control island)."
- moved on the sheet: RL4B, RM2, RNFB, V4B, VR4
