File: amps/6g6b/schematic.kicad_sch (KiCad schematic)
At the start: 91 parts, among them T1 125P7A, T3 125A13A

Commit message: Fix: 6G6-B board had V3's and V4's triode sections swapped against E-FB, and its sheet carried three floating rail labels
- Section swap, read on the E-FB layout page at native resolution:
  V3 (the Bass channel's later stages): the plate carrying the 100K || .002
  (V3B, reached from the "A" turret) is pin 6, its +1.3 V cathode pin 8 and
  its grid pin 7, off the shielded Treble lead. V3A's +150 V plate is pin 1,
  its grid (the Bass Volume lead) pin 2 and its cathode pin 3.
  V4 (the phase inverter): "+300 V." (the 82k side, V4A) sits on pin 1,
  C1's lower lead lands on pin 2, "+280 V." (100k, V4B) on pin 6, and the
  joined cathodes on 8/3.
  The board had both bottles the other way round. It is re-pinned 1<->6,
  2<->7, 3<->8 with new approach routes (V3A/V4A from the left, V3B round
  the socket's right side). The sheet states the units: unit=2 for V3A and
  V4A, unit=1 for V3B and V4B.
- Floating labels. <BP230> sat 2 mm off the end of its wire and is now on
  it. <BP430> and <BP355> were free-standing legends beside a note, touching
  nothing. This sheet does not draw where they leave the chain, so they are
  now a note in the notes band. The netlist drives both rails directly.
- Gates on 6g6b: check_schematics ok; verify_schematic_nets PASS;
  verify_layout_nets PASS (the unit search takes the swapped assignment);
  sheet-vs-board finds no section swap and nothing on RM1/RM2/C1/V3/V4.
  The rows it still lists (CTN2/CTN3 MISPLACED, C14/RD3 sheet-only) were
  there before this wave.
- Not fixed, reported: the supply chain on this sheet and board contradicts
  E-FB and the netlist header. E-FB runs +430 -> TR2 choke -> B (+428) ->
  4700 1W -> +410 -> 27K 1W -> C (+355). The sheet and board put the 4.7k
  ahead of the choke and hang the 27k between +428 and +410. BOM RD1 says
  "before the choke" too.

Co-Authored-By: Claude Opus 5 (1M context) <noreply@anthropic.com>
Parts:
- V3A, V4A: Basing_unit (none) -> 2
- V3B, V4B: Basing_unit (none) -> 1
Connections:
- net BP230: now also C14.1, RD3.2
Other:
- note added: "BP430 (the 5881 screens) and BP355 (the Normal channel's lane) are not drawn off this chain here; both are driven directly as ideal sources in the netlist, at their own chart values (see the sources list)."
- note removed: "BP430 (5881 screens) and BP355 (Normal ch. recovery) tap the same dropper chain the E-FB drawing shows but were not fully traced at this pass; both"
- note removed: "are driven directly as ideal sources in the netlist, printed at their own chart values (see the sources list)."
Changed lines of the file:
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@@
 (kicad_sch (version 20231120) (generator "circuit-codex")
-  (paper "User" 503.47 445.22)
+  (paper "User" 503.47 449.62)
   (title_block
     (title "6G6-B — Blonde Bassman-style")
@@
     (in_bom yes) (on_board yes)
     (property "Reference" "V3A" (at 245.59 145.605 0) (effects (font (size 1.27 1.27)) (justify left)))
-    (property "Value" "7025" (at 245.59 148.005 0) (effects (font (size 1.27 1.27)) (justify left))))
+    (property "Value" "7025" (at 245.59 148.005 0) (effects (font (size 1.27 1.27)) (justify left)))
+    (property "Basing_unit" "2" (at 245.59 150.405 0) (effects (font (size 1.27 1.27)) hide)))
   (wire (pts (xy 224.59 152.005) (xy 228.16 152.005))
     (stroke (width 0) (type default)))
@@
     (in_bom yes) (on_board yes)
     (property "Reference" "V3B" (at 301.59 145.605 0) (effects (font (size 1.27 1.27)) (justify left)))
-    (property "Value" "7025" (at 301.59 148.005 0) (effects (font (size 1.27 1.27)) (justify left))))
+    (property "Value" "7025" (at 301.59 148.005 0) (effects (font (size 1.27 1.27)) (justify left)))
+    (property "Basing_unit" "1" (at 301.59 150.405 0) (effects (font (size 1.27 1.27)) hide)))
   (wire (pts (xy 276.67 144.715) (xy 283.59 144.715))
     (stroke (width 0) (type default)))
@@
     (in_bom yes) (on_board yes)
     (property "Reference" "V4A" (at 353.59 193.605 0) (effects (font (size 1.27 1.27)) (justify left)))
-    (property "Value" "7025" (at 353.59 196.005 0) (effects (font (size 1.27 1.27)) (justify left))))
+    (property "Value" "7025" (at 353.59 196.005 0) (effects (font (size 1.27 1.27)) (justify left)))
+    (property "Basing_unit" "2" (at 353.59 198.405 0) (effects (font (size 1.27 1.27)) hide)))
   (wire (pts (xy 339.59 140.905) (xy 339.59 200.005))
     (stroke (width 0) (type default)))
@@
     (in_bom yes) (on_board yes)
     (property "Reference" "V4B" (at 353.59 229.605 0) (effects (font (size 1.27 1.27)) (justify left)))
-    (property "Value" "7025" (at 353.59 232.005 0) (effects (font (size 1.27 1.27)) (justify left))))
+    (property "Value" "7025" (at 353.59 232.005 0) (effects (font (size 1.27 1.27)) (justify left)))
+    (property "Basing_unit" "1" (at 353.59 234.405 0) (effects (font (size 1.27 1.27)) hide)))
   (wire (pts (xy 347.59 192.385) (xy 347.59 188.905))
     (stroke (width 0) (type default)))
@@
   (wire (pts (xy 175.59 372.005) (xy 181.59 372.005))
     (stroke (width 0) (type default)))
-  (wire (pts (xy 181.59 372.005) (xy 187.59 372.005))
+  (wire (pts (xy 181.59 372.005) (xy 189.59 372.005))
     (stroke (width 0) (type default)))
   (global_label "BP230" (shape input) (at 189.59 372.005 0)
-    (effects (font (size 1.27 1.27)) (justify left)))
-  (text "BP430 (5881 screens) and BP355 (Normal ch. recovery) tap the same dropper chain the E-FB drawing shows but were not fully traced at this pass; both" (at 19.59 320.005 0)
-    (effects (font (size 1.15 1.15)) (justify left)))
-  (text "are driven directly as ideal sources in the netlist, printed at their own chart values (see the sources list)." (at 19.59 323.505 0)
-    (effects (font (size 1.15 1.15)) (justify left)))
-  (global_label "BP430" (shape input) (at 29.59 340.005 0)
-    (effects (font (size 1.27 1.27)) (justify left)))
-  (global_label "BP355" (shape input) (at 29.59 346.005 0)
     (effects (font (size 1.27 1.27)) (justify left)))
   (global_label "HT_TAP" (shape input) (at 219.59 300.005 180)
@@
   (text "3" (at 190.44 136.355 0)
     (effects (font (size 1.1 1.1)) (justify left)))
-  (text "6" (at 240.44 145.655 0)
-    (effects (font (size 1.1 1.1)) (justify left)))
-  (text "7" (at 232.643 150.605 0)
-    (effects (font (size 1.1 1.1)) (justify left)))
-  (text "8" (at 240.44 158.355 0)
-    (effects (font (size 1.1 1.1)) (justify left)))
-  (text "1" (at 296.44 145.655 0)
-    (effects (font (size 1.1 1.1)) (justify left)))
-  (text "2" (at 288.643 150.605 0)
-    (effects (font (size 1.1 1.1)) (justify left)))
-  (text "3" (at 296.44 158.355 0)
-    (effects (font (size 1.1 1.1)) (justify left)))
-  (text "6" (at 348.44 193.655 0)
-    (effects (font (size 1.1 1.1)) (justify left)))
-  (text "7" (at 340.643 198.605 0)
-    (effects (font (size 1.1 1.1)) (justify left)))
-  (text "8" (at 349.89 206.355 0)
-    (effects (font (size 1.1 1.1)) (justify left)))
-  (text "1" (at 348.44 229.655 0)
-    (effects (font (size 1.1 1.1)) (justify left)))
-  (text "2" (at 340.643 234.605 0)
-    (effects (font (size 1.1 1.1)) (justify left)))
-  (text "3" (at 348.44 242.355 0)
+  (text "1" (at 240.44 145.655 0)
+    (effects (font (size 1.1 1.1)) (justify left)))
+  (text "2" (at 232.643 150.605 0)
+    (effects (font (size 1.1 1.1)) (justify left)))
+  (text "3" (at 240.44 158.355 0)
+    (effects (font (size 1.1 1.1)) (justify left)))
+  (text "6" (at 296.44 145.655 0)
+    (effects (font (size 1.1 1.1)) (justify left)))
+  (text "7" (at 288.643 150.605 0)
+    (effects (font (size 1.1 1.1)) (justify left)))
+  (text "8" (at 296.44 158.355 0)
+    (effects (font (size 1.1 1.1)) (justify left)))
+  (text "1" (at 348.44 193.655 0)
+    (effects (font (size 1.1 1.1)) (justify left)))
+  (text "2" (at 340.643 198.605 0)
+    (effects (font (size 1.1 1.1)) (justify left)))
+  (text "3" (at 349.89 206.355 0)
+    (effects (font (size 1.1 1.1)) (justify left)))
+  (text "6" (at 348.44 229.655 0)
+    (effects (font (size 1.1 1.1)) (justify left)))
+  (text "7" (at 340.643 234.605 0)
+    (effects (font (size 1.1 1.1)) (justify left)))
+  (text "8" (at 348.44 242.355 0)
     (effects (font (size 1.1 1.1)) (justify left)))
   (text "3" (at 420.44 193.02 0)
@@
   (text "Power — universal power transformer (TR1, 125P7A), centre-tapped HT winding; two 3-diode series legs form a silicon full-wave bridge (no rectifier tube); 20 uF/600V filters either side of the choke (TR2, 125C1A); 4.7 k/1 W and 27 k/1 W droppers feed the driver and preamp taps." (at 12.7 399.583 0)
     (effects (font (size 1.2 1.2)) (justify left)))
-  (text "Two full channels (Bass, Normal), each with its own Bass/Treble/Volume tone network, mixing through a 470k from each at the node that feeds a long-tailed-pair phase inverter, ahead of a fixed-bias 5881 pair off a solid-state bridge — no rectifier tube." (at 12.7 403.983 0)
+  (text "BP430 (the 5881 screens) and BP355 (the Normal channel's lane) are not drawn off this chain here; both are driven directly as ideal sources in the netlist, at their own chart values (see the sources list)." (at 12.7 403.983 0)
     (effects (font (size 1.2 1.2)) (justify left)))
-  (text "The Bass channel runs on through V3 (V3A -> its own Treble control VR6 -> V3B) before it meets the Normal channel at MIX. Heaters, PT primary, ground switch, fuse and standby switch omitted." (at 12.7 408.383 0)
+  (text "Two full channels (Bass, Normal), each with its own Bass/Treble/Volume tone network, mixing through a 470k from each at the node that feeds a long-tailed-pair phase inverter, ahead of a fixed-bias 5881 pair off a solid-state bridge — no rectifier tube." (at 12.7 408.383 0)
+    (effects (font (size 1.2 1.2)) (justify left)))
+  (text "The Bass channel runs on through V3 (V3A -> its own Treble control VR6 -> V3B) before it meets the Normal channel at MIX. Heaters, PT primary, ground switch, fuse and standby switch omitted." (at 12.7 412.783 0)
     (effects (font (size 1.2 1.2)) (justify left)))
   (sheet_instances (path "/" (page "1")))

Commit message: Fix: 6G6-B supply chain — dropper order, off-board supply parts, and the swapped plate/screen nodes
The E-FB schematic page runs its B+ chain reservoir (+430 V, two 20 uF cans)
-> choke TR2 -> node B (+428 V) -> 4700 1W -> +410 V -> 27k 1W -> +355 V,
with the 56k 1W to the Bass row's +230 V lane hanging off node B. Read again
at 300 dpi, lug by lug. Three things were wrong here.

1. Order. The sheet and the board drew the 4.7k BEFORE the choke and ran the
   27k from node B to +410 V, leaving the +355 V lane off the chain entirely
   — even though notes.md, meta.yaml's source read and RD2's own parts-list
   role all had the chain right. Both drawings now follow the page.

2. Derivation. netlist.cir drove all five rails as ideal sources. Only the
   two ends of the choke are driven now (the drawing prints no choke DCR and
   no rectifier source impedance); +410, +355 and +230 are derived through
   the drawn droppers and gated against the printed chart. They land at
   407.0, 355.0 and 236.5 V — 0.7%, 0.0% and 2.8% off.

3. Plates and screens were the wrong way round. The "+430 V." lead goes UP
   to the output transformer's primary centre tap, so the 5881 plates hang
   on the reservoir node and the +428 V printed at their leads is the
   primary's own DCR; the "+428 V." lead comes DOWN from the two 470 ohm
   screen stoppers to node B, the node the droppers also leave from. The
   corpus had the plates on +428 and the screens on +430, which ran the
   whole output current through the choke. The arithmetic agrees with the
   read: 2 V over the ~17 mA a screens-plus-preamp load draws is about
   120 ohms, which is a 125C1A; over 70 mA of plate current it would be 28.

Board: the layout page draws the bias sub-board and the two three-diode
rectifier legs and nothing else of the supply — no cans, no choke, no
droppers — so C10/C11/C12/C14/C15/L1 come off the board as net_map
not_on_board entries and RD1/RD2/RD3 as netlist_unplaced, with each B+ lane
anchored where its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
Parts:
- added C15: 20u 600V, symbol cx:C
Connections:
- net BP355: now also RD2.2, C15.1
- net BP410: now also RD1.2, RD2.1; no longer RD2.2
- net BP428: now also RD1.1, RS5.2, RS6.2; no longer RD2.1, T3.2 (CT)
- net BP430: now also C10.1, DR3.2 (K), DR6.2 (K), L1.1, T3.2 (CT); no longer RS5.2, RS6.2
- net GND: now also C15.2
Other:
- note added: "Bias supply: silicon diode off an AC tap through a 1 k/1 W, with a 27 k bleeder and a dual 25/50 uF can -> -54 V."
- note added: "Both ends of the choke are driven at their printed figures — the +430 V reservoir, which is also the output transformer's primary centre tap, and node B at +428 V, which feeds the 5881 screen stoppers; the +410 V, +355 V and +230 V lanes are derived through the droppers drawn here and checked against the printed chart. The standby switch between the rectifier and the +430 V node is omitted, so th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"
- note added: "Normal channel and the Bass row all begin."
- note added: "Power — universal power transformer (TR1, 125P7A), centre-tapped HT winding; two 3-diode series legs form a silicon full-wave bridge (no rectifier tube); a 20 uF/600 V filter on every node of the chain, two of them in parallel at the reservoir. The reservoir node also feeds the output transformer primary centre tap, so the 5881 plates hang on it; the choke (TR2, 125C1A) carries it on to node B, w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"
- note removed: "BP430 (the 5881 screens) and BP355 (the Normal channel's lane) are not drawn off this chain here; both are driven directly as ideal sources in the netlist, at their own chart values (see the sources list)."
- note removed: "Bias supply: silicon diode off an AC tap, 1 k/4.7 k dropping through the choke, 27 k bleeder, dual 25/50 uF can -> -54 V."
- note removed: "Power — universal power transformer (TR1, 125P7A), centre-tapped HT winding; two 3-diode series legs form a silicon full-wave bridge (no rectifier tube); 20 uF/600V filters either side of the choke (TR2, 125C1A); 4.7 k/1 W and 27 k/1 W droppers feed the driver and preamp taps."
