File: amps/6g4/schematic.kicad_sch (KiCad schematic)
At the start: 78 parts, among them T1 8087, T2 45216

Commit message: Fix: 6G4 tone network redrawn from the A-FJ sheet — coupler, bass capacitor, a Bass DIVIDER, and the 47MM bright cap
- The sheet draws, per channel: .05 from the input-stage plate into the network;
  250MM to the Treble pot's hot lug and 100K to the slope foot, where the pot's
  cold lug also sits; the 250K-A Bass pot as a DIVIDER from the slope foot to
  ground, .01 across its upper section (hot lug to wiper) and 10K across its
  lower (wiper to ground); the Treble wiper into a 500K-L Volume pot with 47MM
  from its hot lug to its wiper.
- The drawing had neither capacitor, took the 100K straight off the plate — a
  DC path to ground through the stack on the sheet — and strapped the Bass pot
  as a rheostat above the 10K. Checked separately: netlist.cir never carried
  that path (the recovery grid returns through a 1 M leak), so no operating
  point moves; verify_amps 41/0 and op-points.yaml unchanged. Both channels.
- Beyond the brief, read off the same crop: the 47 pF bright capacitor across
  each Volume pot, in no parts list until now (CBR1/CBR2).
- Parts list: CC1T/CC2T .05, CB1T/CB2T .01, CBR1/CBR2 47 pF added; roles of the
  slope, foot and pots rewritten to what they connect. Source description in
  meta.yaml names the whole network.
- Board: the coupler stands on the board at the plate eyelet; the other parts
  hang at the pots where the A-FJ layout page mounts them (kind: part beside
  each control), wired lug to lug; the control groups re-spaced to fit and the
  Volume wipers now reach the recovery grids. Leads fanned by the route helper
  to zero lint findings.
- Sheet notes in visitor voice (no repo file names).
- Declared and walked by the gate in the commit that follows.

Co-Authored-By: Claude Fable 5.1 <noreply@anthropic.com>
Claude-Session: https://claude.ai/code/session_01KBMfdh37HmCL2iWcBiL5J1
Parts:
- removed R1b: 68k, symbol cx:R
- removed RINT: 220k, symbol cx:R
- removed RK1D: 820, symbol cx:R
- removed RS2: 470 1W, symbol cx:R
- removed V2A, V5A: 7025, symbol cx:TRIODE
- removed VRINT: 10M-RA intensity, symbol cx:POT
- removed VRSPD: 4M-RA speed, symbol cx:POT
- removed VRV2: 500k-L vol, symbol cx:POT
- added CB1T, CB2T: .01u, symbol cx:C
- added CBR1, CBR2: 47p, symbol cx:C
- added CC2T: .05u, symbol cx:C
- added CK1D: 25u, symbol cx:C
- added CT1: 250p, symbol cx:C
- added RK2I: 1.5k, symbol cx:R
- added RLPA: 82k 5%, symbol cx:R
- added RM1: 6.8k, symbol cx:R
- added RTAIL: 820 5%, symbol cx:R
- added RTO1: 100k, symbol cx:R
- added RTOFB: 4.7M, symbol cx:R
- added T1: 8087, symbol cx:PT
- added V5B: 7025, symbol cx:TRIODE
- CC1T: renamed from CT1; value 250p -> .05u
- R1b: renamed from RG2I; value 1M -> 68k
- RG2I: renamed from RK2I; value 1.5k -> 1M
- RINT: renamed from V5B; value 7025 -> 220k; symbol cx:TRIODE -> cx:R
- RK1D: renamed from RM1; value 6.8k -> 820
- RK2D: renamed from RTO1; value 100k -> 820
- RS2: renamed from T1; value 8087 -> 470 1W; symbol cx:PT -> cx:R
- V2A: renamed from CK1D; value 25u -> 7025; symbol cx:C -> cx:TRIODE
- V5A: renamed from RTAIL; value 820 5% -> 7025; symbol cx:R -> cx:TRIODE
- VRINT: renamed from RLPA; value 82k 5% -> 10M-RA intensity; symbol cx:R -> cx:POT
- VRSPD: renamed from RTOFB; value 4.7M -> 4M-RA speed; symbol cx:R -> cx:POT
- VRV2: renamed from RK2D; value 820 -> 500k-L vol; symbol cx:R -> cx:POT
Connections:
- net BC: now also RLPA.1; no longer VRINT.1
- net BP1: now also RS2.2, RTO1.1; no longer RK2D.1
- net CH2 IN 1: now also R1b.1
- net GND: now also RK1D.2, RK2D.2, VRB1.3, VRB2.3, VRINT.1, VRSPD.3, VRV2.3, CK1D.2, RK2I.2, RTOFB.2, T1.4 (HT_CT); no longer R1b.2, RS2.4 (HT_CT), V2A.2, VRV2.2
- net GPIA: now also V5A.2 (G), RM1.2; no longer RK1D.2
- net HT_A: now also T1.3 (HT_A); no longer RS2.3 (HT_A)
- net HT_B: now also T1.5 (HT_B); no longer RS2.5 (HT_B)
- net MAINS: now also T1.1 (PRI_1), T1.2 (PRI_2); no longer RS2.1 (PRI_1), RS2.2 (PRI_2)
- net NBIAS: now also VRINT.2 (W)
- net at CC1T.1, RL1I.2, V1.1 (P): no longer RS1T.1
- net at CTO1.2, CTO2.1: now also VRSPD.1
- net at CTO1.1, V2B.1 (P): now also RINT.2, RTO1.2; no longer RK2D.2
- net at CTOFB.2, V2B.2 (G): now also RTOFB.1; no longer VRSPD.1
- net at RGPA.2, RGPB.1, RT2.2: now also RTAIL.1; no longer V5A.1
- net at VRT2.2 (W): now also VRV2.1, CBR2.1
- net at V4.2 (G): now also VRV2.2 (W), CBR2.2
- net at RS1T.2, VRB1.1, VRT1.3: now also CB1T.1; no longer VRB1.2 (W)
- net at RSL1.1: now also VRB1.2 (W), CB1T.2; no longer VRB1.3
- net at RL2I.2, V3.1 (P): now also CC2T.1; no longer CT2.1, RS2T.1
- net at RGPB.2: now also V5B.2 (G); no longer RINT.2 (G)
- net at CK2D.1, V4.3 (K): now also RK2D.1; no longer VRV2.1
- net at V2A.1 (P): now also CC1D.1, RL1D.2
- net at CC1T.2: now also RS1T.1, CT1.1; no longer VRT1.1
- net at RK1D.1: now also V2A.3 (K), CK1D.1; no longer CC1D.2
- net at RS2T.2, VRB2.1, VRT2.3: now also CB2T.1; no longer VRB2.2 (W)
- net at C2.1, RLPB.2: now also V5B.1 (P); no longer RINT.1 (P)
- net at R2b.2, V3.2 (G): now also R1b.2, RG2I.1; no longer R1b.1
- net at VRV1.2 (W): now also V2A.2 (G), CBR1.2
- net at C1.1: now also V5A.1 (P), RLPA.2; no longer VRINT.2
- net at CK2I.1, V3.3 (K): now also RK2I.1; no longer RG2I.1
- net at V8.3 (G2): now also RS2.1
- net at RSL2.1: now also VRB2.2 (W), CB2T.2; no longer VRB2.3
- net at VRT1.2 (W), VRV1.1: now also CBR1.1
- new net: CT1.2, VRT1.1
- new net: RTAIL.2, V5A.3 (K), V5B.3 (K)
- new net: CC1D.2, RM1.1
- new net: RINT.1, VRINT.3
- new net: CC2T.2, CT2.1, RS2T.1
Other:
- note added: "BD/BE1/BE2 (preamp rails) are calibrated ideal sources in the netlist — the drawing's own dropper chain into them was not legible (see the circuit story); only CH1 is a named part in the parts list."
- note added: "C10 stands for the drawing's several HT filter cans; per-node values were not fully resolved at this scan's resolution (see the parts list)"
- note added: "Excluded from the netlist — a running oscillator has no static operating point (see the circuit story)"
- note added: "Heaters, PT primary/mains, pilot lamp and the vibrato-pedal jack's switching are omitted here — see the netlist, the sources list and the board drawing. Bottles are 7025, a low-noise 12AX7 (an alias of the same valve)."
- note removed: "BD/BE1/BE2 (preamp rails) are calibrated ideal sources in netlist.cir — the drawing's own dropper chain into them was not legible (notes.md); only CH1 is a named bom.yaml part."
- note removed: "C10 stands for the drawing's several HT filter cans; per-node values were not fully resolved at this scan's resolution (see bom.yaml)"
- note removed: "Excluded from netlist.cir — a running oscillator has no static operating point (notes.md)"
- note removed: "Heaters, PT primary/mains, pilot lamp and the vibrato-pedal jack's switching are omitted here — see netlist.cir, meta.yaml, layout.yaml. Bottles are 7025, a low-noise 12AX7 (also_known_as)."
- moved on the sheet: CC1T, CK1I, R1a, R1b, R2a, RG1I, RG2I, RK1D, RK1I, RK2D, RL1I, V1

Commit message: Fix: six sheets letter valve sections and bias rows the way their factory drawings do
Sections — the board was right and the sheet printed the other half's pin
numbers (triage verdict rows, crops under the triage scratch):
  AC30 V1    JMI OS/065 (3600x2492): Brilliant grid 2 / plate 1, Normal 7 / 6
  AA964 V1   input 2/1/3, second stage 7/6/8 (6322x3926)
  AA964 V2   phase inverter 7/6/8, tremolo oscillator 2/1/3
  5F6-A V3   the 82k (input) triode on 1/2/3 on the I-EG layout (6402x3641)
  6G4 V5     the 82k triode on 1/2/3 on the A-FJ layout (2250x1269, the only copy)

Bias rows — the 5F4 (C-EG) and 5E4-A (G-EE) drawings run the series
resistor (6800 / 18K) from the transformer's bias tap INTO the selenium
rectifier. The previous commit's rows put the rectifier on the tap and the
resistor after it; both now read tap -> resistor -> rectifier -> node. The
5F4 rectifier sits clear of C17's ground flag.

Worklist after re-export: section swaps 10 -> 5 (three board re-pins in
flight, the 5E5-A whose only copy does not resolve, and the AA1164 V4 still
being read); the 5F4/5E4-A D1 rows stay MISPLACED until their boards take
the tap lead, which the board repair wave is adding.

Gates: check_schematics 40/0 (+selftest), verify_schematic_nets 40 clean,
tone gate, validate, check_value_consistency --strict 0, test_era_values,
verify_sheet_vs_board selftest 19 + drift clean after --export,
check_heaters, verify_layout_nets; regenerating every sheet changes only
these six.

Co-Authored-By: Claude Opus 5 (1M context) <noreply@anthropic.com>
Claude-Session: https://claude.ai/code/session_01KBMfdh37HmCL2iWcBiL5J1
Parts:
- V5A: Basing_unit (none) -> 2
- V5B: Basing_unit (none) -> 1
Changed lines of the file:
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@@
     (in_bom yes) (on_board yes)
     (property "Reference" "V5A" (at 275.336 80.489 0) (effects (font (size 1.27 1.27)) (justify left)))
-    (property "Value" "7025" (at 275.336 82.889 0) (effects (font (size 1.27 1.27)) (justify left))))
+    (property "Value" "7025" (at 275.336 82.889 0) (effects (font (size 1.27 1.27)) (justify left)))
+    (property "Basing_unit" "2" (at 275.336 85.289 0) (effects (font (size 1.27 1.27)) hide)))
   (symbol (lib_id "cx:TRIODE") (at 269.336 136.889 0) (unit 1)
     (in_bom yes) (on_board yes)
     (property "Reference" "V5B" (at 275.336 130.489 0) (effects (font (size 1.27 1.27)) (justify left)))
-    (property "Value" "7025" (at 275.336 132.889 0) (effects (font (size 1.27 1.27)) (justify left))))
+    (property "Value" "7025" (at 275.336 132.889 0) (effects (font (size 1.27 1.27)) (justify left)))
+    (property "Basing_unit" "1" (at 275.336 135.289 0) (effects (font (size 1.27 1.27)) hide)))
   (wire (pts (xy 269.336 79.269) (xy 269.336 75.789))
     (stroke (width 0) (type default)))
@@
   (text "3" (at 186.186 93.239 0)
     (effects (font (size 1.1 1.1)) (justify left)))
-  (text "6" (at 270.186 80.539 0)
-    (effects (font (size 1.1 1.1)) (justify left)))
-  (text "7" (at 262.389 85.489 0)
-    (effects (font (size 1.1 1.1)) (justify left)))
-  (text "8" (at 270.186 93.239 0)
-    (effects (font (size 1.1 1.1)) (justify left)))
-  (text "1" (at 270.186 130.539 0)
-    (effects (font (size 1.1 1.1)) (justify left)))
-  (text "2" (at 262.389 135.489 0)
-    (effects (font (size 1.1 1.1)) (justify left)))
-  (text "3" (at 270.186 143.239 0)
+  (text "1" (at 270.186 80.539 0)
+    (effects (font (size 1.1 1.1)) (justify left)))
+  (text "2" (at 262.389 85.489 0)
+    (effects (font (size 1.1 1.1)) (justify left)))
+  (text "3" (at 270.186 93.239 0)
+    (effects (font (size 1.1 1.1)) (justify left)))
+  (text "6" (at 270.186 130.539 0)
+    (effects (font (size 1.1 1.1)) (justify left)))
+  (text "7" (at 262.389 135.489 0)
+    (effects (font (size 1.1 1.1)) (justify left)))
+  (text "8" (at 270.186 143.239 0)
     (effects (font (size 1.1 1.1)) (justify left)))
   (text "3" (at 334.186 59.904 0)
