File: amps/ab165/schematic.kicad_sch (KiCad schematic)
At the start: 105 parts

Commit message: Fix: state the datasheet unit on 17 dual-triode sections whose sheets printed the other half's pin numbers
The sheet-vs-board gate reported these sockets as SECTION-SWAP; the
2026-09-10 source-read triage found the BOARD right on every one of them
(and both surfaces wrong on the 5G9 tremolo bottle). Each sheet had
lettered the section on the default map (A -> unit 1 -> pins 6/7/8) where
the factory drawing puts that stage on 1/2/3. The draw scripts now state
`unit=` on both halves, with the source cited beside the call, so the
printed socket numbers are the factory's:

- 5f4 V3: driver V3A -> 1/2/3, cathodyne V3B -> 6/7/8
  (crop 5f4-V3-layout-trace.png: +213 V driver plate -> pin 1, +270 V -> 6)
- 5f8a V3: 82k half V3A -> 1/2/3, 100k half V3B -> 6/7/8
  (crop 5f8a-V3-layout-trace.png: +225 -> 6, +19 -> 2, +28.5 -> 8)
- 6161 V1: channel 1 V1A -> 1/2/3 (crop 6161-V1-ch1.png prints 1/2/3);
  6161 V2: 1 MEG-grid half V2A -> 1/2/3, paraphase V2B -> 6/7/8
  (crop 6161-V2.png / 6161-V2-right.png)
- 6g3 V3: 82k half V3A -> 1/2/3 (crop 6g3-V3-layout-wires.png: +230 -> 1,
  +225 -> 6, +20 -> 7)
- aa1164 V3: recovery V3A -> 1/2/3, mixer V3B -> 6/7/8
  (crops aa1164-V3A-recovery-schem.png, aa1164-V3B-mixer-schem.png)
- aa864-bassman V1/V2: input stages 2/1/3, second stages 7/6/8; V4: the
  .1/500 pF-fed 82k half 2/1/3 (crops aa864-V1A-input.png,
  aa864-V1B-second.png, aa864-V2A-input.png, aa864-V2B-second.png,
  aa864-V4-PI.png)
- ab165 V1/V2/V4: same pattern (crops ab165-V1A-input.png,
  ab165-V1B-second.png, ab165-V2A-input.png, ab165-V2B-second.png,
  ab165-V4-PI.png)
- ab763-super V1/V2: slope-plate +270 V -> pin 1 (input stage), .047
  plate -> 6 (crops ab763-super-V1-layout-sh.png, ab763-super-V2-layout-sh.png)
- dr103 V2/V3: gain stages 6/7/8, cathode followers 1/2/3 (crops
  dr103-V2-huss.png, dr103-V3-huss.png — the Huss redraw, not a factory
  print; noted in the script)
- 5g9 V3: oscillator V3A -> 1/2/3, follower V3B -> 6/7/8 (crops
  5g9-V3-strap71-zoom.png, 5g9-V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
Parts:
- V1A, V2A, V4A: Basing_unit (none) -> 2
- V1B, V2B, V4B: Basing_unit (none) -> 1
Changed lines of the file:
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@@
     (in_bom yes) (on_board yes)
     (property "Reference" "V1A" (at 72.7452 39.42 0) (effects (font (size 1.27 1.27)) (justify left)))
-    (property "Value" "12AX7 (7025)" (at 72.7452 41.82 0) (effects (font (size 1.27 1.27)) (justify left))))
+    (property "Value" "12AX7 (7025)" (at 72.7452 41.82 0) (effects (font (size 1.27 1.27)) (justify left)))
+    (property "Basing_unit" "2" (at 72.7452 44.22 0) (effects (font (size 1.27 1.27)) hide)))
   (wire (pts (xy 54.7452 45.82) (xy 59.1252 45.82))
     (stroke (width 0) (type default)))
@@
     (in_bom yes) (on_board yes)
     (property "Reference" "V1B" (at 156.745 39.42 0) (effects (font (size 1.27 1.27)) (justify left)))
-    (property "Value" "12AX7 (7025)" (at 156.745 41.82 0) (effects (font (size 1.27 1.27)) (justify left))))
+    (property "Value" "12AX7 (7025)" (at 156.745 41.82 0) (effects (font (size 1.27 1.27)) (justify left)))
+    (property "Basing_unit" "1" (at 156.745 44.22 0) (effects (font (size 1.27 1.27)) hide)))
   (wire (pts (xy 138.745 45.82) (xy 143.125 45.82))
     (stroke (width 0) (type default)))
@@
     (in_bom yes) (on_board yes)
     (property "Reference" "V2A" (at 72.7452 93.42 0) (effects (font (size 1.27 1.27)) (justify left)))
-    (property "Value" "12AX7 (7025)" (at 72.7452 95.82 0) (effects (font (size 1.27 1.27)) (justify left))))
+    (property "Value" "12AX7 (7025)" (at 72.7452 95.82 0) (effects (font (size 1.27 1.27)) (justify left)))
+    (property "Basing_unit" "2" (at 72.7452 98.22 0) (effects (font (size 1.27 1.27)) hide)))
   (wire (pts (xy 54.7452 99.82) (xy 59.1252 99.82))
     (stroke (width 0) (type default)))
@@
     (in_bom yes) (on_board yes)
     (property "Reference" "V2B" (at 156.745 93.42 0) (effects (font (size 1.27 1.27)) (justify left)))
-    (property "Value" "12AX7 (7025)" (at 156.745 95.82 0) (effects (font (size 1.27 1.27)) (justify left))))
+    (property "Value" "12AX7 (7025)" (at 156.745 95.82 0) (effects (font (size 1.27 1.27)) (justify left)))
+    (property "Basing_unit" "1" (at 156.745 98.22 0) (effects (font (size 1.27 1.27)) hide)))
   (wire (pts (xy 138.745 99.82) (xy 143.125 99.82))
     (stroke (width 0) (type default)))
@@
     (in_bom yes) (on_board yes)
     (property "Reference" "V4A" (at 278.745 39.42 0) (effects (font (size 1.27 1.27)) (justify left)))
-    (property "Value" "12AT7" (at 278.745 41.82 0) (effects (font (size 1.27 1.27)) (justify left))))
+    (property "Value" "12AT7" (at 278.745 41.82 0) (effects (font (size 1.27 1.27)) (justify left)))
+    (property "Basing_unit" "2" (at 278.745 44.22 0) (effects (font (size 1.27 1.27)) hide)))
   (symbol (lib_id "cx:TRIODE") (at 272.745 83.82 0) (unit 1)
     (in_bom yes) (on_board yes)
     (property "Reference" "V4B" (at 278.745 77.42 0) (effects (font (size 1.27 1.27)) (justify left)))
-    (property "Value" "12AT7" (at 278.745 79.82 0) (effects (font (size 1.27 1.27)) (justify left))))
+    (property "Value" "12AT7" (at 278.745 79.82 0) (effects (font (size 1.27 1.27)) (justify left)))
+    (property "Basing_unit" "1" (at 278.745 82.22 0) (effects (font (size 1.27 1.27)) hide)))
   (wire (pts (xy 272.745 38.2) (xy 272.745 34.72))
     (stroke (width 0) (type default)))
@@
   (global_label "-45V B" (shape input) (at 154.745 231.82 90)
     (effects (font (size 1.27 1.27)) (justify left)))
-  (text "6" (at 67.5952 39.47 0)
-    (effects (font (size 1.1 1.1)) (justify left)))
-  (text "7" (at 59.798 44.42 0)
-    (effects (font (size 1.1 1.1)) (justify left)))
-  (text "8" (at 67.5952 52.17 0)
-    (effects (font (size 1.1 1.1)) (justify left)))
-  (text "1" (at 151.595 39.47 0)
-    (effects (font (size 1.1 1.1)) (justify left)))
-  (text "2" (at 143.798 44.42 0)
-    (effects (font (size 1.1 1.1)) (justify left)))
-  (text "3" (at 151.595 52.17 0)
-    (effects (font (size 1.1 1.1)) (justify left)))
-  (text "6" (at 67.5952 93.47 0)
-    (effects (font (size 1.1 1.1)) (justify left)))
-  (text "7" (at 59.798 98.42 0)
-    (effects (font (size 1.1 1.1)) (justify left)))
-  (text "8" (at 67.5952 106.17 0)
-    (effects (font (size 1.1 1.1)) (justify left)))
-  (text "1" (at 151.595 93.47 0)
-    (effects (font (size 1.1 1.1)) (justify left)))
-  (text "2" (at 143.798 98.42 0)
-    (effects (font (size 1.1 1.1)) (justify left)))
-  (text "3" (at 151.595 106.17 0)
+  (text "1" (at 67.5952 39.47 0)
+    (effects (font (size 1.1 1.1)) (justify left)))
+  (text "2" (at 59.798 44.42 0)
+    (effects (font (size 1.1 1.1)) (justify left)))
+  (text "3" (at 67.5952 52.17 0)
+    (effects (font (size 1.1 1.1)) (justify left)))
+  (text "6" (at 151.595 39.47 0)
+    (effects (font (size 1.1 1.1)) (justify left)))
+  (text "7" (at 143.798 44.42 0)
+    (effects (font (size 1.1 1.1)) (justify left)))
+  (text "8" (at 151.595 52.17 0)
+    (effects (font (size 1.1 1.1)) (justify left)))
+  (text "1" (at 67.5952 93.47 0)
+    (effects (font (size 1.1 1.1)) (justify left)))
+  (text "2" (at 59.798 98.42 0)
+    (effects (font (size 1.1 1.1)) (justify left)))
+  (text "3" (at 67.5952 106.17 0)
+    (effects (font (size 1.1 1.1)) (justify left)))
+  (text "6" (at 151.595 93.47 0)
+    (effects (font (size 1.1 1.1)) (justify left)))
+  (text "7" (at 143.798 98.42 0)
+    (effects (font (size 1.1 1.1)) (justify left)))
+  (text "8" (at 151.595 106.17 0)
     (effects (font (size 1.1 1.1)) (justify left)))
   (text "1" (at 217.595 66.47 0)
@@
   (text "3" (at 217.595 79.17 0)
     (effects (font (size 1.1 1.1)) (justify left)))
-  (text "6" (at 273.595 39.47 0)
-    (effects (font (size 1.1 1.1)) (justify left)))
-  (text "7" (at 265.798 44.42 0)
-    (effects (font (size 1.1 1.1)) (justify left)))
-  (text "8" (at 273.595 52.17 0)
-    (effects (font (size 1.1 1.1)) (justify left)))
-  (text "1" (at 273.595 77.47 0)
-    (effects (font (size 1.1 1.1)) (justify left)))
-  (text "2" (at 265.798 82.42 0)
-    (effects (font (size 1.1 1.1)) (justify left)))
-  (text "3" (at 273.595 90.17 0)
+  (text "1" (at 273.595 39.47 0)
+    (effects (font (size 1.1 1.1)) (justify left)))
+  (text "2" (at 265.798 44.42 0)
+    (effects (font (size 1.1 1.1)) (justify left)))
+  (text "3" (at 273.595 52.17 0)
+    (effects (font (size 1.1 1.1)) (justify left)))
+  (text "6" (at 273.595 77.47 0)
+    (effects (font (size 1.1 1.1)) (justify left)))
+  (text "7" (at 265.798 82.42 0)
+    (effects (font (size 1.1 1.1)) (justify left)))
+  (text "8" (at 273.595 90.17 0)
     (effects (font (size 1.1 1.1)) (justify left)))
   (text "3" (at 335.595 34.835 0)

Commit message: Fix: the AB165 and AA864 sheets shorted the mains primary by lettering both cord conductors alike
Both claimed sheets lettered the two conductors of the mains cord with one
global-label name ("MAINS" on the AB165, "AC LINE" on the AA864). A label's
name is a wire, so the fuse's input and the primary's second lead were one
net, and the primary closed on itself through the fuse and the AC switch —
the same fault 9601600 fixed on seventeen other sheets, missed there because
the loop runs through two parts instead of lying on one label. The second
conductor is now "MAINS N" / "AC LINE N".

Read against both drawings (D-FE 7087×4274, H-FD 6061×3777, crops of the
receptacle / ground switch / AC switch corner): one cord conductor runs
through the AC switch to one primary lead, the other through the fuse to the
other lead; the ground switch is a double throw, drawn with the .047 on the
AC-switch side. The AA864's ground-switch label therefore stays on "AC LINE",
the conductor that switch position reaches. Nothing else moves: the fuse
still sits in series with the switch on these sheets, a simplification the
drawings do not make and which is recorded for a separate decision.

check_schematics and verify_schematic_nets clean on all 40 sheets.

Co-Authored-By: Claude Opus 5 (1M context) <noreply@anthropic.com>
Claude-Session: https://claude.ai/code/session_01KBMfdh37HmCL2iWcBiL5J1
Connections:
- net MAINS: no longer CDEATH.1, TR1.2 (PRI_2)
- net at RBIAS.2: now also DBIAS.2 (K)
- net at RLN1.2, RSN.1, V2A.1 (P): no longer CTN.1
- net at CLB1.2, RLB1.2, RSB.1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: no longer CTB.1
- net at VRTB.1: now also CTB.2
- net at VRTN.1: now also CTN.2
- new net MAINS N: CDEATH.1, TR1.2 (PRI_2)
Other:
- moved on the sheet: C1, C10, C11, C12, C13, C14, C15, C2, CB1, CB2, CBB, CBB2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
