File: amps/b15n/schematic.kicad_sch (KiCad schematic)
At the start: 111 parts, among them J1 1/4 in, J2 1/4 in, J3 1/4 in, J4 1/4 in, J5 1/4 in, J6 1/4 in, SW1 SPST, SW2 SPST, SW3 SPST, SW4 SPST, SW5 SPST, SW6 SPST, SW7 SPDT, T1 PT-108, T2 OT-214

Commit message: Fix: deterministic schematic ids and wires split at every join
- _u() is uuid5 over (amp id, emission order), so a regeneration of an
  unchanged script is byte-identical and a drift gate becomes possible
- write() splits wire segments at symbol pins, wire ends and junction dots,
  so the file connects exactly what the drawing shows under KiCad's
  endpoint-only semantics (270 pins were on a wire's interior; net
  partitions unchanged on all 38 sheets)
- all sheets regenerated; aa864-bassman title block was stale (draft) and
  now matches meta.yaml (verified)

Co-Authored-By: Claude Fable 5.1 <noreply@anthropic.com>
Claude-Session: https://claude.ai/code/session_01KBMfdh37HmCL2iWcBiL5J1
Connections:
- net HTB is gone; now on net HTA: T1.5 (HT_B), V6B.1 (A)
Changed lines of the file:
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@@
     (property "Reference" "R1" (at 45.5 44.82 270) (effects (font (size 1.27 1.27)) (justify left)))
     (property "Value" "100k" (at 45.5 47.22 270) (effects (font (size 1.27 1.27)) (justify left))))
-  (wire (pts (xy 31.78 50.82) (xy 44.89 50.82))
-    (stroke (width 0) (type default)))
-  (wire (pts (xy 52.51 50.82) (xy 64.7 50.82))
+  (wire (pts (xy 31.78 50.82) (xy 40.7 50.82))
+    (stroke (width 0) (type default)))
+  (wire (pts (xy 40.7 50.82) (xy 44.89 50.82))
+    (stroke (width 0) (type default)))
+  (wire (pts (xy 52.51 50.82) (xy 56.7 50.82))
+    (stroke (width 0) (type default)))
+  (wire (pts (xy 56.7 50.82) (xy 64.7 50.82))
     (stroke (width 0) (type default)))
   (junction (at 40.7 50.82) (diameter 0) (color 0 0 0 0))
@@
   (wire (pts (xy 52.51 64.82) (xy 64.7 64.82))
     (stroke (width 0) (type default)))
-  (wire (pts (xy 64.7 50.82) (xy 64.7 64.82))
+  (wire (pts (xy 64.7 50.82) (xy 64.7 57.82))
+    (stroke (width 0) (type default)))
+  (wire (pts (xy 64.7 57.82) (xy 64.7 64.82))
     (stroke (width 0) (type default)))
   (junction (at 64.7 50.82) (diameter 0) (color 0 0 0 0))
@@
     (property "Reference" "V1B" (at 206.7 41.23 0) (effects (font (size 1.27 1.27)) (justify left)))
     (property "Value" "6SL7" (at 206.7 43.63 0) (effects (font (size 1.27 1.27)) (justify left))))
-  (wire (pts (xy 149.78 47.63) (xy 193.08 47.63))
+  (wire (pts (xy 149.78 47.63) (xy 186.7 47.63))
+    (stroke (width 0) (type default)))
+  (wire (pts (xy 186.7 47.63) (xy 193.08 47.63))
     (stroke (width 0) (type default)))
   (wire (pts (xy 200.7 40.01) (xy 200.7 33.82))
@@
   (wire (pts (xy 252.51 57.44) (xy 260.7 57.44))
     (stroke (width 0) (type default)))
-  (wire (pts (xy 260.7 49.82) (xy 260.7 57.44))
+  (wire (pts (xy 260.7 49.82) (xy 260.7 53.63))
+    (stroke (width 0) (type default)))
+  (wire (pts (xy 260.7 53.63) (xy 260.7 57.44))
     (stroke (width 0) (type default)))
   (junction (at 260.7 53.63) (diameter 0) (color 0 0 0 0))
@@
     (property "Reference" "R3" (at 45.5 114.82 270) (effects (font (size 1.27 1.27)) (justify left)))
     (property "Value" "100k" (at 45.5 117.22 270) (effects (font (size 1.27 1.27)) (justify left))))
-  (wire (pts (xy 31.78 120.82) (xy 44.89 120.82))
-    (stroke (width 0) (type default)))
-  (wire (pts (xy 52.51 120.82) (xy 64.7 120.82))
+  (wire (pts (xy 31.78 120.82) (xy 40.7 120.82))
+    (stroke (width 0) (type default)))
+  (wire (pts (xy 40.7 120.82) (xy 44.89 120.82))
+    (stroke (width 0) (type default)))
+  (wire (pts (xy 52.51 120.82) (xy 56.7 120.82))
+    (stroke (width 0) (type default)))
+  (wire (pts (xy 56.7 120.82) (xy 64.7 120.82))
     (stroke (width 0) (type default)))
   (junction (at 40.7 120.82) (diameter 0) (color 0 0 0 0))
@@
   (wire (pts (xy 52.51 134.82) (xy 64.7 134.82))
     (stroke (width 0) (type default)))
-  (wire (pts (xy 64.7 120.82) (xy 64.7 134.82))
+  (wire (pts (xy 64.7 120.82) (xy 64.7 127.82))
+    (stroke (width 0) (type default)))
+  (wire (pts (xy 64.7 127.82) (xy 64.7 134.82))
     (stroke (width 0) (type default)))
   (junction (at 64.7 120.82) (diameter 0) (color 0 0 0 0))
@@
     (property "Reference" "V2B" (at 206.7 111.23 0) (effects (font (size 1.27 1.27)) (justify left)))
     (property "Value" "6SL7" (at 206.7 113.63 0) (effects (font (size 1.27 1.27)) (justify left))))
-  (wire (pts (xy 149.78 117.63) (xy 193.08 117.63))
+  (wire (pts (xy 149.78 117.63) (xy 186.7 117.63))
+    (stroke (width 0) (type default)))
+  (wire (pts (xy 186.7 117.63) (xy 193.08 117.63))
     (stroke (width 0) (type default)))
   (wire (pts (xy 200.7 110.01) (xy 200.7 103.82))
@@
   (wire (pts (xy 252.51 127.44) (xy 260.7 127.44))
     (stroke (width 0) (type default)))
-  (wire (pts (xy 260.7 119.82) (xy 260.7 127.44))
+  (wire (pts (xy 260.7 119.82) (xy 260.7 123.63))
+    (stroke (width 0) (type default)))
+  (wire (pts (xy 260.7 123.63) (xy 260.7 127.44))
     (stroke (width 0) (type default)))
   (junction (at 260.7 123.63) (diameter 0) (color 0 0 0 0))
@@
   (text "Printed tone board: both bass caps land on the wiper, and the 120 kOhm link between the two wipers IS the board output." (at 214.7 83.82 0)
     (effects (font (size 1.4 1.4)) (justify left)))
-  (wire (pts (xy 310.7 73.82) (xy 310.7 143.82))
+  (wire (pts (xy 310.7 73.82) (xy 310.7 111.28))
+    (stroke (width 0) (type default)))
+  (wire (pts (xy 310.7 111.28) (xy 310.7 143.82))
     (stroke (width 0) (type default)))
   (wire (pts (xy 310.7 143.82) (xy 310.7 171.82))
@@
     (property "Reference" "V3A" (at 354.7 85.42 0) (effects (font (size 1.27 1.27)) (justify left)))
     (property "Value" "6SL7" (at 354.7 87.82 0) (effects (font (size 1.27 1.27)) (justify left))))
-  (wire (pts (xy 314.7 91.82) (xy 341.08 91.82))
+  (wire (pts (xy 314.7 91.82) (xy 328.7 91.82))
+    (stroke (width 0) (type default)))
+  (wire (pts (xy 328.7 91.82) (xy 341.08 91.82))
     (stroke (width 0) (type default)))
   (junction (at 328.7 91.82) (diameter 0) (color 0 0 0 0))
@@
   (global_label "BP1" (shape input) (at 496.7 125.82 180)
     (effects (font (size 1.27 1.27)) (justify right)))
-  (wire (pts (xy 523.59 123.28) (xy 571.62 123.28))
+  (wire (pts (xy 523.59 123.28) (xy 532.7 123.28))
+    (stroke (width 0) (type default)))
+  (wire (pts (xy 532.7 123.28) (xy 552.7 123.28))
+    (stroke (width 0) (type default)))
+  (wire (pts (xy 552.7 123.28) (xy 564.7 123.28))
+    (stroke (width 0) (type default)))
+  (wire (pts (xy 564.7 123.28) (xy 571.62 123.28))
     (stroke (width 0) (type default)))
   (junction (at 564.7 123.28) (diameter 0) (color 0 0 0 0))
@@
   (wire (pts (xy 438.7 257.82) (xy 438.7 267.82))
     (stroke (width 0) (type default)))
-  (wire (pts (xy 422.7 267.82) (xy 438.7 267.82))
+  (wire (pts (xy 422.7 267.82) (xy 430.7 267.82))
+    (stroke (width 0) (type default)))
+  (wire (pts (xy 430.7 267.82) (xy 438.7 267.82))
     (stroke (width 0) (type default)))
   (junction (at 430.7 267.82) (diameter 0) (color 0 0 0 0))
@@
     (property "Reference" "R38" (at 377.5 283.82 270) (effects (font (size 1.27 1.27)) (justify left)))
     (property "Value" "22k 1W" (at 377.5 286.22 270) (effects (font (size 1.27 1.27)) (justify left))))
-  (wire (pts (xy 398.7 275.82) (xy 398.7 289.82))
+  (wire (pts (xy 398.7 275.82) (xy 398.7 283.44))
+    (stroke (width 0) (type default)))
+  (wire (pts (xy 398.7 283.44) (xy 398.7 289.82))
     (stroke (width 0) (type default)))
   (wire (pts (xy 398.7 289.82) (xy 384.51 289.82))
@@
   (text "Negative-bias supply — R36 taps the 5AR4 plate, which swings below ground on every other half cycle, so D1 conducts toward the bias line. R34 and R35 sit either side of it and R42 separates the two 10 uF cans." (at 470.7 231.82 0)
     (effects (font (size 1.4 1.4)) (justify left)))
-  (wire (pts (xy 422.7 242.58) (xy 470.7 242.58))
+  (wire (pts (xy 422.7 242.58) (xy 438.7 242.58))
+    (stroke (width 0) (type default)))
+  (wire (pts (xy 438.7 242.58) (xy 470.7 242.58))
     (stroke (width 0) (type default)))
   (junction (at 422.7 242.58) (diameter 0) (color 0 0 0 0))
@@
   (global_label "AC L" (shape input) (at 300.7 252.74 180)
     (effects (font (size 1.27 1.27)) (justify right)))
-  (wire (pts (xy 300.7 252.74) (xy 339.62 252.74))
+  (wire (pts (xy 300.7 252.74) (xy 318.7 252.74))
+    (stroke (width 0) (type default)))
+  (wire (pts (xy 318.7 252.74) (xy 339.62 252.74))
     (stroke (width 0) (type default)))
   (junction (at 318.7 252.74) (diameter 0) (color 0 0 0 0))
@@
   (global_label "AC N" (shape input) (at 300.7 262.9 180)
     (effects (font (size 1.27 1.27)) (justify right)))
-  (wire (pts (xy 300.7 262.9) (xy 359.81 262.9))
+  (wire (pts (xy 300.7 262.9) (xy 306.7 262.9))
+    (stroke (width 0) (type default)))
+  (wire (pts (xy 306.7 262.9) (xy 359.81 262.9))
     (stroke (width 0) (type default)))
   (junction (at 306.7 262.9) (diameter 0) (color 0 0 0 0))

Commit message: Fix: schematic wiring on ac15 and b15n
- ac15: the B+1 label named only the EL84 plates/screens and the OT centre
  tap; the standby switch, reservoir and dropper column were a separate
  net the drawing never joined (orphaned rail label)
- b15n: the R38 branch dropped through C16A's grounded pin, shorting the
  screen rail BP2 to chassis (six dependent findings); the paraphase
  divider halves R28/R29 were drawn against each other's anodes and are
  swapped to match netlist and parts list
- both sheets pass connectivity and verify_schematic_nets

Co-Authored-By: Claude Fable 5.1 <noreply@anthropic.com>
Claude-Session: https://claude.ai/code/session_01KBMfdh37HmCL2iWcBiL5J1
Parts:
- R28: renamed from R29; value 510k -> 470k
- R29: renamed from R28; value 470k -> 510k
Connections:
- net BP2: no longer C15.2, C16A.2, C16B.2, C16C.2, C17.2, CBF2.2, CKD1.2, CM2.2, CTA4.2, CTB4.2, J1.2 (S), J2.2 (S), J3.2 (S), J4.2 (S), J5.2 (S), J6.2 (S), R10.2, R12.2, R14.2, R16.2, R20.2, R23.2, R24.2, R25.2, R34.2, R35.2, R41.2, R5.2, R6.2, R8.2, RTA2.2, RTB2.2, SW2.1, SW4.1, SW5.2, SW7.1, T2.5 (SEC_C), V4.4 (K), V5.4 (K), VR1.3, VR4.3, VR7.2 (W)
- new net GND: C15.2, C16A.2, C16B.2, C16C.2, C17.2, CBF2.2, CKD1.2, CM2.2, CTA4.2, CTB4.2, J1.2 (S), J2.2 (S), J3.2 (S), J4.2 (S), J5.2 (S), J6.2 (S), R10.2, R12.2, R14.2, R16.2, R20.2, R23.2, R24.2, R25.2, R34.2, R35.2, R41.2, R5.2, R6.2, R8.2, RTA2.2, RTB2.2, SW2.1, SW4.1, SW5.2, SW7.1, T2.5 (SEC_C), V4.4 (K), V5.4 (K), VR1.3, VR4.3, VR7.2 (W)
Changed lines of the file:
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@@
   (symbol (lib_id "cx:R") (at 374.7 81.63 0) (unit 1)
     (in_bom yes) (on_board yes)
-    (property "Reference" "R28" (at 377.1 80.83 0) (effects (font (size 1.27 1.27)) (justify left)))
-    (property "Value" "470k" (at 377.1 83.23 0) (effects (font (size 1.27 1.27)) (justify left))))
+    (property "Reference" "R29" (at 377.1 80.83 0) (effects (font (size 1.27 1.27)) (justify left)))
+    (property "Value" "510k" (at 377.1 83.23 0) (effects (font (size 1.27 1.27)) (justify left))))
   (wire (pts (xy 374.7 85.44) (xy 374.7 115.82))
     (stroke (width 0) (type default)))
@@
   (symbol (lib_id "cx:R") (at 374.7 119.63 0) (unit 1)
     (in_bom yes) (on_board yes)
-    (property "Reference" "R29" (at 377.1 118.83 0) (effects (font (size 1.27 1.27)) (justify left)))
-    (property "Value" "510k" (at 377.1 121.23 0) (effects (font (size 1.27 1.27)) (justify left))))
+    (property "Reference" "R28" (at 377.1 118.83 0) (effects (font (size 1.27 1.27)) (justify left)))
+    (property "Value" "470k" (at 377.1 121.23 0) (effects (font (size 1.27 1.27)) (justify left))))
   (wire (pts (xy 374.7 123.44) (xy 374.7 157.82))
     (stroke (width 0) (type default)))
@@
     (property "Reference" "R37" (at 377.5 269.82 270) (effects (font (size 1.27 1.27)) (justify left)))
     (property "Value" "22k 1W" (at 377.5 272.22 270) (effects (font (size 1.27 1.27)) (justify left))))
-  (wire (pts (xy 398.7 275.82) (xy 384.51 275.82))
+  (wire (pts (xy 398.7 275.82) (xy 390.7 275.82))
+    (stroke (width 0) (type default)))
+  (wire (pts (xy 390.7 275.82) (xy 384.51 275.82))
     (stroke (width 0) (type default)))
   (wire (pts (xy 376.89 275.82) (xy 366.7 275.82))
@@
     (property "Reference" "R38" (at 377.5 283.82 270) (effects (font (size 1.27 1.27)) (justify left)))
     (property "Value" "22k 1W" (at 377.5 286.22 270) (effects (font (size 1.27 1.27)) (justify left))))
-  (wire (pts (xy 398.7 275.82) (xy 398.7 283.44))
-    (stroke (width 0) (type default)))
-  (wire (pts (xy 398.7 283.44) (xy 398.7 289.82))
-    (stroke (width 0) (type default)))
-  (wire (pts (xy 398.7 289.82) (xy 384.51 289.82))
-    (stroke (width 0) (type default)))
-  (junction (at 398.7 289.82) (diameter 0) (color 0 0 0 0))
+  (junction (at 390.7 275.82) (diameter 0) (color 0 0 0 0))
+  (wire (pts (xy 390.7 275.82) (xy 390.7 289.82))
+    (stroke (width 0) (type default)))
+  (wire (pts (xy 390.7 289.82) (xy 384.51 289.82))
+    (stroke (width 0) (type default)))
   (wire (pts (xy 376.89 289.82) (xy 366.7 289.82))
     (stroke (width 0) (type default)))

Commit message: Add: real tube pin numbers and readable valve glyphs on every schematic
Phase B of the drawing program. A factory service sheet numbers every tube
pin, because the number is what a technician puts a probe on. This corpus
printed none, and the numbers hidden in its symbols were positional
placeholders (P=1, G=2, K=3) that would have published a 6V6GT's plate as
pin 1 when it is pin 3.

1055 electrodes now carry the real number, 1027 lettered (27 are shared
filaments deduped, 1 dropped for want of clear space on the 6G2). Resolved per
instance from reference/tubes/<slug>.yaml through the same alias resolution the
layout renderer uses, so a 12AX7 section and a 6SL7 section each get their own
basing. A valve whose basing the corpus does not carry prints nothing rather
than a wrong number.

Section letters and basing units are now separate things, which cost a detour
worth recording. The RCA 12AX7-A sheet reads "Pin 1 - Plate of Unit No.2 ...
Pin 6 - Plate of Unit No.1", so unit numbering is not pin order; the 5Y3 and
GZ34 number their units in opposite pin order, so nothing positional can
express it. But the section LETTER is a designator, not a basing fact: this
corpus, like every technician, calls the first stage in signal order V1A, and
five amps' prose already did. On four amps the factory sheets put that first
stage on the other half -- the AA764's own schematic prints +200 V on pin 1 --
so those drawings now state their unit explicitly, each citing its source, and
no letter, netlist, parts list or layout comment changed. 183 layout comments
agree with the printed numbers, 0 disagree. A guard fires if two halves of one
bottle resolve to the same unit, which is exactly how this was found.

Glyphs: the cathode gains a bracket and filament hairpin so it can no longer be
confused with the plate bar, the pentode's screen sits on its own row, and a
rectifier draws as one envelope over its sections instead of two apparent
bottles. Line weights are scaled per sheet to a co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
Other:
- note added: "1"
- note added: "2"
- note added: "3"
- note added: "4"
- note added: "5"
- note added: "6"
- note added: "8"

Commit message: Fix: schematic sheet notes no longer name repository files
Thirty-seven committed sheets rendered footnotes and section notes such as
"Heaters and PT primary omitted — see netlist.cir and meta.yaml" or
"excluded from netlist.cir (notes.md)" to visitors through KiCanvas. The
prose sweeps never counted sheets. Rewritten in the site's own words — the
netlist, the sources list, the circuit story, the parts list, the board
drawing — in 59 strings across 33 draw scripts, keeping every technical
claim as it was; the three tone sheets (6G4, 6G5, 6G6-B) are under repair
elsewhere and keep theirs for now. The sweep touched only strings passed to
the sheet's note, text, caption and footnote calls, never a path or a value.

Gates: check_schematics 40/0, connectivity 0 isolated pins;
verify_schematic_nets 40 clean; only the regenerated sheets and their served
copies changed.

Co-Authored-By: Claude Fable 5.1 <noreply@anthropic.com>
Claude-Session: https://claude.ai/code/session_01KBMfdh37HmCL2iWcBiL5J1
Other:
- note added: "The 6.3 V heater chain (green pair, VR7 100 Ohm hum balance, sockets V1..V5 on pins 7/8 and 7/2), the mains side beyond the transformer primary (POWER SW6, POLAR. SW7, the 3 A and 6 A fuses, the switched AC outlet, C18 and CM2) and the panel pilot lamp are omitted here — see the parts list and the board layout. The drawing puts that pilot straight across the mains primary, not on the heater chain."
- note added: "Two printed voltages on the driver cannot be true and are carried as disputed rather than fitted: 3 V across R25 220 Ohm is 13.6 mA, six times a 6SL7 unit's Class-A point and 3.2 W in a 1 W plate, and 2.2 V across R24 1 kOhm needs a 489 V rail behind the drawn 120 kOhm in an amplifier whose highest node is 450 V. See the circuit story."
- note removed: "The 6.3 V heater chain (green pair, VR7 100 Ohm hum balance, sockets V1..V5 on pins 7/8 and 7/2), the mains side beyond the transformer primary (POWER SW6, POLAR. SW7, the 3 A and 6 A fuses, the switched AC outlet, C18 and CM2) and the panel pilot lamp are omitted here — see bom.yaml and the board layout. The drawing puts that pilot straight across the mains primary, not on the heater chain."
- note removed: "Two printed voltages on the driver cannot be true and are carried as disputed rather than fitted: 3 V across R25 220 Ohm is 13.6 mA, six times a 6SL7 unit's Class-A point and 3.2 W in a 1 W plate, and 2.2 V across R24 1 kOhm needs a 489 V rail behind the drawn 120 kOhm in an amplifier whose highest node is 450 V. See notes.md."
Changed lines of the file:
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@@
   (text "Rails: BP1 = the 5AR4 cathode and C17 reservoir, which is also the OT-214 primary centre tap and therefore the 6L6GC plate node (450 V on the drawing) — BP2 = the screen node, one 1 kOhm 10 W dropper below it (445 V) — BP3 = the preamp rail both channels share and BP4 = the driver rail, each behind its own 22 kOhm 1 W dropper off BP2. The two never rejoin." (at 12.7 310.978 0)
     (effects (font (size 1.2 1.2)) (justify left)))
-  (text "The 6.3 V heater chain (green pair, VR7 100 Ohm hum balance, sockets V1..V5 on pins 7/8 and 7/2), the mains side beyond the transformer primary (POWER SW6, POLAR. SW7, the 3 A and 6 A fuses, the switched AC outlet, C18 and CM2) and the panel pilot lamp are omitted here — see bom.yaml and the board layout. The drawing puts that pilot straight across the mains primary, not on the heater chain." (at 12.7 315.378 0)
+  (text "The 6.3 V heater chain (green pair, VR7 100 Ohm hum balance, sockets V1..V5 on pins 7/8 and 7/2), the mains side beyond the transformer primary (POWER SW6, POLAR. SW7, the 3 A and 6 A fuses, the switched AC outlet, C18 and CM2) and the panel pilot lamp are omitted here — see the parts list and the board layout. The drawing puts that pilot straight across the mains primary, not on the heater chain." (at 12.7 315.378 0)
     (effects (font (size 1.2 1.2)) (justify left)))
-  (text "Two printed voltages on the driver cannot be true and are carried as disputed rather than fitted: 3 V across R25 220 Ohm is 13.6 mA, six times a 6SL7 unit's Class-A point and 3.2 W in a 1 W plate, and 2.2 V across R24 1 kOhm needs a 489 V rail behind the drawn 120 kOhm in an amplifier whose highest node is 450 V. See notes.md." (at 12.7 319.778 0)
+  (text "Two printed voltages on the driver cannot be true and are carried as disputed rather than fitted: 3 V across R25 220 Ohm is 13.6 mA, six times a 6SL7 unit's Class-A point and 3.2 W in a 1 W plate, and 2.2 V across R24 1 kOhm needs a 489 V rail behind the drawn 120 kOhm in an amplifier whose highest node is 450 V. See the circuit story." (at 12.7 319.778 0)
     (effects (font (size 1.2 1.2)) (justify left)))
   (text "The OT-214 secondary is tapped — GRN., YEL. and BLK. on the drawing — and the EXT. SPKR. jack J6 normals the internal 8 Ohm speaker. Only the green and black ends are drawn here, with R41 250 Ohm 10 W across them; the yellow tap, J6 and the speaker are the annotation layer." (at 12.7 324.178 0)
