File: amps/b15n/schematic.kicad_sch (KiCad schematic)
At the start: 111 parts, among them J1 1/4 in, J2 1/4 in, J3 1/4 in, J4 1/4 in, J5 1/4 in, J6 1/4 in, SW1 SPST, SW2 SPST, SW3 SPST, SW4 SPST, SW5 SPST, SW6 SPST, SW7 SPDT, T1 PT-108, T2 OT-214

Commit message: Fix: four single-sheet faults — 5G9 oscillator cathode grounded, B15N R36 bridging both rectifier plates, M1959/M1987 bias series resistor drawn as a shunt / after the diode
- 5g9: the factory sheet (crop 5g9-V3-schem.png) prints the oscillator
  cathode at +1.7 V on 1500 ‖ 25 µF, with the ladder's second 1M returned
  to that cathode node. The sheet had the same parts, but R7's ground flag
  stood ON the wire that returns R8 to the cathode, which grounded the
  whole node: RK3, CK3 and R8 all reported "the sheet shorts its two ends
  onto one net". The flag now points left from a shorter stub, clear of
  that wire. No part added — bom.yaml already carried RK3/CK3/R8.
- b15n: the Ampeg 591722 sheet (crop b15n-V6-rect.png, re-read at native
  resolution: R36's lower lead HOPS the B+ and screen lines and lands on
  the R35/D1 node with a dot) hangs R36 100K/2W on the pin-4 RED HT end.
  The sheet's feed wire ran from V6A's plate stub straight across the top
  of V6B's, joining both HT ends into one net (the SPLIT finding). R36 now
  takes its own HTA label. Caption reworded to name pin 4.
- m1959: the Unicord 70-6-11 sheet (crops m1959-bias-series.png,
  m1959-psu.png) runs the HT winding's end through the 27K (22K annotated)
  IN SERIES into the 1008 diode; the sheet drew it as a shunt at the
  diode. RBA is now in series before D1; bom role and circuit story
  reworded. The brief's "C24 on the bias node" does not exist on this
  amp: its bias filters are C17/C18 on sheet and BOM alike, C24 is the PI
  filter on both. The C24 on a bias-diode node was the M1987's rectifier
  snubber (below).
- m1987: the Unicord 70-19-11 sheet (crops m1987-bias.png, m1987-psu.png)
  runs the winding end through 220K into the diode, then 8 µF / 15K; the
  sheet had the diode first and the 220K after it, so RBA and RBB shared
  a node. RBA now sits before D1; RBA and RBB are separated by the diode.
  C24 (the D3 snubber, per bom.yaml) stays on HT_B and no longer shares a
  node with the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
Parts:
- removed R42: 10k, symbol cx:R
- removed SW7: SPDT, symbol cx:SWITCH
- added C15: 10u 100V, symbol cx:C
- added SW6: SPST, symbol cx:SWITCH
- C18: renamed from SW6; value SPST -> .047u 600V; symbol cx:SWITCH -> cx:C
- R42: renamed from C15; value 10u 100V -> 10k; symbol cx:C -> cx:R
- SW7: renamed from C18; value .047u 600V -> SPDT; symbol cx:C -> cx:SWITCH
Connections:
- net -50V: now also R42.1
- net AC L: now also SW6.1; no longer SW7.1
- net GND: now also SW7.1, C15.2; no longer R42.2
- net HTA: no longer T1.5 (HT_B), V6B.1 (A)
- net at T1.1 (PRI_1): now also SW6.2; no longer C18.2
- net at D1.1 (A), R34.1: now also R42.2, C15.1; no longer R42.1
- net at SW7.2: now also C18.2
- new net HTB: T1.5 (HT_B), V6B.1 (A)
Other:
- note added: "Negative-bias supply — R36 taps the pin-4 5AR4 plate, one HT end, which swings below ground every other half cycle so D1 conducts toward the bias line. R34 and R35 flank it, R42 parts the two 10 uF cans."
- note removed: "Negative-bias supply — R36 taps the 5AR4 plate, which swings below ground on every other half cycle, so D1 conducts toward the bias line. R34 and R35 sit either side of it and R42 separates the two 10 uF cans."
Changed lines of the file:
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@@
 (kicad_sch (version 20231120) (generator "circuit-codex")
-  (paper "User" 682.37 374.22)
+  (paper "User" 676.66 374.22)
   (title_block
     (title "B15N — Ampeg B-15N Portaflex-style")
@@
   (global_label "BP4" (shape input) (at 358.7 289.82 180)
     (effects (font (size 1.27 1.27)) (justify right)))
-  (text "Negative-bias supply — R36 taps the 5AR4 plate, which swings below ground on every other half cycle, so D1 conducts toward the bias line. R34 and R35 sit either side of it and R42 separates the two 10 uF cans." (at 470.7 231.82 0)
+  (text "Negative-bias supply — R36 taps the pin-4 5AR4 plate, one HT end, which swings below ground every other half cycle so D1 conducts toward the bias line. R34 and R35 flank it, R42 parts the two 10 uF cans." (at 470.7 231.82 0)
     (effects (font (size 1.4 1.4)) (justify left)))
-  (wire (pts (xy 422.7 242.58) (xy 438.7 242.58))
-    (stroke (width 0) (type default)))
-  (wire (pts (xy 438.7 242.58) (xy 470.7 242.58))
-    (stroke (width 0) (type default)))
-  (junction (at 422.7 242.58) (diameter 1.7) (color 0 0 0 0))
+  (global_label "HTA" (shape input) (at 470.7 242.58 180)
+    (effects (font (size 1.27 1.27)) (justify right)))
   (symbol (lib_id "cx:R") (at 488.7 242.58 90) (unit 1)
     (in_bom yes) (on_board yes)

Commit message: Fix: B15N hung the 10K global feedback on the driver's cathode; both revisions land it on the driver grid, the mixing bus
- On the Ampeg 591722 drawing, sheet 1 and the Rev C copy both run R40 10K
  from the OT's GRN secondary lead down the left edge and into V3 pin 1,
  the driver GRID, where the two channels' 270K mixing resistors meet.
  R25 220 Ohm sits alone on pin 3. The corpus had R40 K3B 0 10k, the sheet
  wired R40 onto R25's top, and the caption, BOM, notes and the K3B
  dispute_note all described R25 as the feedback divider's shunt leg.
- The netlist now reads R40 G3B 0 10k (the secondary is ~0 V DC). With no
  grid current it moves no operating point, and K3B loses the 215-Ohm
  "effective cathode" trim. The sheet carries R40 from the GRN junction to
  the grid line, and the derived board routes R40.a to V3 pin 1 instead of
  R25.a. The notes describe feedback summed into the mixing bus. The
  driver-grid DC-return prose (netlist header, sheet note, the RG3B
  declaration) now names R40.
- K3B dispute_note: the arithmetic stands (3 V over 220 Ohm is 13.6 mA,
  3.2 W in a 1 W plate). Its reasoning no longer rests on R40 sharing the
  node.
- Sheet, schematic-net, layout-net and sheet-board gates are clean on R40
  and R25. The standing VR7/C18/CM2 rows predate this change.

Co-Authored-By: Claude Opus 5 (1M context) <noreply@anthropic.com>
Parts:
- removed R24: 1k, symbol cx:R
- added CKD1: 25u 25V, symbol cx:C
- R24: renamed from CKD1; value 25u 25V -> 1k; symbol cx:C -> cx:R
Connections:
- net GND: now also CKD1.2
- net at R24.1, V3A.3 (K): now also CKD1.1
- net at J5.1 (T), R18.2, R22.2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: now also R40.1
- net at R25.1, V3B.3 (K): no longer R40.1
Other:
- note added: "Both channels sum through 270 kOhm apiece onto the driver grid, which has no grid leak of its own: its DC returns are R40 10 kOhm, the global feedback resistor, to the output transformer's green lead, and the path back out through those two mixing resistors and both tone boards to their 22 kOhm feet. The EXT. AMP. jack J5 taps the same node."
- note added: "Global negative feedback: 10 kOhm from the output transformer's green secondary lead onto the driver grid, the channels' mixing bus. R25 220 Ohm is the driver's own unbypassed cathode resistor."
- note removed: "Both channels sum through 270 kOhm apiece onto the driver grid, which has no grid leak of its own: its DC return runs back out through those two mixing resistors and both tone boards to their 22 kOhm feet. The EXT. AMP. jack J5 taps the same node."
- note removed: "Global negative feedback: 10 kOhm from the output transformer's green secondary lead onto the driver cathode over R25 220 Ohm, which is why that 220 Ohm is a feedback shunt leg rather than a bias resistor."
Changed lines of the file:
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@@
   (junction (at 310.7 143.82) (diameter 1.7) (color 0 0 0 0))
   (junction (at 310.7 111.28) (diameter 1.7) (color 0 0 0 0))
-  (wire (pts (xy 310.7 171.82) (xy 341.08 171.82))
+  (wire (pts (xy 310.7 171.82) (xy 328.7 171.82))
+    (stroke (width 0) (type default)))
+  (wire (pts (xy 328.7 171.82) (xy 341.08 171.82))
     (stroke (width 0) (type default)))
   (symbol (lib_id "cx:JACK") (at 330.7 113.82 0) (unit 1)
@@
   (wire (pts (xy 348.7 179.44) (xy 348.7 182.82))
     (stroke (width 0) (type default)))
-  (junction (at 348.7 182.82) (diameter 1.7) (color 0 0 0 0))
   (symbol (lib_id "cx:R") (at 348.7 186.63 0) (unit 1)
     (in_bom yes) (on_board yes)
@@
   (wire (pts (xy 552.7 205.82) (xy 462.51 205.82))
     (stroke (width 0) (type default)))
-  (wire (pts (xy 454.89 205.82) (xy 364.7 205.82))
-    (stroke (width 0) (type default)))
-  (wire (pts (xy 364.7 205.82) (xy 364.7 182.82))
-    (stroke (width 0) (type default)))
-  (wire (pts (xy 364.7 182.82) (xy 348.7 182.82))
-    (stroke (width 0) (type default)))
-  (text "Global negative feedback: 10 kOhm from the output transformer's green secondary lead onto the driver cathode over R25 220 Ohm, which is why that 220 Ohm is a feedback shunt leg rather than a bias resistor." (at 364.7 213.82 0)
+  (wire (pts (xy 454.89 205.82) (xy 328.7 205.82))
+    (stroke (width 0) (type default)))
+  (wire (pts (xy 328.7 205.82) (xy 328.7 171.82))
+    (stroke (width 0) (type default)))
+  (junction (at 328.7 171.82) (diameter 1.7) (color 0 0 0 0))
+  (text "Global negative feedback: 10 kOhm from the output transformer's green secondary lead onto the driver grid, the channels' mixing bus. R25 220 Ohm is the driver's own unbypassed cathode resistor." (at 364.7 213.82 0)
     (effects (font (size 1.4 1.4)) (justify left)))
   (text "Power supply — PT-108 mains transformer, 5AR4, the STANDBY switch in the HT centre-tap return, one reservoir and a three-section can. No choke." (at 318.7 228.32 0)
@@
   (text "Every crossing drawn here is a crossing: the factory sheet marks \"crosses, does not connect\" with a small S-jog, and this redraw uses the plain KiCad convention instead — a junction dot means a joint and nothing else does." (at 12.7 328.578 0)
     (effects (font (size 1.2 1.2)) (justify left)))
-  (text "Both channels sum through 270 kOhm apiece onto the driver grid, which has no grid leak of its own: its DC return runs back out through those two mixing resistors and both tone boards to their 22 kOhm feet. The EXT. AMP. jack J5 taps the same node." (at 12.7 332.978 0)
+  (text "Both channels sum through 270 kOhm apiece onto the driver grid, which has no grid leak of its own: its DC returns are R40 10 kOhm, the global feedback resistor, to the output transformer's green lead, and the path back out through those two mixing resistors and both tone boards to their 22 kOhm feet. The EXT. AMP. jack J5 taps the same node." (at 12.7 332.978 0)
     (effects (font (size 1.2 1.2)) (justify left)))
   (text "The mains side is the annotation layer, drawn only as far as the sheet settles it: the POWER switch SW6 in one line leg ahead of the transformer primary, and the two 0.047 uF 600 V capacitors it letters C18 and (a third time) C19 — listed CM2 — from the line to chassis, the first through the POLAR. switch SW7. That corner of the published scan is coarse: the parts, their values and their mains-side placement are the sheet's; the exact switching is drawn as the line-to-chassis pair it letters. The 3 A and 6 A fuses, the switched 120 V AC outlet and the panel pilot lamp are not drawn — this circuit puts that pilot straight across the transformer primary, not on the heater chain." (at 12.7 337.378 0)
