File: amps/ga40/schematic.kicad_sch (KiCad schematic)
At the start: 41 parts, among them T1 Gibson (no number printed), T2 Gibson (no number printed)

Commit message: Fix: schematic sheet notes no longer name repository files
Thirty-seven committed sheets rendered footnotes and section notes such as
"Heaters and PT primary omitted — see netlist.cir and meta.yaml" or
"excluded from netlist.cir (notes.md)" to visitors through KiCanvas. The
prose sweeps never counted sheets. Rewritten in the site's own words — the
netlist, the sources list, the circuit story, the parts list, the board
drawing — in 59 strings across 33 draw scripts, keeping every technical
claim as it was; the three tone sheets (6G4, 6G5, 6G6-B) are under repair
elsewhere and keep theirs for now. The sweep touched only strings passed to
the sheet's note, text, caption and footnote calls, never a path or a value.

Gates: check_schematics 40/0, connectivity 0 isolated pins;
verify_schematic_nets 40 clean; only the regenerated sheets and their served
copies changed.

Co-Authored-By: Claude Fable 5.1 <noreply@anthropic.com>
Claude-Session: https://claude.ai/code/session_01KBMfdh37HmCL2iWcBiL5J1
Other:
- note added: "Heaters, the transformer's 5 V and 6.3 V windings, the pilot lamp, the input and speaker jacks and the mains side beyond the transformer (3 A fuse, on/off switch, and the 0.02 µF capacitor the polarity switch grounds onto one line leg or the other) are omitted here — see the parts list and the board drawing. Do not build that mains side as the factory sheet draws it; it predates grounded three-wi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"
- note added: "Rails, lettered from the factory chart's own E(B+) column: BP310 is the post-choke node — the output-transformer centre tap and both 6V6GT screens sit on it, and this circuit has no screen resistors at all; BP280 is the inverter rail one 10 kΩ dropper below it; BP265 the channel-preamp rail one more below that. Because those droppers also carry channel 2 and the tremolo, the netlist drives all th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"
- note added: "the circuit story."
- note removed: "Heaters, the transformer's 5 V and 6.3 V windings, the pilot lamp, the input and speaker jacks and the mains side beyond the transformer (3 A fuse, on/off switch, and the 0.02 µF capacitor the polarity switch grounds onto one line leg or the other) are omitted here — see bom.yaml and layout.yaml. Do not build that mains side as the factory sheet draws it; it predates grounded three-wire practice."
- note removed: "Rails, lettered from the factory chart's own E(B+) column: BP310 is the post-choke node — the output-transformer centre tap and both 6V6GT screens sit on it, and this circuit has no screen resistors at all; BP280 is the inverter rail one 10 kΩ dropper below it; BP265 the channel-preamp rail one more below that. Because those droppers also carry channel 2 and the tremolo, netlist.cir drives all th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"
- note removed: "notes.md."
Changed lines of the file:
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@@
   (text "4" (at 162.186 167.35 0)
     (effects (font (size 1.1 1.1)) (justify left)))
-  (text "Rails, lettered from the factory chart's own E(B+) column: BP310 is the post-choke node — the output-transformer centre tap and both 6V6GT screens sit on it, and this circuit has no screen resistors at all; BP280 is the inverter rail one 10 kΩ dropper below it; BP265 the channel-preamp rail one more below that. Because those droppers also carry channel 2 and the tremolo, netlist.cir drives all three rails at the printed figures rather than deriving a chain missing half its load." (at 12.7 256.098 0)
+  (text "Rails, lettered from the factory chart's own E(B+) column: BP310 is the post-choke node — the output-transformer centre tap and both 6V6GT screens sit on it, and this circuit has no screen resistors at all; BP280 is the inverter rail one 10 kΩ dropper below it; BP265 the channel-preamp rail one more below that. Because those droppers also carry channel 2 and the tremolo, the netlist drives all three rails at the printed figures rather than deriving a chain missing half its load." (at 12.7 256.098 0)
     (effects (font (size 1.2 1.2)) (justify left)))
   (text "Channel 2's 5879 and the 6SQ7 tremolo oscillator are lettered as bottles and left undrawn. Channel 2's screen is fed through the tremolo's Depth network — modulating that screen is how this amplifier makes tremolo — and neither the network nor the channel-2 screen dropper resolves on the only published drawing of this revision. The chart says the same thing loudly: +32 V on that screen against +95 V on channel 1's, off the same +265 V rail. What is legible of both is written out in" (at 12.7 260.498 0)
     (effects (font (size 1.2 1.2)) (justify left)))
-  (text "notes.md." (at 12.7 264.898 0)
+  (text "the circuit story." (at 12.7 264.898 0)
     (effects (font (size 1.2 1.2)) (justify left)))
   (text "A published restoration records the supply-can complement as 20/10/10/10 µF at 450 WVDC. Three of the four are lettered here; the fourth most likely sits on the +280 V inverter rail, where this reading places no can. The gap is left visible rather than filled." (at 12.7 269.298 0)
     (effects (font (size 1.2 1.2)) (justify left)))
-  (text "Heaters, the transformer's 5 V and 6.3 V windings, the pilot lamp, the input and speaker jacks and the mains side beyond the transformer (3 A fuse, on/off switch, and the 0.02 µF capacitor the polarity switch grounds onto one line leg or the other) are omitted here — see bom.yaml and layout.yaml. Do not build that mains side as the factory sheet draws it; it predates grounded three-wire practice." (at 12.7 273.698 0)
+  (text "Heaters, the transformer's 5 V and 6.3 V windings, the pilot lamp, the input and speaker jacks and the mains side beyond the transformer (3 A fuse, on/off switch, and the 0.02 µF capacitor the polarity switch grounds onto one line leg or the other) are omitted here — see the parts list and the board drawing. Do not build that mains side as the factory sheet draws it; it predates grounded three-wire practice." (at 12.7 273.698 0)
     (effects (font (size 1.2 1.2)) (justify left)))
   (text "The factory drawing letters no reference designators — not on the bottles, not on the passives — so the designators on this sheet are this corpus's own, functional ones: RL a plate load, RS a screen dropper, CK a cathode bypass, RD a rail dropper." (at 12.7 278.098 0)

Commit message: Fix: the 6G5's rectifier was connected to nothing; 17 sheets shorted the mains by naming both leads alike
6G5 power supply. The sheet drew four diodes as a "silicon bridge" whose
HT_A/HT_B labels stopped 6 mm short of their wires. D1/D2's anodes sat on
the tremolo's cathode node (a tremolo wire's end touched the old diode
stub), D3/D4 ran from ground to the reservoir, and TR1's centre tap floated
under an open-pin waiver whose stated reason was the bridge itself.
A-FJ (Schematic Heaven 2153x1437, read enlarged): each HT end of TR1 runs
through a leg of three silicon diodes, every + (cathode) toward the +460 V
reservoir; the centre tap is grounded; TR1's second secondary terminal is a
bias tap feeding the 6G4's network part for part: rectifier, 8-150, 10K,
then 8-150 and a 56K bleeder at the -55 V line. Redrawn as the drawing
shows: D1-D6, TR1 with its tap pin, the centre tap to ground, the bias
network (CBIAS 25 uF -> 8 uF; RBIAS2, CBIAS2, RBIAS1 added), the waiver
deleted, and the notes, meta, netlist header and parts list no longer say
bridge. Not yet carried: the drawing's second 20-600 at the reservoir and
the standby switch (this sheet omits chassis switches by its own note);
and the tremolo ladder still runs through the transformer's corner of the
sheet, a layout clash rather than a connection, queued for its own redraw.

Mains. Two global labels with one name are one net. 16 of 24 power
transformers on the sheets carried a label named MAINS on both primary
leads, so the winding's two pins were one net: 5E4-A, 5E5-A, 5F4, 5G9,
6161, 6G2, 6G3, 6G4, AA1164, AA764, AA764-Vibro, AA964, AB763, AB763
Super, AB763 Twin, GA-40. The 6G5's loop ran from one MAINS label through
switch, fuse and winding back to the same name. No gate models the primary,
so a copy-pasted idiom did this. The second lead is now MAINS N, the AC15's
idiom; the AA1164's and AA964's second AC row, drawn under the first row's
name, is the neutral. The death and across-the-line caps stay on the le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
Connections:
- net MAINS: no longer T1.2 (PRI_2)
- new net MAINS N: T1.2 (PRI_2)
Changed lines of the file:
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@@
   (wire (pts (xy 44.446 172.4) (xy 39.336 172.4))
     (stroke (width 0) (type default)))
-  (global_label "MAINS" (shape input) (at 39.336 172.4 180)
+  (global_label "MAINS N" (shape input) (at 39.336 172.4 180)
     (effects (font (size 1.27 1.27)) (justify right)))
   (wire (pts (xy 62.226 167.32) (xy 67.336 167.32))

Commit message: Fix: the GA-40 sheet tied the channel-1 volume wiper to the +265 V rail
The sheet's coupler run from CV1 to the VR1 wiper drops down x=129.3, and the 750 kΩ screen dropper's BP265 lead ended on that run at y=48.05, so the writer split the wire there and CV1.2 and the wiper landed on BP265. That is what the gate read as CF3, RD2, RL1 and RS1 misplaced: the sheet's rail net carried CV1.2 and VR1.lug2, the board's did not.

Read the GA-40 factory drawing (schematicheaven ga40.pdf, the 1022x758 native scan, the only copy), crop (180,80)-(340,170): the .01 runs from the 5879 plate node straight to the 1M volume's wiper arrow, the track's top to the 470K and its bottom to ground. Nothing joins it to the rail the 100K and 750K drop to. The board (CV1.b to VR1.lug2) was right; the sheet was wrong.

The BP265 label now hangs down at x=125.3, short of the coupler's run, and VR1's lettering is pinned to the right of the pot, where it sat before. No netlist, voltage or board change. The sheet-board gate now passes for ga40. FW-19 P10b.

Co-Authored-By: Claude Opus 5.5 <noreply@anthropic.com>
Claude-Session: https://claude.ai/code/session_01KBMfdh37HmCL2iWcBiL5J1
Signed-off-by: AnalogMaker <theanalogmaker@gmail.com>
Parts:
- removed CK4, CKO: 20u, symbol cx:C
- removed V3: 6SQ7, symbol cx:TRIODE
- removed VR3: 1M, symbol cx:POT
- added CT1: .005u, symbol cx:C
- added RK4: 1k, symbol cx:R
- added RKO: 200, symbol cx:R
- added V2: 5879, symbol cx:PENTODE
- CK4: renamed from RK4; value 1k -> 20u; symbol cx:R -> cx:C
- CKO: renamed from RKO; value 200 -> 20u; symbol cx:R -> cx:C
- V3: renamed from V2; value 5879 -> 6SQ7; symbol cx:PENTODE -> cx:TRIODE
- VR3: renamed from CT1; value .005u -> 1M; symbol cx:C -> cx:POT
Connections:
- net BP265: no longer CV1.2, VR1.2 (W)
- net GND: now also VR3.2 (W), RK4.2, RKO.2
- net KOUT: now also RKO.1
- net at CC1.1, RL4A.2, V4A.1 (P): now also CT1.1; no longer VR3.1
- net at CK4.1, V4A.3 (K), V4B.3 (K): now also RK4.1
- new net: CT1.2, VR3.1
- new net: CV1.2, VR1.2 (W)
Changed lines of the file:
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@@
   (wire (pts (xy 105.336 48.05) (xy 113.526 48.05))
     (stroke (width 0) (type default)))
-  (wire (pts (xy 121.146 48.05) (xy 129.336 48.05))
+  (wire (pts (xy 121.146 48.05) (xy 125.336 48.05))
     (stroke (width 0) (type default)))
-  (global_label "BP265" (shape input) (at 129.336 48.05 0)
-    (effects (font (size 1.27 1.27)) (justify left)))
+  (global_label "BP265" (shape input) (at 125.336 48.05 270)
+    (effects (font (size 1.27 1.27)) (justify right)))
   (junction (at 105.336 48.05) (diameter 1.7) (color 0 0 0 0))
   (symbol (lib_id "cx:C") (at 105.336 51.86 0) (unit 1)
@@
   (wire (pts (xy 121.146 37.32) (xy 129.336 37.32))
     (stroke (width 0) (type default)))
-  (wire (pts (xy 129.336 37.32) (xy 129.336 48.05))
-    (stroke (width 0) (type default)))
-  (wire (pts (xy 129.336 48.05) (xy 129.336 53.32))
+  (wire (pts (xy 129.336 37.32) (xy 129.336 53.32))
     (stroke (width 0) (type default)))
   (wire (pts (xy 129.336 53.32) (xy 144.416 53.32))
@@
   (symbol (lib_id "cx:POT") (at 139.336 45.13 0) (unit 1)
     (in_bom yes) (on_board yes)
-    (property "Reference" "VR1" (at 143.538 43.49 0) (effects (font (size 1.27 1.27)) (justify left)))
-    (property "Value" "1M" (at 143.538 45.89 0) (effects (font (size 1.27 1.27)) (justify left))))
+    (property "Reference" "VR1" (at 143.536 43.49 0) (effects (font (size 1.27 1.27)) (justify left)))
+    (property "Value" "1M" (at 143.536 45.89 0) (effects (font (size 1.27 1.27)) (justify left))))
   (wire (pts (xy 144.416 53.32) (xy 144.416 45.13))
     (stroke (width 0) (type default)))
