File: amps/5f8a/schematic.kicad_sch (KiCad schematic)
At the start: 74 parts, among them T3 45268

Commit message: Fix: the 5F6, 5F8-A and 5F6-A sheets fed the selenium bias rectifier from an HT end; it takes its own tap
All three factory schematics bring the bias feed down to its OWN winding terminal, between the upper HT end and the centre tap. It is not the HT end. At 3x zoom the vertical feed line crosses the upper "325 V AC" (5F8-A: "300 V AC") lead with no junction dot and ends on the next terminal down:
- 5F6 (F-EG) schematic page, crop (3560,3580)-(3900,3880), in the context of (3550,2850)-(4650,4100);
- 5F8-A (I-EG), native 6310x3506, crop (3250,2800)-(3800,3350);
- 5F6-A (I-EG), crop (3550,3500)-(4000,3950).
The layout pages agree. 5F6 crop (900,2200)-(2900,3800) and 5F8-A crop (600,1300)-(2400,2000) each draw a dedicated RED-BLUE transformer lead to SEL. RECT. "+", separate from the two RED HT leads that go to the rectifier plates.

So red-blue is a separate tap, as on the 6G6-B, and the sheets were the surface in error: each lettered D1's anode HT_B, putting the bias rectifier on the rectifier plate node. Each sheet now letters it HT_TAP. sch_map.yaml winding_labels declares HT_TAP: tap, so the UNFED RECTIFIER walk still sees D1 fed, and HT_B's note drops "also feeds bias rectifier D1". The 5F6 and 5F8-A boards, which wire PT.red-blue to D1, declare net_map.leads "<HT_TAP>": PT.red-blue. The 5F6-A board does not place D1 (a declared not_on_board), so it needs no lead.

Sheet-board: 5F6 misplaced [D1] -> [] (both drawings claim verified; it now PASSes), 5F8-A misplaced [D1] -> []. verify_schematic_nets PASS for all three, and 48/48 rectifiers fed. No netlist change: the bias supply is the ideal NBIAS source in every netlist. FW-19 P10c.

Co-Authored-By: Claude Opus 5.5 <noreply@anthropic.com>
Claude-Session: https://claude.ai/code/session_01KBMfdh37HmCL2iWcBiL5J1
Signed-off-by: AnalogMaker <theanalogmaker@gmail.com>
Connections:
- net HT_B: no longer D1.2 (K)
- new net HT_TAP: D1.2 (K)
Changed lines of the file:
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@@
   (global_label "GND" (shape input) (at 155.926 166.922 270)
     (effects (font (size 1.27 1.27)) (justify right)))
-  (global_label "HT_B" (shape input) (at 151.836 177.502 180)
+  (global_label "HT_TAP" (shape input) (at 151.836 177.502 180)
     (effects (font (size 1.27 1.27)) (justify right)))
   (wire (pts (xy 151.836 177.502) (xy 155.646 177.502))
