File: amps/aa1164/schematic.kicad_sch (KiCad schematic)
At the start: 95 parts, among them SW1 SPST, SW2 SPDT

Commit message: Fix: the AA1164 sheet strapped the Speed control at the wrong lug and lettered V1's sections backwards
Both faults were the sheet's; the board already drew what the K-FD pages draw,
which is why the sheet-vs-board gate had been carrying them.

Read off the two K-FD pages of D 045427 (the layout page 5734 x 4467, the
circuit page 5554 x 4346 - the cached copies ARE the file's embedded images, so
these are native reads):

- Speed strap. Layout page, crop (2500,500)-(2820,800): the 3.0M-RA control is
  drawn from the rear with its three lugs at the top, a lead arcs from the LEFT
  lug over to the wiper lug, the 100K hangs off that same left lug down to a
  ground triangle inside the control's outline, and the RIGHT lug alone carries
  the long lead to the board. The sheet had the strap on the other end - wiper
  tied to the Speed-node lug, the 100K on the far end. A rheostat either way and
  the same track in circuit, but the wrong lug pair, and the two drawings then
  disagreed over a control they both draw.

- V1's sections. Circuit page, crop (300,480)-(1700,1250): the input triode,
  the one fed through the two 68K stoppers, is lettered plate 1, grid 2,
  cathode 3; the stage after the Volume control is lettered 6 at its plate and
  8 at its cathode. Layout page, crop (4620,2350)-(5050,2780): the 7025 socket
  takes the lead from the Instruments jacks on pin 2 and prints +1.3 V on the
  lead at pin 3. A 12AX7's unit 1 IS pins 6/7/8 (RCA basing 9A), so the input
  stage is unit 2 and the second stage unit 1 - the opposite of the letter-rank
  default the sheet had been taking. Both sections now print the numbers both
  factory pages print.

Gates: check_schematics (0 failures, connectivity clean), verify_schematic_nets
(aa1164 PASS, claimed), verify_sheet_vs_board - aa1164 goes from a SECTION-SWAP
plus its MISPLACED survivors to "sheet and board draw the same circuit over
every anchored and resolved part"; test_era_values, check_value_consistency
--strict, check_ton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
Parts:
- V1A: Basing_unit (none) -> 2
- V1B: Basing_unit (none) -> 1
Connections:
- net at CTO1.2, CTO2.2, VRSPD.1: no longer VRSPD.2 (W)
- net at RSPD.1, VRSPD.3: now also VRSPD.2 (W)
Changed lines of the file:
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@@
     (in_bom yes) (on_board yes)
     (property "Reference" "V1A" (at 66.4724 38.35 0) (effects (font (size 1.27 1.27)) (justify left)))
-    (property "Value" "12AX7 (7025)" (at 66.4724 40.75 0) (effects (font (size 1.27 1.27)) (justify left))))
+    (property "Value" "12AX7 (7025)" (at 66.4724 40.75 0) (effects (font (size 1.27 1.27)) (justify left)))
+    (property "Basing_unit" "2" (at 66.4724 43.15 0) (effects (font (size 1.27 1.27)) hide)))
   (wire (pts (xy 46.4724 44.75) (xy 52.8524 44.75))
     (stroke (width 0) (type default)))
@@
     (in_bom yes) (on_board yes)
     (property "Reference" "V1B" (at 170.472 38.35 0) (effects (font (size 1.27 1.27)) (justify left)))
-    (property "Value" "12AX7 (7025)" (at 170.472 40.75 0) (effects (font (size 1.27 1.27)) (justify left))))
+    (property "Value" "12AX7 (7025)" (at 170.472 40.75 0) (effects (font (size 1.27 1.27)) (justify left)))
+    (property "Basing_unit" "1" (at 170.472 43.15 0) (effects (font (size 1.27 1.27)) hide)))
   (wire (pts (xy 152.472 44.75) (xy 156.852 44.75))
     (stroke (width 0) (type default)))
@@
     (property "Reference" "VRSPD" (at 105.872 275.15 270) (effects (font (size 1.27 1.27)) (justify left)))
     (property "Value" "3M speed" (at 105.872 277.55 270) (effects (font (size 1.27 1.27)) (justify left))))
-  (wire (pts (xy 110.472 263.67) (xy 106.662 263.67))
-    (stroke (width 0) (type default)))
-  (wire (pts (xy 106.662 263.67) (xy 106.662 268.75))
-    (stroke (width 0) (type default)))
-  (junction (at 106.662 268.75) (diameter 1.548) (color 0 0 0 0))
   (symbol (lib_id "cx:R") (at 120.472 268.75 90) (unit 1)
     (in_bom yes) (on_board yes)
     (property "Reference" "RSPD" (at 117.272 262.75 270) (effects (font (size 1.27 1.27)) (justify left)))
     (property "Value" "100k" (at 117.272 265.15 270) (effects (font (size 1.27 1.27)) (justify left))))
-  (wire (pts (xy 114.282 268.75) (xy 116.662 268.75))
-    (stroke (width 0) (type default)))
+  (wire (pts (xy 114.282 268.75) (xy 115.472 268.75))
+    (stroke (width 0) (type default)))
+  (wire (pts (xy 115.472 268.75) (xy 116.662 268.75))
+    (stroke (width 0) (type default)))
+  (wire (pts (xy 110.472 263.67) (xy 115.472 263.67))
+    (stroke (width 0) (type default)))
+  (wire (pts (xy 115.472 263.67) (xy 115.472 268.75))
+    (stroke (width 0) (type default)))
+  (junction (at 115.472 268.75) (diameter 1.548) (color 0 0 0 0))
   (wire (pts (xy 124.282 268.75) (xy 126.472 268.75))
     (stroke (width 0) (type default)))
@@
   (polyline (pts (xy 252.572 49.105) (xy 254.472 47.505) (xy 260.472 49.585) (xy 266.472 47.505) (xy 268.372 49.105))
     (stroke (width 0.524) (type default) (color 197 163 255 1)) (fill (type none)))
-  (text "6" (at 61.3224 38.4 0)
+  (text "1" (at 61.3224 38.4 0)
     (effects (font (size 1.1 1.1)) (justify left)))
-  (text "7" (at 53.5252 43.35 0)
+  (text "2" (at 53.5252 43.35 0)
     (effects (font (size 1.1 1.1)) (justify left)))
-  (text "8" (at 61.3224 51.1 0)
+  (text "3" (at 61.3224 51.1 0)
     (effects (font (size 1.1 1.1)) (justify left)))
-  (text "1" (at 165.322 38.4 0)
+  (text "6" (at 165.322 38.4 0)
     (effects (font (size 1.1 1.1)) (justify left)))
-  (text "2" (at 157.525 43.35 0)
+  (text "7" (at 157.525 43.35 0)
     (effects (font (size 1.1 1.1)) (justify left)))
-  (text "3" (at 165.322 51.1 0)
+  (text "8" (at 165.322 51.1 0)
     (effects (font (size 1.1 1.1)) (justify left)))
   (text "6" (at 255.322 40.52 0)

Commit message: AA1164: input leak at jack 1's tip, reverb pedal on the recovery grid (V1 audit)
K-FD hangs the 1M from jack 1's tip, jack side of its 68k (schematic
5554x4346 crop 200,550,1500,900; layout 5734x4467 crop 4600,450,650,600);
the sheet had it on the grid bus. R1a is declared a series_bridge so the
netlist's RGN1 GN1 0 still binds, as on the 5F4. The reverb pedal jack is
wired to the Reverb Output tip, the recovery grid (crops 1300,2450,600,900
and layout 3200,2850,1200,400); the sheet had it on the Reverb wiper. The
BOM's 'one jack symbol' note is corrected. No DC node moves.

Co-Authored-By: Claude Opus 5.5 <noreply@anthropic.com>
Claude-Session: https://claude.ai/code/session_01KBMfdh37HmCL2iWcBiL5J1
Signed-off-by: AnalogMaker <theanalogmaker@gmail.com>
Parts:
- removed CDEATH: .047u, symbol cx:C
- removed CF2, CF3: 20u, symbol cx:C
- removed CTO4: .02u, symbol cx:C
- removed F1: 1A SB, symbol cx:FUSE
- removed RB2: 22k, symbol cx:R
- removed RGR1: 220k, symbol cx:R
- removed RH1: 100, symbol cx:R
- removed RKPI: 1k, symbol cx:R
- removed RTO1: 1M, symbol cx:R
- removed V4A: 12AX7, symbol cx:TRIODE
- removed VRREV: 100k rev, symbol cx:POT
- removed VRT: 250k treb, symbol cx:POT
- added CINT: .1u, symbol cx:C
- added CKR1: 25u, symbol cx:C
- added JREV: reverb fsw, symbol cx:JACK
- added JVIB: vibrato fsw, symbol cx:JACK
- added RB1: 100k 5%, symbol cx:R
- added RD1, RD2: 18k 1W, symbol cx:R
- added RH2: 100, symbol cx:R
- added RS: 100k, symbol cx:R
- added RTAIL: 56k, symbol cx:R
- added RTOP: 220k, symbol cx:R
- added SW1: SPST, symbol cx:SWITCH
- added SW2: SPDT, symbol cx:SWITCH
- CDEATH: renamed from SW2; value SPDT -> .047u; symbol cx:SWITCH -> cx:C
- CF2: renamed from RD1; value 18k 1W -> 20u; symbol cx:R -> cx:C
- CF3: renamed from RD2; value 18k 1W -> 20u; symbol cx:R -> cx:C
- CTO4: renamed from CINT; value .1u -> .02u
- DB1: renamed from RB1; value 100k 5% -> Si; symbol cx:R -> cx:DIODE_SS
- F1: renamed from SW1; value SPST -> 1A SB; symbol cx:SWITCH -> cx:FUSE
- RB2: renamed from DB1; value Si -> 22k; symbol cx:DIODE_SS -> cx:R
- RGR1: renamed from CKR1; value 25u -> 220k; symbol cx:C -> cx:R
- RKPI: renamed from RTAIL; value 56k -> 1k
- RTO1: renamed from JVIB; value vibrato fsw -> 1M; symbol cx:JACK -> cx:R
- V4A: renamed from RTOP; value 220k -> 12AX7; symbol cx:R -> cx:TRIODE; Basing_unit (none) -> 2
- VRREV: renamed from JREV; value reverb fsw -> 100k rev; symbol cx:JACK -> cx:POT
- VRT: renamed from RS; value 100k -> 250k treb; symbol cx:R -> cx:POT
- renumbered RH2 to RH1
Connections:
- net AC LINE: now also F1.1
- net B+2: now also RD1.1, RTOP.1; no longer V4A.1
- net B+3: now also RD1.2, RD2.1; no longer CF2.2
- net B+4: now also RD2.2; no longer CF3.2
- net BIAS FILTER: now also DB1.1 (A)
- net GND: now also CF2.2, CF3.2, CTO4.2, RB2.2, RGN1.1, RH1.2, VRREV.3, CKR1.2, JREV.2 (S), JVIB.2 (S), RH2.1, RTAIL.2, SW2.2; no longer CDEATH.2, RGN1.2, RH1.1, RKPI.2, VRREV.2 (S)
- net HTR_A: now also RH1.1
- net HTR_B: now also RH2.2; no longer RH1.2
- net HT_B: now also RB1.2; no longer DB1.2
- net INPUT 1: now also RGN1.2
- net MAINS: now also SW1.2; no longer F1.2
- net MAINS N: now also CDEATH.1
- net at R1a.2, R1b.2, V1A.2 (G): no longer RGN1.1
- net at RKPI.1: now also C2.1, V4B.3 (K); no longer RGPI.2
- net at CCR1.2: now also VRREV.1
- net at CTO1.1, RTOUT.1: now also V4A.1 (P), RTOP.2; no longer V4A.2
- net at CTO4.1, RTOUT.2: now also CINT.1
- net at CT.1, RLN1.2, V1A.1 (P): now also RS.1; no longer VRT.1
- net at CT.2: now also VRT.1
- net at TANK.3 (OUT_H), V3A.2 (G): now also RGR1.1, JREV.1 (T)
- net at RKR1.1, V3A.3 (K): now also CKR1.1; no longer RGR1.1
- net at VRVOL.1: now also VRT.2 (W)
- net at CB1.2, VRB.1, VRB.2 (W): now also VRT.3
- net at CTO3.1: now also RTO1.1, V4A.2 (G)
- net at CB1.1, CB2.1: now also RS.2; no longer VRT.2
- net at CKTO.1, RKTO.1, RTO2.1: now also V4A.3 (K)
- net at RMR.1: now also VRREV.2 (W); no longer VRREV.1 (T)
- net at CTO2.1, CTO3.2, RTO2.2: now also JVIB.1 (T); no longer RTO1.1 (T)
- net at VRINT.1: now also CINT.2; no longer CTO4.2
- new net: F1.2, SW1.1
- new net: RGPI.2, RKPI.2, RTAIL.1
- new net: CDEATH.2, SW2.1
- new net: DB1.2 (K), RB1.1
Other:
- moved on the sheet: CTO4, R1a, RH1, RKPI
Changed lines of the file:
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@@
   (global_label "INPUT 1" (shape input) (at 20.4724 40.75 180)
     (effects (font (size 1.27 1.27)) (justify right)))
-  (symbol (lib_id "cx:R") (at 32.4724 40.75 90) (unit 1)
-    (in_bom yes) (on_board yes)
-    (property "Reference" "R1a" (at 29.2724 34.75 270) (effects (font (size 1.27 1.27)) (justify left)))
-    (property "Value" "68k" (at 29.2724 37.15 270) (effects (font (size 1.27 1.27)) (justify left))))
-  (wire (pts (xy 20.4724 40.75) (xy 28.6624 40.75))
-    (stroke (width 0) (type default)))
-  (wire (pts (xy 36.2824 40.75) (xy 46.4724 40.75))
-    (stroke (width 0) (type default)))
+  (symbol (lib_id "cx:R") (at 38.4724 40.75 90) (unit 1)
+    (in_bom yes) (on_board yes)
+    (property "Reference" "R1a" (at 35.2724 34.75 270) (effects (font (size 1.27 1.27)) (justify left)))
+    (property "Value" "68k" (at 35.2724 37.15 270) (effects (font (size 1.27 1.27)) (justify left))))
+  (wire (pts (xy 20.4724 40.75) (xy 26.4724 40.75))
+    (stroke (width 0) (type default)))
+  (wire (pts (xy 26.4724 40.75) (xy 34.6624 40.75))
+    (stroke (width 0) (type default)))
+  (wire (pts (xy 42.2824 40.75) (xy 46.4724 40.75))
+    (stroke (width 0) (type default)))
+  (junction (at 26.4724 40.75) (diameter 1.548) (color 0 0 0 0))
+  (symbol (lib_id "cx:R") (at 26.4724 36.94 0) (unit 1)
+    (in_bom yes) (on_board yes)
+    (property "Reference" "RGN1" (at 28.6724 36.94 0) (effects (font (size 1.27 1.27)) (justify left)))
+    (property "Value" "1M" (at 28.6724 39.34 0) (effects (font (size 1.27 1.27)) (justify left))))
+  (global_label "GND" (shape input) (at 26.4724 33.13 90)
+    (effects (font (size 1.27 1.27)) (justify left)))
   (global_label "INPUT 2" (shape input) (at 20.4724 48.75 180)
     (effects (font (size 1.27 1.27)) (justify right)))
-  (symbol (lib_id "cx:R") (at 32.4724 48.75 90) (unit 1)
-    (in_bom yes) (on_board yes)
-    (property "Reference" "R1b" (at 29.2724 42.75 270) (effects (font (size 1.27 1.27)) (justify left)))
-    (property "Value" "68k" (at 29.2724 45.15 270) (effects (font (size 1.27 1.27)) (justify left))))
-  (wire (pts (xy 20.4724 48.75) (xy 28.6624 48.75))
-    (stroke (width 0) (type default)))
-  (wire (pts (xy 36.2824 48.75) (xy 46.4724 48.75))
+  (symbol (lib_id "cx:R") (at 38.4724 48.75 90) (unit 1)
+    (in_bom yes) (on_board yes)
+    (property "Reference" "R1b" (at 35.2724 42.75 270) (effects (font (size 1.27 1.27)) (justify left)))
+    (property "Value" "68k" (at 35.2724 45.15 270) (effects (font (size 1.27 1.27)) (justify left))))
+  (wire (pts (xy 20.4724 48.75) (xy 34.6624 48.75))
+    (stroke (width 0) (type default)))
+  (wire (pts (xy 42.2824 48.75) (xy 46.4724 48.75))
     (stroke (width 0) (type default)))
   (wire (pts (xy 46.4724 40.75) (xy 46.4724 44.75))
@@
     (stroke (width 0) (type default)))
   (junction (at 46.4724 44.75) (diameter 1.548) (color 0 0 0 0))
-  (symbol (lib_id "cx:R") (at 46.4724 52.56 0) (unit 1)
-    (in_bom yes) (on_board yes)
-    (property "Reference" "RGN1" (at 48.6724 49.36 0) (effects (font (size 1.27 1.27)) (justify left)))
-    (property "Value" "1M" (at 48.6724 51.76 0) (effects (font (size 1.27 1.27)) (justify left))))
-  (global_label "GND" (shape input) (at 46.4724 56.37 270)
-    (effects (font (size 1.27 1.27)) (justify right)))
   (symbol (lib_id "cx:TRIODE") (at 60.4724 44.75 0) (unit 1)
     (in_bom yes) (on_board yes)
@@
   (global_label "GND" (shape input) (at 122.472 102.29 270)
     (effects (font (size 1.27 1.27)) (justify right)))
-  (wire (pts (xy 118.632 97.21) (xy 132.472 97.21))
+  (wire (pts (xy 118.632 97.21) (xy 126.472 97.21))
+    (stroke (width 0) (type default)))
+  (wire (pts (xy 126.472 97.21) (xy 132.472 97.21))
     (stroke (width 0) (type default)))
   (wire (pts (xy 132.472 97.21) (xy 132.472 104.75))
     (stroke (width 0) (type default)))
+  (junction (at 126.472 97.21) (diameter 1.548) (color 0 0 0 0))
+  (symbol (lib_id "cx:JACK") (at 116.472 120.75 0) (mirror y) (unit 1)
+    (in_bom yes) (on_board yes)
+    (property "Reference" "JREV" (at 112.472 114.15 0) (effects (font (size 1.27 1.27)) (justify left)))
+    (property "Value" "reverb fsw" (at 112.472 116.55 0) (effects (font (size 1.27 1.27)) (justify left))))
+  (wire (pts (xy 126.472 97.21) (xy 126.472 118.21))
+    (stroke (width 0) (type default)))
+  (wire (pts (xy 126.472 118.21) (xy 121.552 118.21))
+    (stroke (width 0) (type default)))
+  (global_label "GND" (shape input) (at 121.552 123.29 270)
+    (effects (font (size 1.27 1.27)) (justify right)))
   (symbol (lib_id "cx:TRIODE") (at 144.472 104.75 0) (unit 1)
     (in_bom yes) (on_board yes)
@@
   (wire (pts (xy 173.552 97.46) (xy 180.472 97.46))
     (stroke (width 0) (type default)))
-  (junction (at 180.472 97.46) (diameter 1.548) (color 0 0 0 0))
   (symbol (lib_id "cx:R") (at 186.472 97.46 90) (unit 1)
     (in_bom yes) (on_board yes)
@@
   (global_label "MIXG" (shape input) (at 198.472 97.46 0)
     (effects (font (size 1.27 1.27)) (justify left)))
-  (symbol (lib_id "cx:JACK") (at 208.472 112.75 0) (unit 1)
-    (in_bom yes) (on_board yes)
-    (property "Reference" "JREV" (at 211.472 106.15 0) (effects (font (size 1.27 1.27)) (justify left)))
-    (property "Value" "reverb fsw" (at 211.472 108.55 0) (effects (font (size 1.27 1.27)) (justify left))))
-  (wire (pts (xy 180.472 97.46) (xy 180.472 110.21))
-    (stroke (width 0) (type default)))
-  (wire (pts (xy 180.472 110.21) (xy 203.392 110.21))
-    (stroke (width 0) (type default)))
-  (wire (pts (xy 203.392 115.29) (xy 198.472 115.29))
-    (stroke (width 0) (type default)))
-  (global_label "GND" (shape input) (at 198.472 115.29 270)
-    (effects (font (size 1.27 1.27)) (justify right)))
   (text "Bias supply — 100 k feed off the HT winding, silicon rectifier, 25 µF can, 22 k bleeder; the Intensity control's track ends here and its wiper is the -34 V line" (at 258.472 98.75 0)
     (effects (font (size 1.3 1.3)) (justify left)))
