File: amps/ab763-twin/schematic.kicad_sch (KiCad schematic)
At the start: 130 parts, among them T1 125P34A · 340-0-340 V, T2 125C1A, T3 125A29A, T4 125A20B

Commit message: AB763 Twin: input leaks at jack 1's tip; mains fuse in the BOM (V1 audit)
C-FD hangs each channel's 1M from jack 1's tip, jack side of its 68k
(schematic 6138x4384, Normal crop 230,950,760,1650; the Vibrato pair is
drawn the same at 230,2050,760,2750): jack 2's contact -> jack 1's tip,
jack 1's contact -> ground. The sheet had both leaks on the grid bus.
R1n/R1v are declared series_bridge so the netlist's RGN1 GN1 0 and
RGV1 GV1 0 still bind (the AA1164 idiom). The board already mounts both
leaks at the jacks, off the eyelet board. The BOM's 'one jack per
channel' note is corrected, and the 2½ A slo-blo mains fuse both pages
print (schematic crop 3900,3900,4700,4300) is added. No DC node moves.

Co-Authored-By: Claude Opus 5.5 <noreply@anthropic.com>
Claude-Session: https://claude.ai/code/session_01KBMfdh37HmCL2iWcBiL5J1
Signed-off-by: AnalogMaker <theanalogmaker@gmail.com>
Parts:
- removed CBV, CCD1: .1u, symbol cx:C
- removed CKRD, CKTO1, CKTO2: 25u, symbol cx:C
- removed CPIA: .001u, symbol cx:C
- removed CTO1: .01u, symbol cx:C
- removed CTV: 250p, symbol cx:C
- removed R2v: 68k, symbol cx:R
- removed RBAL1: 220k 1W, symbol cx:R
- removed RBIAS: 470 1W, symbol cx:R
- removed RFB2: 820, symbol cx:R
- removed RLPA: 82k 5%, symbol cx:R
- removed RLV1: 100k, symbol cx:R
- removed RST1, RST2, RST3, RST4: 1.5k, symbol cx:R
- removed RTAIL: 470, symbol cx:R
- removed V1B: 12AX7 (7025), symbol cx:TRIODE
- added C11: 70u 350V, symbol cx:C
- added CB1: 25u 50V, symbol cx:C
- added RGPA, RGV1, RTOG1: 1M, symbol cx:R
- added RKV1: 1.5k, symbol cx:R
- added RLN2: 100k, symbol cx:R
- added RLPB: 100k 5%, symbol cx:R
- added RSC1, RSC2, RSC3, RSC4: 470 1W, symbol cx:R
- added RT22: 22k, symbol cx:R
- added RTO10: 10M, symbol cx:R
- added T4: 125A20B, symbol cx:OT_SE
- added V6B: 12AT7, symbol cx:TRIODE
- added VRBV: 250k-A bass, symbol cx:POT
- added VRINT: 50k-RA int, symbol cx:POT
- added VRSPD: 3M-RA speed, symbol cx:POT
- added VRTV: 250k-A treb, symbol cx:POT
- CBV: renamed from VRBV; value 250k-A bass -> .1u; symbol cx:POT -> cx:C
- CCD1: renamed from RMIXV; value 220k -> .1u; symbol cx:R -> cx:C
- CKRD: renamed from T4; value 125A20B -> 25u; symbol cx:OT_SE -> cx:C
- CKTO1: renamed from CTO3; value .02u -> 25u
- CKTO2: renamed from RTO10; value 10M -> 25u; symbol cx:R -> cx:C
- CPIA: renamed from V6B; value 12AT7 -> .001u; symbol cx:TRIODE -> cx:C
- CTO1: renamed from RTOG1; value 1M -> .01u; symbol cx:R -> cx:C
- CTO3: renamed from VRSPD; value 3M-RA speed -> .02u; symbol cx:POT -> cx:C
- CTV: renamed from VRTV; value 250k-A treb -> 250p; symbol cx:POT -> cx:C
- DBIAS: renamed from CB1; value 25u 50V -> Si; symbol cx:C -> cx:DIODE_SS
- R2v: renamed from RGV1; value 1M -> 68k
- RBAL1: renamed from C11; value 70u 350V -> 220k 1W; symbol cx:C -> cx:R
- RBIAS: renamed from DBIAS; value Si -> 470 1W; symbol cx:DIODE_SS -> cx:R
- RFB2: renamed from RGPA; value 1M -> 820
- RLPA: renamed from RLPB; value 100k 5% -> 82k 5%
- RLV1: renamed from RKV1; value 1.5k -> 100k
- RMIXV: renamed from VRINT; value 50k-RA int -> 220k; symbol cx:POT -> cx:R
- RST1: renamed from RSC1; value 470 1W -> 1.5k
- RST2: renamed from RSC2; value 470 1W -> 1.5k
- RST3: renamed from RSC3; value 470 1W -> 1.5k
- RST4: renamed from RSC4; value 470 1W -> 1.5k
- RTAIL: renamed from RT22; value 22k -> 470
- V1B: renamed from RLN2; value 100k -> 12AX7 (7025); symbol cx:R -> cx:TRIODE
Connections:
- net B+1: now also RBAL1.1
- net B+2: now also RSC1.2, RSC2.2, RSC3.2, RSC4.2, RTO10.1; no longer CKTO2.1, RST1.2, RST2.2, RST3.2, RST4.2
- net B+3: now also RLPB.1
- net B+4: now also RLV1.1, RLN2.1; no longer V1B.1
- net BIAS FILTER: now also CB1.1; no longer RBIAS.1 (A)
- net BIAS TAP: now also RBIAS.1
- net GND: now also CKRD.2, CKTO1.2, CKTO2.2, RGN1.1, C11.2, CB1.2, RGV1.1, RKV1.2, T4.4 (SEC_C), VRINT.3; no longer CKRD.4 (SEC_C), DBIAS.2, R2v.2, RBAL1.2, RGN1.2, RLV1.2, RMIXV.3
- net MIXER: now also CPIA.1, RMIXV.2; no longer CCD1.2
- net NORM 1: now also RGN1.2
- net PHOTOCELL: now also VRINT.2 (W); no longer RMIXV.2 (W)
- net REVERB TANK: now also T4.3 (SEC_H); no longer CKRD.3 (SEC_H)
- net SPKR: now also RFB2.1
- net VIB 1: now also RGV1.2
- net VIB 2: now also R2v.1
- net at C1.2, RGL1.2: now also RST1.1, RST2.1
- net at V7.2 (G1): now also RST1.2
- net at RKRD.1, V3A.3 (K), V3B.3 (K): now also CKRD.1
- net at R1n.2, R2n.2, V1A.2 (G): no longer RGN1.1
- net at CKA.1, RKA.1, V2B.3 (K): now also V1B.3 (K)
- net at RTOG2.1, RTOG3.1: now also RTOG1.1; no longer CTO1.1
- net at RKTO1.1, V5A.3 (K): now also CKTO1.1
- net at C2.2, RGL2.1: now also RST3.1, RST4.1
- net at V9.2 (G1): now also RST3.2
- net at CKV1.1, V2A.3 (K): now also RKV1.1; no longer RLV1.1
- net at R1v.2, V2A.2 (G): now also R2v.2; no longer R2v.1
- net at CBV2.1, RSV.2: now also CBV.1
- net at RTO1.2, V5A.1 (P): now also CTO3.1; no longer CKTO1.1
- net at C10.2, RBAL2.1: now also RBAL1.2, C11.1; no longer RBAL1.1
- net at CPIB.2, RGPB.2: now also V6B.2 (G); no longer CPIA.2 (G)
- net at V6A.3 (K): now also RTAIL.2, V6B.3 (K); no longer CPIA.3 (K)
- net at CTO2.1, V5B.2 (G): now also CTO1.1, RTOG1.2; no longer CTO1.2
- net at OPTO.1 (L1), V5B.1 (P): now also RTO10.2; no longer CKTO2.2
- net at V8.3 (G2): now also RSC2.1; no longer RST2.1
- net at CTO3.2: now also CTO1.2, VRSPD.2 (W); no longer CKTO1.2
- net at V10.2 (G1): now also RST4.2
- net at V10.3 (G2): now also RSC4.1; no longer RST4.1
- net at RLD1.2, V4A.1 (P): now also CCD1.1
- net at RMIXV.1: now also CCD1.2, VRINT.1; no longer CCD1.1
- net at CBRV.1, VRVV.1: now also VRTV.2 (W); no longer CTV.2 (W)
- net at RSV.1, V2A.1 (P): now also CTV.1, RLV1.2
- net at V7.3 (G2): now also RSC1.1; no longer RST1.1
- net at CPIB.1, RFB1.1: now also RFB2.2, RT22.1; no longer RTAIL.1
- net at RKTO2.1, V5B.3 (K): now also CKTO2.1
- net at V6A.2 (G): now also CPIA.2, RGPA.1; no longer RFB2.1
- net at VRMV.1, VRMV.2 (W): now also VRBV.3; no longer CBV.3
- net at CCN2.1: now also V1B.1 (P), RLN2.2; no longer V1B.2
- net at CBRN.2, VRVN.2 (W): now also V1B.2 (G)
- net at V9.3 (G2): now also RSC3.1; no longer RST3.1
- net at RBIAS.2: now also DBIAS.2 (K)
- net at V8.2 (G1): now also RST2.2
- net at C1.1, V6A.1 (P): now also RLPA.2
- net at RTOSP.1: now also VRSPD.3; no longer CTO3.3
- new net: RGPA.2, RGPB.1, RT22.2, RTAIL.1
- new net: C2.1, RLPB.2, V6B.1 (P)
- new net: CTV.2, VRTV.1
- new net: VRBV.1, VRBV.2 (W), VRTV.3
- now unconnected: CBV.2 (W)
Other:
- moved on the sheet: CKTO1, DBIAS, R1n, R2v, RFB2, RLPA, RLV1, RST1, RST2, RST3, RST4, RTAIL
Changed lines of the file:
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@@
   (global_label "NORM 2" (shape input) (at 19.6088 43.889 180)
     (effects (font (size 1.27 1.27)) (justify right)))
-  (symbol (lib_id "cx:R") (at 29.6088 35.889 90) (unit 1)
-    (in_bom yes) (on_board yes)
-    (property "Reference" "R1n" (at 26.4088 29.889 270) (effects (font (size 1.27 1.27)) (justify left)))
-    (property "Value" "68k" (at 26.4088 32.289 270) (effects (font (size 1.27 1.27)) (justify left))))
-  (wire (pts (xy 19.6088 35.889) (xy 25.7988 35.889))
-    (stroke (width 0) (type default)))
-  (wire (pts (xy 33.4188 35.889) (xy 47.6088 35.889))
-    (stroke (width 0) (type default)))
-  (symbol (lib_id "cx:R") (at 29.6088 43.889 90) (unit 1)
-    (in_bom yes) (on_board yes)
-    (property "Reference" "R2n" (at 26.4088 37.889 270) (effects (font (size 1.27 1.27)) (justify left)))
-    (property "Value" "68k" (at 26.4088 40.289 270) (effects (font (size 1.27 1.27)) (justify left))))
-  (wire (pts (xy 19.6088 43.889) (xy 25.7988 43.889))
-    (stroke (width 0) (type default)))
-  (wire (pts (xy 33.4188 43.889) (xy 47.6088 43.889))
+  (symbol (lib_id "cx:R") (at 37.6088 35.889 90) (unit 1)
+    (in_bom yes) (on_board yes)
+    (property "Reference" "R1n" (at 34.4088 29.889 270) (effects (font (size 1.27 1.27)) (justify left)))
+    (property "Value" "68k" (at 34.4088 32.289 270) (effects (font (size 1.27 1.27)) (justify left))))
+  (wire (pts (xy 19.6088 35.889) (xy 25.6088 35.889))
+    (stroke (width 0) (type default)))
+  (wire (pts (xy 25.6088 35.889) (xy 33.7988 35.889))
+    (stroke (width 0) (type default)))
+  (wire (pts (xy 41.4188 35.889) (xy 47.6088 35.889))
+    (stroke (width 0) (type default)))
+  (junction (at 25.6088 35.889) (diameter 1.7) (color 0 0 0 0))
+  (symbol (lib_id "cx:R") (at 25.6088 32.079 0) (unit 1)
+    (in_bom yes) (on_board yes)
+    (property "Reference" "RGN1" (at 27.8088 32.079 0) (effects (font (size 1.27 1.27)) (justify left)))
+    (property "Value" "1M" (at 27.8088 34.479 0) (effects (font (size 1.27 1.27)) (justify left))))
+  (global_label "GND" (shape input) (at 25.6088 28.269 90)
+    (effects (font (size 1.27 1.27)) (justify left)))
+  (symbol (lib_id "cx:R") (at 37.6088 43.889 90) (unit 1)
+    (in_bom yes) (on_board yes)
+    (property "Reference" "R2n" (at 34.4088 37.889 270) (effects (font (size 1.27 1.27)) (justify left)))
+    (property "Value" "68k" (at 34.4088 40.289 270) (effects (font (size 1.27 1.27)) (justify left))))
+  (wire (pts (xy 19.6088 43.889) (xy 33.7988 43.889))
+    (stroke (width 0) (type default)))
+  (wire (pts (xy 41.4188 43.889) (xy 47.6088 43.889))
     (stroke (width 0) (type default)))
   (wire (pts (xy 47.6088 35.889) (xy 47.6088 39.889))
@@
     (stroke (width 0) (type default)))
   (junction (at 47.6088 39.889) (diameter 1.7) (color 0 0 0 0))
-  (symbol (lib_id "cx:R") (at 47.6088 47.699 0) (unit 1)
-    (in_bom yes) (on_board yes)
-    (property "Reference" "RGN1" (at 49.8088 44.499 0) (effects (font (size 1.27 1.27)) (justify left)))
-    (property "Value" "1M" (at 49.8088 46.899 0) (effects (font (size 1.27 1.27)) (justify left))))
-  (global_label "GND" (shape input) (at 47.6088 51.509 270)
-    (effects (font (size 1.27 1.27)) (justify right)))
   (symbol (lib_id "cx:TRIODE") (at 59.6088 39.889 0) (unit 1)
     (in_bom yes) (on_board yes)
@@
   (global_label "VIB 2" (shape input) (at 19.6088 101.889 180)
     (effects (font (size 1.27 1.27)) (justify right)))
-  (symbol (lib_id "cx:R") (at 29.6088 93.889 90) (unit 1)
-    (in_bom yes) (on_board yes)
-    (property "Reference" "R1v" (at 26.4088 87.889 270) (effects (font (size 1.27 1.27)) (justify left)))
-    (property "Value" "68k" (at 26.4088 90.289 270) (effects (font (size 1.27 1.27)) (justify left))))
-  (wire (pts (xy 19.6088 93.889) (xy 25.7988 93.889))
-    (stroke (width 0) (type default)))
-  (wire (pts (xy 33.4188 93.889) (xy 47.6088 93.889))
-    (stroke (width 0) (type default)))
-  (symbol (lib_id "cx:R") (at 29.6088 101.889 90) (unit 1)
-    (in_bom yes) (on_board yes)
-    (property "Reference" "R2v" (at 26.4088 95.889 270) (effects (font (size 1.27 1.27)) (justify left)))
-    (property "Value" "68k" (at 26.4088 98.289 270) (effects (font (size 1.27 1.27)) (justify left))))
-  (wire (pts (xy 19.6088 101.889) (xy 25.7988 101.889))
-    (stroke (width 0) (type default)))
-  (wire (pts (xy 33.4188 101.889) (xy 47.6088 101.889))
+  (symbol (lib_id "cx:R") (at 37.6088 93.889 90) (unit 1)
+    (in_bom yes) (on_board yes)
+    (property "Reference" "R1v" (at 34.4088 87.889 270) (effects (font (size 1.27 1.27)) (justify left)))
+    (property "Value" "68k" (at 34.4088 90.289 270) (effects (font (size 1.27 1.27)) (justify left))))
+  (wire (pts (xy 19.6088 93.889) (xy 25.6088 93.889))
+    (stroke (width 0) (type default)))
+  (wire (pts (xy 25.6088 93.889) (xy 33.7988 93.889))
+    (stroke (width 0) (type default)))
+  (wire (pts (xy 41.4188 93.889) (xy 47.6088 93.889))
+    (stroke (width 0) (type default)))
+  (junction (at 25.6088 93.889) (diameter 1.7) (color 0 0 0 0))
+  (symbol (lib_id "cx:R") (at 25.6088 90.079 0) (unit 1)
+    (in_bom yes) (on_board yes)
+    (property "Reference" "RGV1" (at 27.8088 90.079 0) (effects (font (size 1.27 1.27)) (justify left)))
+    (property "Value" "1M" (at 27.8088 92.479 0) (effects (font (size 1.27 1.27)) (justify left))))
+  (global_label "GND" (shape input) (at 25.6088 86.269 90)
+    (effects (font (size 1.27 1.27)) (justify left)))
+  (symbol (lib_id "cx:R") (at 37.6088 101.889 90) (unit 1)
+    (in_bom yes) (on_board yes)
+    (property "Reference" "R2v" (at 34.4088 95.889 270) (effects (font (size 1.27 1.27)) (justify left)))
+    (property "Value" "68k" (at 34.4088 98.289 270) (effects (font (size 1.27 1.27)) (justify left))))
+  (wire (pts (xy 19.6088 101.889) (xy 33.7988 101.889))
+    (stroke (width 0) (type default)))
+  (wire (pts (xy 41.4188 101.889) (xy 47.6088 101.889))
     (stroke (width 0) (type default)))
   (wire (pts (xy 47.6088 93.889) (xy 47.6088 97.889))
@@
     (stroke (width 0) (type default)))
   (junction (at 47.6088 97.889) (diameter 1.7) (color 0 0 0 0))
-  (symbol (lib_id "cx:R") (at 47.6088 105.699 0) (unit 1)
-    (in_bom yes) (on_board yes)
-    (property "Reference" "RGV1" (at 49.8088 102.499 0) (effects (font (size 1.27 1.27)) (justify left)))
-    (property "Value" "1M" (at 49.8088 104.899 0) (effects (font (size 1.27 1.27)) (justify left))))
-  (global_label "GND" (shape input) (at 47.6088 109.509 270)
-    (effects (font (size 1.27 1.27)) (justify right)))
   (symbol (lib_id "cx:TRIODE") (at 59.6088 97.889 0) (unit 1)
     (in_bom yes) (on_board yes)
