File: amps/aa964/schematic.kicad_sch (KiCad schematic)
At the start: 69 parts, among them SW1 AC sw, SW2 gnd sw

Commit message: AA964: input leak at jack 1's tip; pedal role, bias-feed tolerance (V1 audit)
L-FD hangs the 1M from jack 1's tip, jack side of its 68k (cited
schematic 1471x934, crop 60,160,300,420; cited layout 2166x1591 puts the
1M inside jack 1's ring): jack 2's contact -> jack 1's tip, jack 1's
contact -> ground. The sheet had it on the grid bus. R1n is declared a
series_bridge so the netlist's RG1A G1A 0 still binds. The board already
mounts the leak at the jacks.

BOM: the vibrato pedal grounds the phase-shift ladder's middle node
(CTO2/CTO3/RTO1), as both surfaces already draw it, not the oscillator
grid (schematic crop 0,520,960,760); the bias feed is 100K 5% on the
layout (crop 270,430,660,600). A draw-script comment that cited the
uncited I-FD capture's dimensions as the L-FD drawing is corrected. No
DC node moves.

Co-Authored-By: Claude Opus 5.5 <noreply@anthropic.com>
Claude-Session: https://claude.ai/code/session_01KBMfdh37HmCL2iWcBiL5J1
Signed-off-by: AnalogMaker <theanalogmaker@gmail.com>
Parts:
- removed CB, CC: 20u, symbol cx:C
- removed FUSE: 1A SB, symbol cx:FUSE
- removed RBF: 100k 5%, symbol cx:R
- removed RG1A, RTO2: 1M, symbol cx:R
- removed RKPI: 1k, symbol cx:R
- removed SW2: gnd sw, symbol cx:SWITCH
- removed V2A: 12AX7, symbol cx:TRIODE
- added CDEATH: .047u 600V, symbol cx:C
- added DBIAS: Si, symbol cx:DIODE_SS
- added RD2, RD3: 18k 1W, symbol cx:R
- added RGPI, RTO1: 1M, symbol cx:R
- added RTO: 220k, symbol cx:R
- added SW1: AC sw, symbol cx:SWITCH
- added V1A: 7025, symbol cx:TRIODE
- CB: renamed from RD2; value 18k 1W -> 20u; symbol cx:R -> cx:C
- CC: renamed from RD3; value 18k 1W -> 20u; symbol cx:R -> cx:C
- FUSE: renamed from SW1; value AC sw -> 1A SB; symbol cx:SWITCH -> cx:FUSE
- RBF: renamed from DBIAS; value Si -> 100k 5%; symbol cx:DIODE_SS -> cx:R
- RG1A: renamed from V1A; value 7025 -> 1M; symbol cx:TRIODE -> cx:R; Basing_unit 2 -> (none)
- RKPI: renamed from RTAIL; value 56k -> 1k
- RTAIL: renamed from RGPI; value 1M -> 56k
- SW2: renamed from CDEATH; value .047u 600V -> gnd sw; symbol cx:C -> cx:SWITCH
- V2A: renamed from RTO; value 220k -> 12AX7; symbol cx:R -> cx:TRIODE; Basing_unit (none) -> 2
- renumbered RTO1 to RTO2
Connections:
- net AC 117 V: now also FUSE.1
- net AC N: now also SW2.1
- net B+2: now also RD2.1, RTO.1; no longer V2A.1
- net B+3: now also RD2.2, RD3.1; no longer CB.2
- net B+4: now also RD3.2; no longer CC.2
- net BIAS: now also DBIAS.1 (A); no longer RBF.1 (A)
- net GND: now also CB.2, CC.2, RG1A.2, RTAIL.2, RTO2.2, CDEATH.2; no longer RKPI.2, SW2.2
- net HT_B: now also RBF.1
- net INPUT 1: now also RG1A.1
- net MAINS: now also SW1.2; no longer FUSE.2
- net at CTO1.1, RTOUT.2: now also V2A.1 (P), RTO.2; no longer V2A.2
- net at CTO3.1: now also RTO2.1, V2A.2 (G)
- net at CKTO.1, RKTO.1: now also V2A.3 (K), RTO1.1; no longer RTO2.1
- net at R1n.2, R2n.2: now also V1A.2 (G); no longer RG1A.2 (G)
- net at RBF.2: now also DBIAS.2 (K)
- net at C2.1, V2B.3 (K): now also RKPI.1
- net at CT.1, RL1A.2, RS.1: now also V1A.1 (P); no longer RG1A.1 (P)
- net at CK1A.1, RK1A.1: now also V1A.3 (K); no longer RG1A.3 (K)
- net at CTO2.1, CTO3.2, JVIB.1 (T): now also RTO1.2; no longer RTO2.2
- net at CC1.2, V2B.2 (G): now also RGPI.1; no longer RTAIL.1
- new net: FUSE.2, SW1.1
- new net: CDEATH.1, SW2.2
- new net: RGPI.2, RKPI.2, RTAIL.1
Other:
- moved on the sheet: R1n, RKPI, RTAIL, RTO2
Changed lines of the file:
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@@
   (wire (pts (xy 36.2824 46.7) (xy 48.4724 46.7))
     (stroke (width 0) (type default)))
-  (symbol (lib_id "cx:R") (at 32.4724 54.7 90) (unit 1)
+  (symbol (lib_id "cx:R") (at 38.4724 54.7 90) (unit 1)
     (in_bom yes) (on_board yes)
-    (property "Reference" "R1n" (at 29.2724 48.7 270) (effects (font (size 1.27 1.27)) (justify left)))
-    (property "Value" "68k" (at 29.2724 51.1 270) (effects (font (size 1.27 1.27)) (justify left))))
-  (wire (pts (xy 20.4724 54.7) (xy 28.6624 54.7))
+    (property "Reference" "R1n" (at 35.2724 48.7 270) (effects (font (size 1.27 1.27)) (justify left)))
+    (property "Value" "68k" (at 35.2724 51.1 270) (effects (font (size 1.27 1.27)) (justify left))))
+  (wire (pts (xy 20.4724 54.7) (xy 26.4724 54.7))
     (stroke (width 0) (type default)))
-  (wire (pts (xy 36.2824 54.7) (xy 48.4724 54.7))
+  (wire (pts (xy 26.4724 54.7) (xy 34.6624 54.7))
+    (stroke (width 0) (type default)))
+  (wire (pts (xy 42.2824 54.7) (xy 48.4724 54.7))
     (stroke (width 0) (type default)))
   (wire (pts (xy 48.4724 46.7) (xy 48.4724 50.7))
@@
     (stroke (width 0) (type default)))
   (junction (at 48.4724 50.7) (diameter 1.448) (color 0 0 0 0))
-  (symbol (lib_id "cx:R") (at 48.4724 58.51 0) (unit 1)
+  (junction (at 26.4724 54.7) (diameter 1.448) (color 0 0 0 0))
+  (symbol (lib_id "cx:R") (at 26.4724 58.51 0) (unit 1)
     (in_bom yes) (on_board yes)
-    (property "Reference" "RG1A" (at 50.6724 55.31 0) (effects (font (size 1.27 1.27)) (justify left)))
-    (property "Value" "1M" (at 50.6724 57.71 0) (effects (font (size 1.27 1.27)) (justify left))))
-  (global_label "GND" (shape input) (at 48.4724 62.32 270)
+    (property "Reference" "RG1A" (at 28.6724 58.51 0) (effects (font (size 1.27 1.27)) (justify left)))
+    (property "Value" "1M" (at 28.6724 60.91 0) (effects (font (size 1.27 1.27)) (justify left))))
+  (global_label "GND" (shape input) (at 26.4724 62.32 270)
     (effects (font (size 1.27 1.27)) (justify right)))
   (symbol (lib_id "cx:TRIODE") (at 60.4724 50.7 0) (unit 1)
