File: amps/ab763/schematic.kicad_sch (KiCad schematic)
At the start: 119 parts, among them T1 125P33A, T2 125C3A, T3 125A1A, T4 125A20B

Commit message: Fix: the AB763 board joined the +420 V and +415 V eyelets with a bare wire
The board stood the off-board choke in with one run, C10.a to C11.a, so the reservoir (B+1) and the post-choke node (B+2) were one net and the gate merged C11, RS1, RS2, RTO10 and RTO2 into B+1. Read the C-FD layout (refs 2026-09-27-p4/ab763-1.png, 4400x3400), crop (1480,1580)-(2000,2200): the board's left end letters two eyelets, '+420 V.' with a RED lead and '+415 V' with a YELLOW lead, both running off the board to the choke. The board now runs C10.a to the choke stub's RED lead and its YELLOW lead to C11.a; the OT centre tap stays on C10.a.

The same split exposed one sheet error the gate cannot see (transformer leads have no board vocabulary). The C-FD schematic (ab763-2.png, 4400x3400), crop (780,2250)-(1200,2850), runs TR4's B+ lead to box [B]; crop (2400,1700)-(3300,2100) puts [B] on the post-choke side of TR2. The sheet hung T4's primary on B+1; it now lands on B+2, where the board's T4.red and the AB763 Twin sheet already have it. Both rails are the netlist's BP1, so no netlist or voltage change; schematic and wiring gates pass. FW-19 P10b.

Co-Authored-By: Claude Opus 5.5 <noreply@anthropic.com>
Claude-Session: https://claude.ai/code/session_01KBMfdh37HmCL2iWcBiL5J1
Signed-off-by: AnalogMaker <theanalogmaker@gmail.com>
Changed lines of the file:
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@@
   (wire (pts (xy 94.7188 126.818) (xy 94.7188 130.278))
     (stroke (width 0) (type default)))
-  (global_label "B+1" (shape input) (at 94.7188 130.278 90)
+  (global_label "B+2" (shape input) (at 94.7188 130.278 90)
     (effects (font (size 1.27 1.27)) (justify left)))
   (wire (pts (xy 112.499 121.738) (xy 117.609 121.738))

Commit message: Fix: the AB763 6V6 grids take 1.5 kΩ stoppers, and its bias supply has one 25 µF can
V1 source audit (docs/plans/active/2026-10-03-verification-hardening/ab763.md),
read on the C-FD natives extracted from refs/2026-09-27-p4/ab763_cfd.pdf
(schematic 6070x4274, layout 6026x3650):

- The schematic letters "1500" in each 6V6 grid lead, between the 220K leak /
  0.1 coupler node and the grid (crop 3700,610,5460,2360), and the layout mounts
  one 1500 on each 6V6 socket, pin 5 to the pin-1 tie lug (750,2350,1800,2900).
  The corpus had neither. R7s/R8s are added to the parts list and the sheet and
  declared series_bridge in sch_map.yaml, the way the 5E3 and 5F10 carry their
  socket-mounted 1.5k stoppers; the netlist runs G61/G62 through them.
- The bias filter is one capacitor. The schematic draws a single symbol
  lettered "-25 / +50" and the layout's bias sub-box a single can "25 50"
  (crops 4300,2850,4800,3500 and 500,1050,1500,1500): 25 µF at 50 V. The corpus
  had split it into CB1 25 µF and a phantom CB2 50 µF; CB2 is removed from the
  parts list, sheet, board scope list and notes.

The sheet and the board shared both errors, so no gate could see them.
Stoppers carry no DC grid current and capacitors are open at DC: no operating
point moves.

Co-Authored-By: Claude Opus 5.5 <noreply@anthropic.com>
Claude-Session: https://claude.ai/code/session_01KBMfdh37HmCL2iWcBiL5J1
Signed-off-by: AnalogMaker <theanalogmaker@gmail.com>
Parts:
- removed C10: 16u, symbol cx:C
- removed CB2: 50u, symbol cx:C
- removed RGL2: 220k, symbol cx:R
- removed V7: 6V6GT, symbol cx:PENTODE
- added R7s, R8s: 1.5k, symbol cx:R
- added RGL1: 220k, symbol cx:R
- added T2: 125C3A, symbol cx:CHOKE
- added T3: 125A1A, symbol cx:OT_PP
- C10: renamed from T2; value 125C3A -> 16u; symbol cx:CHOKE -> cx:C
- RGL2: renamed from RS2; value 470 1W -> 220k
- RS2: renamed from T3; value 125A1A -> 470 1W; symbol cx:OT_PP -> cx:R
- V7: renamed from RGL1; value 220k -> 6V6GT; symbol cx:R -> cx:PENTODE
Connections:
- net -35V: now also RGL2.2, RGL1.2; no longer V7.2
- net B+1: now also T2.1, T3.2 (CT); no longer RS2.2 (CT)
- net B+2: now also RS2.2, T2.2; no longer C10.2, RGL2.2
- net GND: now also C10.2, V7.4 (K), T3.5 (SEC_C); no longer RS2.5 (SEC_C)
- net SPKR: now also T3.4 (SEC_H); no longer RS2.4 (SEC_H)
- net at C2.2: now also RGL2.1, R8s.1; no longer V8.2 (G1)
- net at RS2.1: now also V8.3 (G2)
- net at V7.1 (P): now also T3.1 (PRI_A); no longer C1.2
- net at RS1.1: now also V7.3 (G2)
- net at V8.1 (P): now also T3.3 (PRI_B); no longer RS2.3 (PRI_B)
- new net: R8s.2, V8.2 (G1)
- new net: C1.2, R7s.1, RGL1.1
- new net: R7s.2, V7.2 (G1)
Other:
- note added: "Bias supply — off an HT tap → -35 V (25u 50 V, 10k-L divider)"
- note removed: "Bias supply — off an HT tap → -35 V (25u/50u, 10k-L divider)"
- moved on the sheet: RGL2
Changed lines of the file:
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@@
   (wire (pts (xy 291.609 97.178) (xy 291.609 116.278))
     (stroke (width 0) (type default)))
-  (wire (pts (xy 291.609 68.278) (xy 319.989 68.278))
+  (symbol (lib_id "cx:R") (at 307.609 68.278 90) (unit 1)
+    (in_bom yes) (on_board yes)
+    (property "Reference" "R7s" (at 304.409 62.278 270) (effects (font (size 1.27 1.27)) (justify left)))
+    (property "Value" "1.5k" (at 304.409 64.678 270) (effects (font (size 1.27 1.27)) (justify left))))
+  (wire (pts (xy 291.609 68.278) (xy 303.799 68.278))
+    (stroke (width 0) (type default)))
+  (wire (pts (xy 311.419 68.278) (xy 319.989 68.278))
     (stroke (width 0) (type default)))
   (symbol (lib_id "cx:PENTODE") (at 327.609 67.643 0) (unit 1)
@@
   (global_label "GND" (shape input) (at 327.609 75.263 270)
     (effects (font (size 1.27 1.27)) (justify right)))
-  (wire (pts (xy 291.609 116.278) (xy 319.989 116.278))
+  (symbol (lib_id "cx:R") (at 307.609 116.278 90) (unit 1)
+    (in_bom yes) (on_board yes)
+    (property "Reference" "R8s" (at 304.409 110.278 270) (effects (font (size 1.27 1.27)) (justify left)))
+    (property "Value" "1.5k" (at 304.409 112.678 270) (effects (font (size 1.27 1.27)) (justify left))))
+  (wire (pts (xy 291.609 116.278) (xy 303.799 116.278))
+    (stroke (width 0) (type default)))
+  (wire (pts (xy 311.419 116.278) (xy 319.989 116.278))
     (stroke (width 0) (type default)))
   (symbol (lib_id "cx:PENTODE") (at 327.609 115.643 0) (unit 1)
@@
   (global_label "GND" (shape input) (at 171.609 241.898 270)
     (effects (font (size 1.27 1.27)) (justify right)))
-  (text "Bias supply — off an HT tap → -35 V (25u/50u, 10k-L divider)" (at 197.609 205.278 0)
+  (text "Bias supply — off an HT tap → -35 V (25u 50 V, 10k-L divider)" (at 197.609 205.278 0)
     (effects (font (size 1.3 1.3)) (justify left)))
   (global_label "HT_B" (shape input) (at 197.609 220.278 180)
@@
   (symbol (lib_id "cx:C") (at 225.609 224.088 0) (unit 1)
     (in_bom yes) (on_board yes)
-    (property "Reference" "CB1" (at 218.928 224.226 0) (effects (font (size 1.27 1.27)) (justify left)))
-    (property "Value" "25u" (at 218.928 226.626 0) (effects (font (size 1.27 1.27)) (justify left))))
+    (property "Reference" "CB1" (at 227.809 220.888 0) (effects (font (size 1.27 1.27)) (justify left)))
+    (property "Value" "25u" (at 227.809 223.288 0) (effects (font (size 1.27 1.27)) (justify left))))
   (global_label "GND" (shape input) (at 225.609 227.898 270)
     (effects (font (size 1.27 1.27)) (justify right)))
-  (junction (at 231.609 220.278) (diameter 1.46) (color 0 0 0 0))
-  (symbol (lib_id "cx:C") (at 231.609 224.088 0) (unit 1)
-    (in_bom yes) (on_board yes)
-    (property "Reference" "CB2" (at 233.809 220.888 0) (effects (font (size 1.27 1.27)) (justify left)))
-    (property "Value" "50u" (at 233.809 223.288 0) (effects (font (size 1.27 1.27)) (justify left))))
-  (global_label "GND" (shape input) (at 231.609 227.898 270)
-    (effects (font (size 1.27 1.27)) (justify right)))
   (wire (pts (xy 231.609 220.278) (xy 234.609 220.278))
